File: RemoteLabs_supervisor_PCB/_autosave-MCU_supervisor.kicad_sch (KiCad schematic)
At the start: 20 parts

Commit message: lunchtime backup
Connections:
- net LATCH: now reaches U?.1 (STROBE)
- net MOSI: now reaches U?.2 (DATA)
- net SCK: now reaches U?.3 (CLOCK)
Changed lines of the file:
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@@
+    (stroke (width 0) (type default) (color 0 0 0 0))
+  )
+  (wire (pts (xy 231.14 48.26) (xy 234.95 48.26))
     (stroke (width 0) (type default) (color 0 0 0 0))
   )
@@
     (stroke (width 0) (type default) (color 0 0 0 0))
   )
+  (wire (pts (xy 231.14 52.07) (xy 234.95 52.07))
+    (stroke (width 0) (type default) (color 0 0 0 0))
+  )
   (wire (pts (xy 203.2 96.52) (xy 212.09 96.52))
     (stroke (width 0) (type default) (color 0 0 0 0))
@@
   )
   (wire (pts (xy 55.88 57.15) (xy 67.31 57.15))
+    (stroke (width 0) (type default) (color 0 0 0 0))
+  )
+  (wire (pts (xy 231.14 55.88) (xy 234.95 55.88))
     (stroke (width 0) (type default) (color 0 0 0 0))
   )
@@
     (effects (font (size 1.27 1.27)) (justify left bottom))
   )
+  (global_label "MOSI" (shape input) (at 231.14 48.26 180) (fields_autoplaced)
+    (effects (font (size 1.27 1.27)) (justify right))
+    (property "Intersheet References" "${INTERSHEET_REFS}" (id 0) (at 224.1307 48.1806 0)
+      (effects (font (size 1.27 1.27)) (justify right) hide)
+    )
+  )
+  (global_label "SCK" (shape input) (at 231.14 52.07 180) (fields_autoplaced)
+    (effects (font (size 1.27 1.27)) (justify right))
+    (property "Intersheet References" "${INTERSHEET_REFS}" (id 0) (at 224.9774 51.9906 0)
+      (effects (font (size 1.27 1.27)) (justify right) hide)
+    )
+  )
+  (global_label "LATCH" (shape input) (at 231.14 55.88 180) (fields_autoplaced)
+    (effects (font (size 1.27 1.27)) (justify right))
+    (property "Intersheet References" "${INTERSHEET_REFS}" (id 0) (at 223.0421 55.8006 0)
+      (effects (font (size 1.27 1.27)) (justify right) hide)
+    )
+  )
   (hierarchical_label "ENCODER_INDEX" (shape input) (at 246.38 119.38 0)
     (effects (font (size 1.27 1.27)) (justify left))
   )
+  (hierarchical_label "MOSI" (shape input) (at 219.71 50.8 180)
+    (effects (font (size 1.27 1.27)) (justify right))
+  )
   (hierarchical_label "STDNT_SRVO_RX_1" (shape input) (at 203.2 111.76 180)
     (effects (font (size 1.27 1.27)) (justify right))
@@
     (effects (font (size 1.27 1.27)) (justify right))
   )
-  (hierarchical_label "STUDENT_SERV_EN" (shape output) (at 198.12 60.96 0)
-    (effects (font (size 1.27 1.27)) (justify left))
-  )
-  (hierarchical_label "STEPP_DIR" (shape output) (at 198.12 52.07 0)
+  (hierarchical_label "STUDENT_SERV_EN" (shape output) (at 260.35 60.96 0)
+    (effects (font (size 1.27 1.27)) (justify left))
+  )
+  (hierarchical_label "STEPP_DIR" (shape output) (at 260.35 52.07 0)
     (effects (font (size 1.27 1.27)) (justify left))
   )
@@
     (effects (font (size 1.27 1.27)) (justify left))
   )
-  (hierarchical_label "STUDENT_STEP_EN" (shape output) (at 198.12 58.42 0)
+  (hierarchical_label "STUDENT_STEP_EN" (shape output) (at 260.35 58.42 0)
     (effects (font (size 1.27 1.27)) (justify left))
   )
@@
     (effects (font (size 1.27 1.27)) (justify left))
   )
-  (hierarchical_label "STEPP_RST" (shape output) (at 198.12 49.53 0)
+  (hierarchical_label "STEPP_RST" (shape output) (at 260.35 49.53 0)
     (effects (font (size 1.27 1.27)) (justify left))
   )
@@
     (effects (font (size 1.27 1.27)) (justify left))
   )
-  (hierarchical_label "STUDENT_M_EN" (shape output) (at 198.12 55.88 0)
+  (hierarchical_label "STUDENT_M_EN" (shape output) (at 260.35 55.88 0)
     (effects (font (size 1.27 1.27)) (justify left))
   )
@@
     (effects (font (size 1.27 1.27)) (justify right))
   )
-  (hierarchical_label "STEPP_EN" (shape output) (at 198.12 46.99 0)
-    (effects (font (size 1.27 1.27)) (justify left))
-  )
+  (hierarchical_label "STEPP_EN" (shape output) (at 260.35 46.99 0)
+    (effects (font (size 1.27 1.27)) (justify left))
+  )
