File: RemoteLabs_supervisor_PCB/RemoteLabs_supervisor_PCB.kicad_sch (KiCad schematic)
At the start: 1 part

Commit message: adding test sketch
Parts:
- added J?: Super_Prog_Header, Connector_PinHeader_1.27mm:PinHeader_1x05_P1.27mm_Vertical, symbol 000_Pin_Headers_Immo:Conn_01x05_Male
- added J?: LightingStrip Header, symbol Connector:Conn_01x03_Male
- added R?: 300r, Resistor_SMD:R_0805_2012Metric_Pad1.20x1.40mm_HandSolder, symbol 000_Resistors_Immo:Resistor_0805
Connections:
- net Supervisor MCU/MCU_RESET: now also J?.5 (Pin_5)
- net Supervisor MCU/PROG_RX: now also J?.4 (Pin_4)
- net Supervisor MCU/PROG_TX: now also J?.3 (Pin_3)
- net GNDA renamed GND
- net GND: now also J?.1 (Pin_1)
- new net: J?.2 (Pin_2), R?.2
- new net 3V3_DC_MCU: J?.2 (Pin_2)
- new net 5V_DC_IN: J?.1 (Pin_1)
- new net GND_D: J?.3 (Pin_3)
- new net ~{LIGHT_STRIP}: R?.1
Other:
- sheet Analog Sensor Buffers ports: added VCC; removed 5V_VCC, GND_A
- sheet Digital Sensor Buffers ports: added VCC; removed 5V_VCC
- sheet Output Logic ports: added VCC; removed 5V_VCC
- sheet Power Input & Distribution ports: added 3V3_DC_MCU; removed none
- sheet Servo Control ports: added GND_P; removed GND_p

Commit message: sdf
Parts:
- J?: value LightingStrip Header -> WS2821B Header
Connections:
- net ~{LIGHT_STRIP} renamed DIGI_LIGHTS
Other:
- sheet Analog Sensor Buffers ports: added GND_A; removed none
- note added: "Does Student Need Mode Controls?"
- note added: "INH Pins just need to be tied HIGH to enable DC Motor Driver - Might not need student control at all?"
- note added: "IS: limit being spoofed to student or raw (buffered) input?"
- note added: "Is Fault Digi or Analog O/P"
- note added: "What is needed for OE Index?"
- note removed: "?"
- moved on the sheet: J?, R?, TP?

Commit message: Schematic Work
Other:
- sheet DC Motor Controller ports: added INHIBIT; removed INH_1, INH_2
- sheet Stepper Motor Controller ports: added RESET, SLEEP; removed DISABLE
- sheet Supervisor MCU ports: added none; removed !!~{FLT}!!
- note added: "Fault is Digital Low when fault detected"
- note removed: "Is Fault Digi or Analog O/P"
Changed lines of the file:
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@@
+    (stroke (width 0) (type default) (color 0 0 0 0))
+  )
+  (wire (pts (xy 227.33 77.47) (xy 229.87 77.47))
     (stroke (width 0) (type default) (color 0 0 0 0))
   )
@@
   )
   (wire (pts (xy 111.76 31.75) (xy 114.3 31.75))
-    (stroke (width 0) (type default) (color 0 0 0 0))
-  )
-  (wire (pts (xy 208.28 38.1) (xy 229.87 38.1))
     (stroke (width 0) (type default) (color 0 0 0 0))
   )
@@
     (effects (font (size 1.27 1.27)) (justify left bottom))
   )
-  (text "Is Fault Digi or \nAnalog\nO/P" (at 213.36 96.52 0)
+  (text "Fault is Digital\nLow when fault \ndetected" (at 220.98 106.68 0)
     (effects (font (size 1.27 1.27)) (justify left bottom))
   )
@@
     (property "Intersheet References" "${INTERSHEET_REFS}" (id 0) (at 67.3041 25.3206 0)
       (effects (font (size 1.27 1.27)) (justify left) hide)
+    )
+  )
+  (global_label "3V3_DC_MCU" (shape input) (at 227.33 77.47 180) (fields_autoplaced)
+    (effects (font (size 1.27 1.27)) (justify right))
+    (property "Intersheet References" "${INTERSHEET_REFS}" (id 0) (at 212.8821 77.3906 0)
+      (effects (font (size 1.27 1.27)) (justify right) hide)
     )
   )
@@
       (effects (font (size 1.27 1.27)) (justify right))
     )
-    (pin "!!~{FLT}!!" input (at 149.86 78.74 0)
-      (effects (font (size 1.27 1.27)) (justify right))
-    )
     (pin "MODE_1" output (at 149.86 50.8 0)
       (effects (font (size 1.27 1.27)) (justify right))
@@
       (effects (font (size 1.27 1.27)) (justify left))
     )
-    (pin "ENABLE" input (at 229.87 81.28 180)
-      (effects (font (size 1.27 1.27)) (justify left))
-    )
-    (pin "MODE_0" input (at 229.87 69.85 180)
-      (effects (font (size 1.27 1.27)) (justify left))
-    )
-    (pin "MODE_1" input (at 229.87 72.39 180)
-      (effects (font (size 1.27 1.27)) (justify left))
-    )
-    (pin "MODE_2" input (at 229.87 74.93 180)
-      (effects (font (size 1.27 1.27)) (justify left))
-    )
-    (pin "DISABLE" input (at 229.87 78.74 180)
+    (pin "ENABLE" input (at 229.87 80.01 180)
+      (effects (font (size 1.27 1.27)) (justify left))
+    )
+    (pin "MODE_0" input (at 229.87 68.58 180)
+      (effects (font (size 1.27 1.27)) (justify left))
+    )
+    (pin "MODE_1" input (at 229.87 71.12 180)
+      (effects (font (size 1.27 1.27)) (justify left))
+    )
+    (pin "MODE_2" input (at 229.87 73.66 180)
       (effects (font (size 1.27 1.27)) (justify left))
     )
@@
     )
     (pin "FAULT_OUT" output (at 229.87 92.71 180)
+      (effects (font (size 1.27 1.27)) (justify left))
+    )
+    (pin "SLEEP" input (at 229.87 77.47 180)
+      (effects (font (size 1.27 1.27)) (justify left))
+    )
+    (pin "RESET" input (at 229.87 82.55 180)
       (effects (font (size 1.27 1.27)) (justify left))
     )
@@
       (effects (font (size 1.27 1.27)) (justify left))
     )
-    (pin "INH_2" input (at 229.87 38.1 180)
-      (effects (font (size 1.27 1.27)) (justify left))
-    )
     (pin "IN_2" input (at 229.87 31.75 180)
       (effects (font (size 1.27 1.27)) (justify left))
@@
       (effects (font (size 1.27 1.27)) (justify left))
     )
-    (pin "INH_1" input (at 229.87 35.56 180)
+    (pin "INHIBIT" input (at 229.87 35.56 180)
       (effects (font (size 1.27 1.27)) (justify left))
     )
@@
       (effects (font (size 1.27 1.27)) (justify right))
     )
-    (pin "OUT_M_INH_2" output (at 208.28 38.1 0)
+    (pin "OUT_M_INH_2" output (at 208.28 39.37 0)
       (effects (font (size 1.27 1.27)) (justify right))
     )
@@
       (reference "C?") (unit 1) (value "100n") (footprint "Capacitor_SMD:C_0805_2012Metric_Pad1.18x1.45mm_HandSolder")
     )
+    (path "/58677001-4fa9-4c82-8bf8-e3f98fe8c902/1b274f9f-14ca-4bae-b091-e56120d79f86"
+      (reference "C?") (unit 1) (value "100n") (footprint "Capacitor_SMD:C_0805_2012Metric_Pad1.18x1.45mm_HandSolder")
+    )
     (path "/8cce862e-92d4-4b11-b295-b482621a1385/1b274f9f-14ca-4bae-b091-e56120d79f86"
-      (reference "C?") (unit 1) (value "100n") (footprint "Capacitor_SMD:C_0805_2012Metric_Pad1.18x1.45mm_HandSolder")
-    )
-    (path "/58677001-4fa9-4c82-8bf8-e3f98fe8c902/1b274f9f-14ca-4bae-b091-e56120d79f86"
       (reference "C?") (unit 1) (value "100n") (footprint "Capacitor_SMD:C_0805_2012Metric_Pad1.18x1.45mm_HandSolder")
     )
@@
       (reference "C?") (unit 1) (value "10u") (footprint "Capacitor_SMD:CP_Elec_6.3x5.9")
     )
+    (path "/58677001-4fa9-4c82-8bf8-e3f98fe8c902/a23093a8-ca6b-41b9-8efa-cf6603cc916b"
+      (reference "C?") (unit 1) (value "100n") (footprint "Capacitor_SMD:C_0805_2012Metric_Pad1.18x1.45mm_HandSolder")
+    )
     (path "/8cce862e-92d4-4b11-b295-b482621a1385/a23093a8-ca6b-41b9-8efa-cf6603cc916b"
-      (reference "C?") (unit 1) (value "100n") (footprint "Capacitor_SMD:C_0805_2012Metric_Pad1.18x1.45mm_HandSolder")
-    )
-    (path "/58677001-4fa9-4c82-8bf8-e3f98fe8c902/a23093a8-ca6b-41b9-8efa-cf6603cc916b"
       (reference "C?") (unit 1) (value "100n") (footprint "Capacitor_SMD:C_0805_2012Metric_Pad1.18x1.45mm_HandSolder")
     )
@@
       (reference "R1") (unit 1) (value "2k2") (footprint "Resistor_SMD:R_0805_2012Metric_Pad1.20x1.40mm_HandSolder")
     )
+    (path "/0d587a0a-c67c-4fed-9eec-791a57f2bb2e/12711d54-27d6-4e42-8088-f7a42f7c1094"
+      (reference "R?") (unit 1) (value "1k") (footprint "Resistor_SMD:R_0805_2012Metric_Pad1.20x1.40mm_HandSolder")
+    )
     (path "/3053d1d3-1dd5-4dac-b6cb-5e7828c7a42e/1646c3f2-8b13-40e6-bd0a-8755e7c99a1c"
       (reference "R?") (unit 1) (value "2k7") (footprint "Resistor_SMD:R_0805_2012Metric_Pad1.20x1.40mm_HandSolder")
@@
       (reference "R?") (unit 1) (value "1M") (footprint "Resistor_SMD:R_0805_2012Metric_Pad1.20x1.40mm_HandSolder")
     )
+    (path "/0d587a0a-c67c-4fed-9eec-791a57f2bb2e/5646c51c-d3f4-4339-9f33-10fadba61865"
+      (reference "R?") (unit 1) (value "1k") (footprint "Resistor_SMD:R_0805_2012Metric_Pad1.20x1.40mm_HandSolder")
+    )
+    (path "/9266ad98-56ad-4979-a534-eef1d9b8c163/5a9a5221-ae94-4768-b191-97e75e809df1"
+      (reference "R?") (unit 1) (value "470r") (footprint "Resistor_SMD:R_0805_2012Metric_Pad1.20x1.40mm_HandSolder")
+    )
+    (path "/0d587a0a-c67c-4fed-9eec-791a57f2bb2e/740bcc10-8b55-4692-b5eb-b30fe6818d55"
+      (reference "R?") (unit 1) (value "1k") (footprint "Resistor_SMD:R_0805_2012Metric_Pad1.20x1.40mm_HandSolder")
+    )
     (path "/0d587a0a-c67c-4fed-9eec-791a57f2bb2e/7bc06db4-6fdc-4aae-b383-86fcd3395d18"
       (reference "R?") (unit 1) (value "330r") (footprint "Resistor_SMD:R_0805_2012Metric_Pad1.20x1.40mm_HandSolder")
     )
+    (path "/9266ad98-56ad-4979-a534-eef1d9b8c163/83a0c178-0561-47c1-afa2-6579c8ee9f74"
+      (reference "R?") (unit 1) (value "470r") (footprint "Resistor_SMD:R_0805_2012Metric_Pad1.20x1.40mm_HandSolder")
+    )
     (path "/283d3eb1-906d-460d-a87d-d328f41afedd/8d64857c-8c3e-4a46-b93d-6ae8d03fb4ca"
       (reference "R?") (unit 1) (value "Resistor_0805") (footprint "Resistor_SMD:R_0805_2012Metric_Pad1.20x1.40mm_HandSolder")
@@
       (reference "R?") (unit 1) (value "10k") (footprint "Resistor_SMD:R_0805_2012Metric_Pad1.20x1.40mm_HandSolder")
     )
+    (path "/0d587a0a-c67c-4fed-9eec-791a57f2bb2e/758cc32e-478c-4f82-bbbf-2e2e44bc0576"
+      (reference "SW?") (unit 1) (value "Stepper_Mode") (footprint "")
+    )
     (path "/1fcb30e3-51c0-4114-9903-50e7d65dc82a"

Commit message: lunchtime backup
Other:
- sheet DC Motor Controller ports: added ENABLE; removed INHIBIT
- sheet Output Logic ports: added none; removed OUT_M_INH_1, OUT_M_INH_2, STUDENT_M_INH_1, STUDENT_M_INH_2, STUDENT_M_IN_1, STUDENT_M_IN_2, SUPERVISOR_M_INH_1, SUPERVISOR_M_INH_2, SUPERVISOR_M_IN_1, SUPERVISOR_M_IN_2
- sheet Supervisor MCU ports: added DC_MOTOR_DIR1, DC_MOTOR_DIR2, DC_MOTOR_IS1, DC_MOTOR_IS2, DC_MOTOR_PWM, ENCODER_INDEX, NEOPIXELS, PIXEL_DATA, STDNT_DC_M_DIR_1, STDNT_SRVO_RX_1, STDNT_SRVO_RX_2, STEPP_DIR, STEPP_EN, STEPP_FLT, STEPP_RST, STEPP_STEP; removed !!~{EN}!!, DC_MOTOR_DRIVE_A, DC_MOTOR_DRIVE_B, INDEX, STEP, ~{LIGHT_STRIP}, ~{RST}??, ~{SLP}??
- note removed: "Does Student Need Mode Controls?"

Commit message: Circuit Design 85-90% complete
Connections:
- net DIGI_LIGHTS renamed Output Logic/PIXEL_DATA_OUT
Other:
- sheet Output Logic ports: added MOTOR_DIR_A, MOTOR_DIR_B, MOTOR_OUT_1, MOTOR_OUT_2, OUT_M_ENABLE, PIXEL_DATA_OUT, STEPP_STEP_OUT, STEP_EN_OUT, STUDENT_MOTOR_EN, STUDENT_MOTOR_ENABLE, STUDENT_MOTOR_PWM, STUDENT_PIXEL_DATA, STUDENT_PIXEL_ENABLE, STUDENT_STEP_EN, SUPERVISOR_MOTOR_EN, SUPERVISOR_MOTOR_PWM, SUPERVISOR_PIXEL_DATA, SUPERVISOR_STEP_EN; removed OUT_M_IN_1, OUT_M_IN_2, STEP_OUT, STUDENT_M_ENABLE
- sheet Supervisor MCU ports: added DC_MOTOR_EN, STDNT_DC_M_DIR_2, STUDENT_M_EN, STUDENT_PIXEL_EN, STUDENT_SERV_EN, STUDENT_STEP_EN, THERMO; removed DIRECTION, NEOPIXELS
- note added: "Answer: Have some digital pins left to do it, but rather save them for something else, maybe provide header pins to enable this later"
- moved on the sheet: J?, R?

Commit message: nearing circut deisng complete
Other:
- sheet Student MCU ports: added 3V3_DC_IN, 5V_DC_IN, DC_MOTOR_DIR1, DC_MOTOR_DIR2, DC_MOTOR_EN, DC_MOTOR_IS1, DC_MOTOR_IS2, DC_MOTOR_PWM, ENCODER_A, ENCODER_B, ENCODER_INDEX, GND_D, LIMIT_1, LIMIT_2, MCU_RESET, PIXEL_DATA, PROG_RX, PROG_TX, SERVO_1, SERVO_2, STEPP_DIR, STEPP_EN, STEPP_FLT, STEPP_RST, STEPP_STEP, THERMO; removed none
- sheet analogSensors ports: added VCC; removed 5V_IN

Commit message: V1.0 Circuit Design Complete
Parts:
- added J?: Student_Prog_Header, Connector_PinHeader_1.27mm:PinHeader_1x05_P1.27mm_Vertical, symbol 000_Pin_Headers_Immo:Conn_01x05_Male
- gave numbers to parts that had none: 4
Connections:
- net 3V3_DC_MCU: now also J?.2 (Pin_2)
- net GND: now also J?.1 (Pin_1)
- net Student MCU/MCU_RESET: now also J?.5 (Pin_5)
- net Student MCU/PROG_RX: now also J?.4 (Pin_4)
- net Student MCU/PROG_TX: now also J?.3 (Pin_3)
Other:
- sheet Output Logic ports: added STEP_RST_OUT, STUDENT_STEP_RST, SUPERVISOR_STEP_RST; removed SERVO_PWM_OUT, STUDENT_SERVO_ENABLE, STUDENT_SERVO_PWM, SUPERVISOR_SERVO_PWM
- sheet Power Input & Distribution ports: added USP_PWR_IN; removed 5V_DC_MCU
- sheet Student MCU ports: added V_USB; removed 5V_DC_IN
- sheet Supervisor MCU ports: added V_USB; removed 5V_DC_IN, LIMIT_3, STUDENT_SERV_EN
- note removed: "Answer: Have some digital pins left to do it, but rather save them for something else, maybe provide header pins to enable this later"
- note removed: "IS: limit being spoofed to student or raw (buffered) input?"
- note removed: "What is needed for OE Index?"
- moved on the sheet: TP1

Commit message: ERC checks run
Parts:
- added J27: Analog Buffer, symbol Connector:Conn_01x03_Male
- gave numbers to parts that had none: 1
Connections:
- new net A_BUFFER_IN: J27.1 (Pin_1)
- new net A_BUFFER_OUT_A: J27.2 (Pin_2)
- new net A_BUFFER_OUT_B: J27.3 (Pin_3)
Other:
- note removed: "INH Pins just need to be tied HIGH to enable DC Motor Driver - Might not need student control at all?"
- moved on the sheet: J1, J2, R5
