File: RemoteLabs_supervisor_PCB/RemoteLabs_supervisor_PCB.kicad_sch (KiCad schematic)
At the start: 14 parts, among them J1 Super_Prog_Header, J2 WS2821B Header, J26 Student_Prog_Header, J27 Analog Buffer

Commit message: PCB layout
Parts:
- J1, J26: footprint Connector_PinHeader_2.54mm:PinHeader_1x05_P2.54mm_Vertical -> Connector_Molex:Molex_KK-254_AE-6410-05A_1x05_P2.54mm_Vertical; symbol 000_Pin_Headers_Immo:Conn_01x05_Male -> 000_Pin_Headers_Immo:Molex_5pin_2.54mm_M
Changed lines of the file:
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@@
     (pin "1")
   )
-  (symbol (lib_id "000_Pin_Headers_Immo:Conn_01x05_Male") (at 76.835 41.91 0) (unit 1)
+  (symbol (lib_id "000_Pin_Headers_Immo:Molex_5pin_2.54mm_M") (at 76.835 41.91 0) (unit 1)
     (in_bom yes) (on_board yes)
     (property "Reference" "J1" (id 0) (at 76.835 33.02 0))
     (property "Value" "Super_Prog_Header" (id 1) (at 74.295 39.37 90))
-    (property "Footprint" "Connector_PinHeader_2.54mm:PinHeader_1x05_P2.54mm_Vertical" (id 2) (at 76.835 41.91 0)
+    (property "Footprint" "Connector_Molex:Molex_KK-254_AE-6410-05A_1x05_P2.54mm_Vertical" (id 2) (at 78.74 52.07 0)
       (effects (font (size 1.27 1.27)) hide)
     )
@@
     (pin "2")
   )
-  (symbol (lib_id "000_Pin_Headers_Immo:Conn_01x05_Male") (at 73.025 182.245 0) (unit 1)
+  (symbol (lib_id "000_Pin_Headers_Immo:Molex_5pin_2.54mm_M") (at 73.025 182.245 0) (unit 1)
     (in_bom yes) (on_board yes)
     (property "Reference" "J26" (id 0) (at 73.025 173.355 0))
     (property "Value" "Student_Prog_Header" (id 1) (at 70.485 179.705 90))
-    (property "Footprint" "Connector_PinHeader_2.54mm:PinHeader_1x05_P2.54mm_Vertical" (id 2) (at 73.025 182.245 0)
+    (property "Footprint" "Connector_Molex:Molex_KK-254_AE-6410-05A_1x05_P2.54mm_Vertical" (id 2) (at 74.93 192.405 0)
       (effects (font (size 1.27 1.27)) hide)
     )
@@
     )
     (path "/ef79b516-f387-4bff-98aa-61eff96e72d2/f51bc9d0-b778-4a7d-ab8d-5001d2ab64e6"
-      (reference "C7") (unit 1) (value "1u") (footprint "Capacitor_SMD:C_0805_2012Metric_Pad1.18x1.45mm_HandSolder")
+      (reference "C7") (unit 1) (value "1u") (footprint "Capacitor_Tantalum_SMD:CP_EIA-2012-12_Kemet-R_Pad1.30x1.05mm_HandSolder")
     )
     (path "/ef79b516-f387-4bff-98aa-61eff96e72d2/0204e619-04da-4e69-aaad-63ec75faaa3d"
@@
     )
     (path "/0d587a0a-c67c-4fed-9eec-791a57f2bb2e/6870b48b-975a-4d6e-abfa-505a0108f8d3"
-      (reference "C17") (unit 1) (value "1u") (footprint "Capacitor_SMD:C_0805_2012Metric_Pad1.18x1.45mm_HandSolder")
+      (reference "C17") (unit 1) (value "1u") (footprint "Capacitor_Tantalum_SMD:CP_EIA-2012-12_Kemet-R_Pad1.30x1.05mm_HandSolder")
     )
     (path "/0d587a0a-c67c-4fed-9eec-791a57f2bb2e/5aa831b5-f34c-4177-b0fc-50fc07865184"
@@
     )
     (path "/20bc3c73-e2bf-488f-a0c1-38700b58a060"
-      (reference "J1") (unit 1) (value "Super_Prog_Header") (footprint "Connector_PinHeader_2.54mm:PinHeader_1x05_P2.54mm_Vertical")
+      (reference "J1") (unit 1) (value "Super_Prog_Header") (footprint "Connector_Molex:Molex_KK-254_AE-6410-05A_1x05_P2.54mm_Vertical")
     )
     (path "/9f02ea00-3ee8-4183-95b6-7d59f1944b3b"
@@
     )
     (path "/586ec748-563a-478a-82db-706fb951336a/3d412b69-c529-4e16-8a2a-e7a8b0ecba07"
-      (reference "J3") (unit 1) (value "XT60_connector_DC_45A_male") (footprint "Connector_AMASS:AMASS_XT60PW-M")
+      (reference "J3") (unit 1) (value "XT60_60A_male") (footprint "Connector_AMASS:AMASS_XT60PW-M")
     )
     (path "/586ec748-563a-478a-82db-706fb951336a/7e87b1c4-c7af-4837-a2de-ad1fe5674fd5"
@@
     )
     (path "/e3a5c764-2bf9-4c0b-b94d-393b25109771"
-      (reference "J26") (unit 1) (value "Student_Prog_Header") (footprint "Connector_PinHeader_2.54mm:PinHeader_1x05_P2.54mm_Vertical")
+      (reference "J26") (unit 1) (value "Student_Prog_Header") (footprint "Connector_Molex:Molex_KK-254_AE-6410-05A_1x05_P2.54mm_Vertical")
     )
     (path "/14c3136c-ef8c-4e68-91a4-4c8b13db2bc5"
@@
       (reference "JP4") (unit 1) (value "Xtal/IC") (footprint "000_Connectors_Immo:SolderJumper-3_P1.3mm_Bridged12_RoundedPad1.0x1.5mm_NumberLabels")
     )
-    (path "/ef79b516-f387-4bff-98aa-61eff96e72d2/d492626d-bd18-4011-91d9-0b9d2c4eb55f"
-      (reference "JP5") (unit 1) (value "Xtal/IC") (footprint "000_Connectors_Immo:SolderJumper-3_P1.3mm_Bridged12_RoundedPad1.0x1.5mm_NumberLabels")
-    )
     (path "/0d587a0a-c67c-4fed-9eec-791a57f2bb2e/d9ede1d9-98fb-4bf6-9188-b8434de8eed0"
       (reference "JP6") (unit 1) (value "Xtal/IC") (footprint "000_Connectors_Immo:SolderJumper-3_P1.3mm_Bridged12_RoundedPad1.0x1.5mm_NumberLabels")
@@
       (reference "JP7") (unit 1) (value "Xtal/IC") (footprint "000_Connectors_Immo:SolderJumper-3_P1.3mm_Bridged12_RoundedPad1.0x1.5mm_NumberLabels")
     )
-    (path "/0d587a0a-c67c-4fed-9eec-791a57f2bb2e/1afbb630-15d4-42df-9faa-8ce8c1fd627a"
-      (reference "JP8") (unit 1) (value "Xtal/IC") (footprint "000_Connectors_Immo:SolderJumper-3_P1.3mm_Bridged12_RoundedPad1.0x1.5mm_NumberLabels")
-    )
     (path "/0d587a0a-c67c-4fed-9eec-791a57f2bb2e/26e9e77b-c4f0-439a-94a1-c5ad551b03df"
       (reference "JP9") (unit 1) (value "Reset Jumper") (footprint "000_Connectors_Immo:SolderJumper-2_P1.3mm_Open_Pad1.0x1.5mm")
     )
+    (path "/ef79b516-f387-4bff-98aa-61eff96e72d2/27c64e6c-34e2-4309-a9fd-258ec95a64a3"
+      (reference "JP10") (unit 1) (value "Reset Jumper") (footprint "000_Connectors_Immo:SolderJumper-2_P1.3mm_Open_Pad1.0x1.5mm")
+    )
     (path "/5e0c70ac-7a7e-4605-86e1-28eee540aa4a"
       (reference "NT1") (unit 1) (value "NetTie") (footprint "NetTie:NetTie-2_SMD_Pad0.5mm")
@@
       (reference "TP1") (unit 1) (value "GND") (footprint "TestPoint:TestPoint_Pad_D1.5mm")
     )
-    (path "/586ec748-563a-478a-82db-706fb951336a/95346655-713c-47f9-86ef-c2883667dda4"
-      (reference "TP4") (unit 1) (value "5V_SERVO") (footprint "TestPoint:TestPoint_Pad_D1.5mm")
-    )
     (path "/586ec748-563a-478a-82db-706fb951336a/c60d923a-3025-4983-8cf5-e15e10785356"

Commit message: PCB layout
Parts:
- added H1, H2, H3, H4, H5, H6: MountingHole, MountingHole:MountingHole_3.2mm_M3_Pad_Via, symbol Mechanical:MountingHole_M3
- J2: footprint Connector_PinHeader_2.54mm:PinHeader_1x03_P2.54mm_Vertical -> Connector_Molex:Molex_KK-254_AE-6410-03A_1x03_P2.54mm_Vertical; symbol Connector:Conn_01x03_Male -> 000_Connectors_Immo:3pin_molex_2.54mm_male
Changed lines of the file:
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@@
     (pin "1")
+  )
+  (symbol (lib_id "Mechanical:MountingHole_M3") (at 122.555 192.405 0) (unit 1)
+    (in_bom yes) (on_board yes) (fields_autoplaced)
+    (property "Reference" "H2" (id 0) (at 125.73 191.1349 0)
+      (effects (font (size 1.27 1.27)) (justify left))
+    )
+    (property "Value" "MountingHole" (id 1) (at 125.73 193.6749 0)
+      (effects (font (size 1.27 1.27)) (justify left))
+    )
+    (property "Footprint" "MountingHole:MountingHole_3.2mm_M3_Pad_Via" (id 2) (at 122.555 192.405 0)
+      (effects (font (size 1.27 1.27)) hide)
+    )
+    (property "Datasheet" "~" (id 3) (at 122.555 192.405 0)
+      (effects (font (size 1.27 1.27)) hide)
+    )
   )
   (symbol (lib_id "Device:NetTie_2") (at 31.75 59.69 0) (unit 1)
@@
     (pin "1")
   )
+  (symbol (lib_id "Mechanical:MountingHole_M3") (at 122.555 187.325 0) (unit 1)
+    (in_bom yes) (on_board yes) (fields_autoplaced)
+    (property "Reference" "H1" (id 0) (at 125.73 186.0549 0)
+      (effects (font (size 1.27 1.27)) (justify left))
+    )
+    (property "Value" "MountingHole" (id 1) (at 125.73 188.5949 0)
+      (effects (font (size 1.27 1.27)) (justify left))
+    )
+    (property "Footprint" "MountingHole:MountingHole_3.2mm_M3_Pad_Via" (id 2) (at 122.555 187.325 0)
+      (effects (font (size 1.27 1.27)) hide)
+    )
+    (property "Datasheet" "~" (id 3) (at 122.555 187.325 0)
+      (effects (font (size 1.27 1.27)) hide)
+    )
+  )
   (symbol (lib_id "000_Resistors_Immo:Resistor_0805") (at 108.585 116.205 90) (unit 1)
     (in_bom yes) (on_board yes) (fields_autoplaced)
@@
     (pin "1")
   )
+  (symbol (lib_id "Mechanical:MountingHole_M3") (at 140.335 192.405 0) (unit 1)
+    (in_bom yes) (on_board yes) (fields_autoplaced)
+    (property "Reference" "H4" (id 0) (at 143.51 191.1349 0)
+      (effects (font (size 1.27 1.27)) (justify left))
+    )
+    (property "Value" "MountingHole" (id 1) (at 143.51 193.6749 0)
+      (effects (font (size 1.27 1.27)) (justify left))
+    )
+    (property "Footprint" "MountingHole:MountingHole_3.2mm_M3_Pad_Via" (id 2) (at 140.335 192.405 0)
+      (effects (font (size 1.27 1.27)) hide)
+    )
+    (property "Datasheet" "~" (id 3) (at 140.335 192.405 0)
+      (effects (font (size 1.27 1.27)) hide)
+    )
+  )
+  (symbol (lib_id "Mechanical:MountingHole_M3") (at 158.75 192.405 0) (unit 1)
+    (in_bom yes) (on_board yes) (fields_autoplaced)
+    (property "Reference" "H6" (id 0) (at 161.925 191.1349 0)
+      (effects (font (size 1.27 1.27)) (justify left))
+    )
+    (property "Value" "MountingHole" (id 1) (at 161.925 193.6749 0)
+      (effects (font (size 1.27 1.27)) (justify left))
+    )
+    (property "Footprint" "MountingHole:MountingHole_3.2mm_M3_Pad_Via" (id 2) (at 158.75 192.405 0)
+      (effects (font (size 1.27 1.27)) hide)
+    )
+    (property "Datasheet" "~" (id 3) (at 158.75 192.405 0)
+      (effects (font (size 1.27 1.27)) hide)
+    )
+  )
   (symbol (lib_id "power:GNDD") (at 80.645 177.165 90) (unit 1)
     (in_bom yes) (on_board yes) (fields_autoplaced)
@@
     )
     (pin "1")
+  )
+  (symbol (lib_id "Mechanical:MountingHole_M3") (at 140.335 187.325 0) (unit 1)
+    (in_bom yes) (on_board yes) (fields_autoplaced)
+    (property "Reference" "H3" (id 0) (at 143.51 186.0549 0)
+      (effects (font (size 1.27 1.27)) (justify left))
+    )
+    (property "Value" "MountingHole" (id 1) (at 143.51 188.5949 0)
+      (effects (font (size 1.27 1.27)) (justify left))
+    )
+    (property "Footprint" "MountingHole:MountingHole_3.2mm_M3_Pad_Via" (id 2) (at 140.335 187.325 0)
+      (effects (font (size 1.27 1.27)) hide)
+    )
+    (property "Datasheet" "~" (id 3) (at 140.335 187.325 0)
+      (effects (font (size 1.27 1.27)) hide)
+    )
   )
   (symbol (lib_id "power:GNDD") (at 65.405 107.95 0) (unit 1)
@@
     (pin "1")
   )
-  (symbol (lib_id "Connector:Conn_01x03_Male") (at 262.89 156.845 0) (mirror y) (unit 1)
+  (symbol (lib_id "000_Connectors_Immo:3pin_molex_2.54mm_male") (at 262.89 156.845 0) (mirror y) (unit 1)
     (in_bom yes) (on_board yes)
     (property "Reference" "J2" (id 0) (at 261.62 149.225 0))
     (property "Value" "WS2821B Header" (id 1) (at 262.255 151.765 0))
-    (property "Footprint" "Connector_PinHeader_2.54mm:PinHeader_1x03_P2.54mm_Vertical" (id 2) (at 262.89 156.845 0)
+    (property "Footprint" "Connector_Molex:Molex_KK-254_AE-6410-03A_1x03_P2.54mm_Vertical" (id 2) (at 259.461 163.83 0)
       (effects (font (size 1.27 1.27)) hide)
     )
@@
     )
     (pin "1")
+  )
+  (symbol (lib_id "Mechanical:MountingHole_M3") (at 158.75 187.325 0) (unit 1)
+    (in_bom yes) (on_board yes) (fields_autoplaced)
+    (property "Reference" "H5" (id 0) (at 161.925 186.0549 0)
+      (effects (font (size 1.27 1.27)) (justify left))
+    )
+    (property "Value" "MountingHole" (id 1) (at 161.925 188.5949 0)
+      (effects (font (size 1.27 1.27)) (justify left))
+    )
+    (property "Footprint" "MountingHole:MountingHole_3.2mm_M3_Pad_Via" (id 2) (at 158.75 187.325 0)
+      (effects (font (size 1.27 1.27)) hide)
+    )
+    (property "Datasheet" "~" (id 3) (at 158.75 187.325 0)
+      (effects (font (size 1.27 1.27)) hide)
+    )
   )
   (symbol (lib_id "000_Resistors_Immo:Resistor_0805") (at 104.14 111.125 90) (unit 1)
@@
       (reference "FB2") (unit 1) (value "BLM18PG471") (footprint "Inductor_SMD:L_0805_2012Metric_Pad1.05x1.20mm_HandSolder")
     )
+    (path "/2d1d28f4-c238-451f-be2e-9e08e8cd4ee7"
+      (reference "H1") (unit 1) (value "MountingHole") (footprint "MountingHole:MountingHole_3.2mm_M3_Pad_Via")
+    )
+    (path "/1c741d7c-0741-43b4-824a-7f67568e467d"
+      (reference "H2") (unit 1) (value "MountingHole") (footprint "MountingHole:MountingHole_3.2mm_M3_Pad_Via")
+    )
+    (path "/861afc69-35ac-425d-ad57-ba17f5b41b6c"
+      (reference "H3") (unit 1) (value "MountingHole") (footprint "MountingHole:MountingHole_3.2mm_M3_Pad_Via")
+    )
+    (path "/70478d78-e383-4d8a-b275-d772b62cb463"
+      (reference "H4") (unit 1) (value "MountingHole") (footprint "MountingHole:MountingHole_3.2mm_M3_Pad_Via")
+    )
+    (path "/c92c8b98-585f-4866-b931-6fae4c8082b7"
+      (reference "H5") (unit 1) (value "MountingHole") (footprint "MountingHole:MountingHole_3.2mm_M3_Pad_Via")
+    )
+    (path "/70d49a9e-0d44-4486-a0ba-962d0db48d64"
+      (reference "H6") (unit 1) (value "MountingHole") (footprint "MountingHole:MountingHole_3.2mm_M3_Pad_Via")
+    )
     (path "/20bc3c73-e2bf-488f-a0c1-38700b58a060"
       (reference "J1") (unit 1) (value "Super_Prog_Header") (footprint "Connector_Molex:Molex_KK-254_AE-6410-05A_1x05_P2.54mm_Vertical")
     )
     (path "/9f02ea00-3ee8-4183-95b6-7d59f1944b3b"
-      (reference "J2") (unit 1) (value "WS2821B Header") (footprint "Connector_PinHeader_2.54mm:PinHeader_1x03_P2.54mm_Vertical")
+      (reference "J2") (unit 1) (value "WS2821B Header") (footprint "Connector_Molex:Molex_KK-254_AE-6410-03A_1x03_P2.54mm_Vertical")
     )
     (path "/586ec748-563a-478a-82db-706fb951336a/3d412b69-c529-4e16-8a2a-e7a8b0ecba07"
@@
     )
     (path "/586ec748-563a-478a-82db-706fb951336a/7e87b1c4-c7af-4837-a2de-ad1fe5674fd5"
-      (reference "J4") (unit 1) (value "Strip Lighting") (footprint "Connector_PinHeader_1.27mm:PinHeader_1x02_P1.27mm_Vertical")
+      (reference "J4") (unit 1) (value "Strip Lighting") (footprint "Connector_Molex:Molex_KK-254_AE-6410-02A_1x02_P2.54mm_Vertical")
     )
     (path "/586ec748-563a-478a-82db-706fb951336a/fee95448-10a7-4ed4-8a9a-2c61dc26fdd6"
@@
     )
     (path "/5841138f-45b5-44f1-8a37-3c7876e2034c/f6833c7f-3380-437f-a302-f8d62ee108d2"
-      (reference "J19") (unit 1) (value "Stepper Motor Output") (footprint "Connector_PinHeader_2.54mm:PinHeader_1x04_P2.54mm_Vertical")
+      (reference "J19") (unit 1) (value "Stepper Motor Output") (footprint "Connector_JST:JST_XH_B4B-XH-A_1x04_P2.50mm_Vertical")
     )
     (path "/fc507f37-311a-4a88-8803-5135386aa883/17670654-bb51-4b1f-9150-1dc49391563f"
@@
     )
     (path "/3053d1d3-1dd5-4dac-b6cb-5e7828c7a42e/dced00b5-ead7-46bd-ad39-3400c2dba3fa"
-      (reference "J23") (unit 1) (value "limit_switch_A") (footprint "Connector_PinHeader_2.54mm:PinHeader_1x02_P2.54mm_Vertical")
+      (reference "J23") (unit 1) (value "limit_switch_A") (footprint "Connector_Molex:Molex_KK-254_AE-6410-02A_1x02_P2.54mm_Vertical")
     )
     (path "/3053d1d3-1dd5-4dac-b6cb-5e7828c7a42e/f71c8b0d-7bb4-442f-a424-e7bf445805bf"
-      (reference "J24") (unit 1) (value "limit_switch_B") (footprint "Connector_PinHeader_2.54mm:PinHeader_1x02_P2.54mm_Vertical")
+      (reference "J24") (unit 1) (value "limit_switch_B") (footprint "Connector_Molex:Molex_KK-254_AE-6410-02A_1x02_P2.54mm_Vertical")
     )
     (path "/3053d1d3-1dd5-4dac-b6cb-5e7828c7a42e/e7ac43f2-b37d-4a71-ba1f-0cf526594e32"
-      (reference "J25") (unit 1) (value "Optical Encoder") (footprint "Connector_PinHeader_2.54mm:PinHeader_1x05_P2.54mm_Vertical")
+      (reference "J25") (unit 1) (value "Optical Encoder") (footprint "Connector_Molex:Molex_KK-254_AE-6410-05A_1x05_P2.54mm_Vertical")
     )
     (path "/e3a5c764-2bf9-4c0b-b94d-393b25109771"
