File: RemoteLabs_supervisor_PCB/dc_motor_controller.kicad_sch (KiCad schematic)
At the start: 0 parts

Commit message: started working on schematic
Parts:
- added A?: Infineon Motor Shield Uno, Module:Arduino_UNO_R3, symbol 000_Modules_Immo:Infineon Motor Shield Uno
- added J?: MotorController_PWR_OP, symbol Connector:Screw_Terminal_01x03
- added J?: MotorController_PWR_IP, TerminalBlock:TerminalBlock_Altech_AK300-2_P5.00mm, symbol Connector:Screw_Terminal_01x02
- added J?: Motor Output, symbol Connector:Screw_Terminal_01x03
Connections:
- new net: J?.1 (Pin_1), J?.3 (Pin_3) (x2)
- new net: J?.2 (Pin_2), J?.2 (Pin_2)
- new net 12V_IN: J?.1 (Pin_1)
- new net GND_D: A?.29 (GND), A?.6 (GND), A?.7 (GND)
- new net GND_PWR: J?.2 (Pin_2)
- new net INH_1: A?.27 (INH_1)
- new net INH_2: A?.28 (INH_2)
- new net IN_1: A?.18 (IN_1)
- new net IN_2: A?.26 (IN_2)
- new net I_SENSE_1: A?.9 (IS_1)
- new net I_SENSE_2: A?.10 (IS_2)
- no-connect marks 0 -> 7
Other:
- note added: "These Pins are connected OFF BOARD with wire"
Changed lines of the file:
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@@
 (kicad_sch (version 20211123) (generator eeschema)
   (paper "A4")
+  (junction (at 124.46 100.33) (diameter 0) (color 0 0 0 0)
+  )
+  (no_connect (at 152.4 127))
+  (no_connect (at 148.59 127))
+  (no_connect (at 137.16 72.39))
+  (no_connect (at 139.7 72.39))
+  (no_connect (at 138.43 129.54))
+  (no_connect (at 163.83 120.65))
+  (no_connect (at 163.83 123.19))
+  (wire (pts (xy 137.16 49.53) (xy 137.16 54.61))
+    (stroke (width 0) (type default) (color 0 0 0 0))
+  )
+  (polyline (pts (xy 138.43 137.16) (xy 142.24 137.16))
+    (stroke (width 0) (type default) (color 0 0 0 0))
+  )
+  (polyline (pts (xy 148.59 133.35) (xy 144.78 133.35))
+    (stroke (width 0) (type default) (color 0 0 0 0))
+  )
+  (wire (pts (xy 147.32 148.59) (xy 147.32 151.13))
+    (stroke (width 0) (type default) (color 0 0 0 0))
+  )
+  (polyline (pts (xy 148.59 127) (xy 148.59 133.35))
+    (stroke (width 0) (type default) (color 0 0 0 0))
+  )
+  (wire (pts (xy 163.83 115.57) (xy 168.91 115.57))
+    (stroke (width 0) (type default) (color 0 0 0 0))
+  )
+  (wire (pts (xy 119.38 100.33) (xy 124.46 100.33))
+    (stroke (width 0) (type default) (color 0 0 0 0))
+  )
+  (wire (pts (xy 127 101.6) (xy 124.46 101.6))
+    (stroke (width 0) (type default) (color 0 0 0 0))
+  )
+  (wire (pts (xy 144.78 148.59) (xy 144.78 151.13))
+    (stroke (width 0) (type default) (color 0 0 0 0))
+  )
+  (wire (pts (xy 163.83 91.44) (xy 168.91 91.44))
+    (stroke (width 0) (type default) (color 0 0 0 0))
+  )
+  (polyline (pts (xy 138.43 129.54) (xy 138.43 137.16))
+    (stroke (width 0) (type default) (color 0 0 0 0))
+  )
+  (polyline (pts (xy 137.16 60.96) (xy 137.16 72.39))
+    (stroke (width 0) (type default) (color 0 0 0 0))
+  )
+  (polyline (pts (xy 144.78 133.35) (xy 144.78 143.51))
+    (stroke (width 0) (type default) (color 0 0 0 0))
+  )
+  (wire (pts (xy 142.24 148.59) (xy 142.24 151.13))
+    (stroke (width 0) (type default) (color 0 0 0 0))
+  )
+  (wire (pts (xy 119.38 109.22) (xy 127 109.22))
+    (stroke (width 0) (type default) (color 0 0 0 0))
+  )
+  (wire (pts (xy 168.91 85.09) (xy 163.83 85.09))
+    (stroke (width 0) (type default) (color 0 0 0 0))
+  )
+  (polyline (pts (xy 152.4 127) (xy 152.4 137.16))
+    (stroke (width 0) (type default) (color 0 0 0 0))
+  )
+  (wire (pts (xy 124.46 99.06) (xy 127 99.06))
+    (stroke (width 0) (type default) (color 0 0 0 0))
+  )
+  (wire (pts (xy 124.46 101.6) (xy 124.46 100.33))
+    (stroke (width 0) (type default) (color 0 0 0 0))
+  )
+  (polyline (pts (xy 147.32 137.16) (xy 147.32 143.51))
+    (stroke (width 0) (type default) (color 0 0 0 0))
+  )
+  (wire (pts (xy 139.7 49.53) (xy 139.7 54.61))
+    (stroke (width 0) (type default) (color 0 0 0 0))
+  )
+  (polyline (pts (xy 142.24 137.16) (xy 142.24 143.51))
+    (stroke (width 0) (type default) (color 0 0 0 0))
+  )
+  (wire (pts (xy 119.38 111.76) (xy 127 111.76))
+    (stroke (width 0) (type default) (color 0 0 0 0))
+  )
+  (polyline (pts (xy 139.7 59.69) (xy 139.7 72.39))
+    (stroke (width 0) (type default) (color 0 0 0 0))
+  )
+  (wire (pts (xy 124.46 100.33) (xy 124.46 99.06))
+    (stroke (width 0) (type default) (color 0 0 0 0))
+  )
+  (wire (pts (xy 163.83 88.9) (xy 168.91 88.9))
+    (stroke (width 0) (type default) (color 0 0 0 0))
+  )
+  (polyline (pts (xy 152.4 137.16) (xy 147.32 137.16))
+    (stroke (width 0) (type default) (color 0 0 0 0))
+  )
+  (wire (pts (xy 163.83 93.98) (xy 168.91 93.98))
+    (stroke (width 0) (type default) (color 0 0 0 0))
+  )
+  (text "These Pins are connected OFF BOARD\nwith wire" (at 154.94 135.89 0)
+    (effects (font (size 1.27 1.27)) (justify left bottom))
+  )
+  (text "These Pins are connected OFF BOARD\nwith wire" (at 140.97 66.04 0)
+    (effects (font (size 1.27 1.27)) (justify left bottom))
+  )
+  (hierarchical_label "IN_1" (shape input) (at 168.91 115.57 0)
+    (effects (font (size 1.27 1.27)) (justify left))
+  )
+  (hierarchical_label "GND_D" (shape passive) (at 119.38 100.33 180)
+    (effects (font (size 1.27 1.27)) (justify right))
+  )
+  (hierarchical_label "I_SENSE_2" (shape output) (at 119.38 111.76 180)
+    (effects (font (size 1.27 1.27)) (justify right))
+  )
+  (hierarchical_label "INH_1" (shape input) (at 168.91 91.44 0)
+    (effects (font (size 1.27 1.27)) (justify left))
+  )
+  (hierarchical_label "IN_2" (shape input) (at 168.91 93.98 0)
+    (effects (font (size 1.27 1.27)) (justify left))
+  )
+  (hierarchical_label "GND_D" (shape passive) (at 168.91 85.09 0)
+    (effects (font (size 1.27 1.27)) (justify left))
+  )
+  (hierarchical_label "INH_2" (shape input) (at 168.91 88.9 0)
+    (effects (font (size 1.27 1.27)) (justify left))
+  )
+  (hierarchical_label "12V_IN" (shape input) (at 139.7 49.53 90)
+    (effects (font (size 1.27 1.27)) (justify left))
+  )
+  (hierarchical_label "GND_PWR" (shape input) (at 137.16 49.53 90)
+    (effects (font (size 1.27 1.27)) (justify left))
+  )
+  (hierarchical_label "I_SENSE_1" (shape output) (at 119.38 109.22 180)
+    (effects (font (size 1.27 1.27)) (justify right))
+  )
+  (symbol (lib_id "000_Modules_Immo:Infineon Motor Shield Uno") (at 147.32 102.87 0) (unit 1)
+    (in_bom yes) (on_board yes)
+    (property "Reference" "A?" (id 0) (at 144.78 69.85 0))
+    (property "Value" "Infineon Motor Shield Uno" (id 1) (at 156.21 72.39 0))
+    (property "Footprint" "Module:Arduino_UNO_R3" (id 2) (at 182.88 165.1 0)
+      (effects (font (size 1.27 1.27) italic) hide)
+    )
+    (property "Datasheet" "https://docs.rs-online.com/91cb/0900766b81490d99.pdf" (id 3) (at 182.88 165.1 0)
+      (effects (font (size 1.27 1.27)) hide)
+    )
+    (pin "1")
+    (pin "10")
+    (pin "11")
+    (pin "12")
+    (pin "13")
+    (pin "14")
+    (pin "15")
+    (pin "16")
+    (pin "17")
+    (pin "18")
+    (pin "19")
+    (pin "2")
+    (pin "20")
+    (pin "21")
+    (pin "22")
+    (pin "23")
+    (pin "24")
+    (pin "25")
+    (pin "26")
+    (pin "27")
+    (pin "28")
+    (pin "29")
+    (pin "3")
+    (pin "30")
+    (pin "31")
+    (pin "32")
+    (pin "33")
+    (pin "34")
+    (pin "35")
+    (pin "36")
+    (pin "37")
+    (pin "4")
+    (pin "5")
+    (pin "6")
+    (pin "7")
+    (pin "8")
+    (pin "9")
+  )
+  (symbol (lib_id "Connector:Screw_Terminal_01x03") (at 144.78 143.51 90) (unit 1)
+    (in_bom yes) (on_board yes) (fields_autoplaced)
+    (property "Reference" "J?" (id 0) (at 149.86 142.2399 90)
+      (effects (font (size 1.27 1.27)) (justify right))
+    )
+    (property "Value" "MotorController_PWR_OP" (id 1) (at 149.86 144.7799 90)
+      (effects (font (size 1.27 1.27)) (justify right))
+    )
+    (property "Footprint" "" (id 2) (at 144.78 143.51 0)
+      (effects (font (size 1.27 1.27)) hide)
+    )
+    (property "Datasheet" "~" (id 3) (at 144.78 143.51 0)
+      (effects (font (size 1.27 1.27)) hide)
+    )
+    (pin "1")
+    (pin "2")
+    (pin "3")
+  )
+  (symbol (lib_id "Connector:Screw_Terminal_01x02") (at 139.7 59.69 270) (unit 1)
+    (in_bom yes) (on_board yes)
+    (property "Reference" "J?" (id 0) (at 118.11 57.15 90)
+      (effects (font (size 1.27 1.27)) (justify left))
+    )
+    (property "Value" "MotorController_PWR_IP" (id 1) (at 111.76 59.69 90)
+      (effects (font (size 1.27 1.27)) (justify left))
+    )
+    (property "Footprint" "TerminalBlock:TerminalBlock_Altech_AK300-2_P5.00mm" (id 2) (at 139.7 59.69 0)
+      (effects (font (size 1.27 1.27)) hide)
+    )
+    (property "Datasheet" "~" (id 3) (at 139.7 59.69 0)
+      (effects (font (size 1.27 1.27)) hide)
+    )
+    (pin "1")
+    (pin "2")
+  )
+  (symbol (lib_id "Connector:Screw_Terminal_01x03") (at 144.78 156.21 270) (unit 1)
+    (in_bom yes) (on_board yes)
+    (property "Reference" "J?" (id 0) (at 149.86 154.9399 90)
+      (effects (font (size 1.27 1.27)) (justify left))
+    )
+    (property "Value" "Motor Output" (id 1) (at 149.86 157.48 90)
+      (effects (font (size 1.27 1.27)) (justify left))
+    )
+    (property "Footprint" "" (id 2) (at 144.78 156.21 0)
+      (effects (font (size 1.27 1.27)) hide)
+    )
+    (property "Datasheet" "~" (id 3) (at 144.78 156.21 0)
+      (effects (font (size 1.27 1.27)) hide)
+    )
+    (pin "1")
+    (pin "2")
+    (pin "3")
+  )
 )

Commit message: Schematric work
Parts:
- added F?: 2A, Fuse:Fuseholder_Cylinder-5x20mm_Stelvio-Kontek_PTF78_Horizontal_Open, symbol 000_Protection_Immo:Fuse
Connections:
- net 12V_IN: now also F?.1; no longer J?.1 (Pin_1)
- new net: F?.2, J?.1 (Pin_1)
Changed lines of the file:
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@@
+    (stroke (width 0) (type default) (color 0 0 0 0))
+  )
+  (wire (pts (xy 139.7 44.45) (xy 139.7 54.61))
     (stroke (width 0) (type default) (color 0 0 0 0))
   )
@@
     (stroke (width 0) (type default) (color 0 0 0 0))
   )
-  (wire (pts (xy 139.7 49.53) (xy 139.7 54.61))
-    (stroke (width 0) (type default) (color 0 0 0 0))
-  )
   (polyline (pts (xy 142.24 137.16) (xy 142.24 143.51))
     (stroke (width 0) (type default) (color 0 0 0 0))
@@
   )
   (wire (pts (xy 163.83 93.98) (xy 168.91 93.98))
+    (stroke (width 0) (type default) (color 0 0 0 0))
+  )
+  (wire (pts (xy 139.7 33.02) (xy 139.7 36.83))
     (stroke (width 0) (type default) (color 0 0 0 0))
   )
@@
     (effects (font (size 1.27 1.27)) (justify left))
   )
-  (hierarchical_label "12V_IN" (shape input) (at 139.7 49.53 90)
+  (hierarchical_label "12V_IN" (shape input) (at 139.7 33.02 90)
     (effects (font (size 1.27 1.27)) (justify left))
   )
@@
     (pin "3")
   )
+  (symbol (lib_id "000_Protection_Immo:Fuse") (at 139.7 40.64 0) (unit 1)
+    (in_bom yes) (on_board yes) (fields_autoplaced)
+    (property "Reference" "F?" (id 0) (at 142.24 39.3699 0)
+      (effects (font (size 1.27 1.27)) (justify left))
+    )
+    (property "Value" "2A" (id 1) (at 142.24 41.9099 0)
+      (effects (font (size 1.27 1.27)) (justify left))
+    )
+    (property "Footprint" "Fuse:Fuseholder_Cylinder-5x20mm_Stelvio-Kontek_PTF78_Horizontal_Open" (id 2) (at 137.922 40.64 90)
+      (effects (font (size 1.27 1.27)) hide)
+    )
+    (property "Datasheet" "~" (id 3) (at 139.7 40.64 0)
+      (effects (font (size 1.27 1.27)) hide)
+    )
+    (pin "1")
+    (pin "2")
+  )
 )

Commit message: update
Other:
- moved on the sheet: F?
Changed lines of the file:
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@@
   (no_connect (at 163.83 120.65))
   (no_connect (at 163.83 123.19))
-  (wire (pts (xy 137.16 49.53) (xy 137.16 54.61))
+  (wire (pts (xy 137.16 40.64) (xy 137.16 54.61))
     (stroke (width 0) (type default) (color 0 0 0 0))
   )
@@
     (stroke (width 0) (type default) (color 0 0 0 0))
   )
-  (wire (pts (xy 139.7 44.45) (xy 139.7 54.61))
+  (wire (pts (xy 139.7 52.07) (xy 139.7 54.61))
     (stroke (width 0) (type default) (color 0 0 0 0))
   )
@@
     (stroke (width 0) (type default) (color 0 0 0 0))
   )
-  (wire (pts (xy 139.7 33.02) (xy 139.7 36.83))
+  (wire (pts (xy 139.7 40.64) (xy 139.7 44.45))
     (stroke (width 0) (type default) (color 0 0 0 0))
   )
@@
     (effects (font (size 1.27 1.27)) (justify left))
   )
-  (hierarchical_label "12V_IN" (shape input) (at 139.7 33.02 90)
-    (effects (font (size 1.27 1.27)) (justify left))
-  )
-  (hierarchical_label "GND_PWR" (shape input) (at 137.16 49.53 90)
+  (hierarchical_label "12V_IN" (shape input) (at 139.7 40.64 90)
+    (effects (font (size 1.27 1.27)) (justify left))
+  )
+  (hierarchical_label "GND_PWR" (shape input) (at 137.16 40.64 90)
     (effects (font (size 1.27 1.27)) (justify left))
   )
@@
     (pin "3")
   )
-  (symbol (lib_id "000_Protection_Immo:Fuse") (at 139.7 40.64 0) (unit 1)
+  (symbol (lib_id "000_Protection_Immo:Fuse") (at 139.7 48.26 0) (unit 1)
     (in_bom yes) (on_board yes) (fields_autoplaced)
-    (property "Reference" "F?" (id 0) (at 142.24 39.3699 0)
-      (effects (font (size 1.27 1.27)) (justify left))
-    )
-    (property "Value" "2A" (id 1) (at 142.24 41.9099 0)
-      (effects (font (size 1.27 1.27)) (justify left))
-    )
-    (property "Footprint" "Fuse:Fuseholder_Cylinder-5x20mm_Stelvio-Kontek_PTF78_Horizontal_Open" (id 2) (at 137.922 40.64 90)
-      (effects (font (size 1.27 1.27)) hide)
-    )
-    (property "Datasheet" "~" (id 3) (at 139.7 40.64 0)
-      (effects (font (size 1.27 1.27)) hide)
-    )
+    (property "Reference" "F?" (id 0) (at 142.24 46.9899 0)
+      (effects (font (size 1.27 1.27)) (justify left))
+    )
+    (property "Value" "2A" (id 1) (at 142.24 49.5299 0)
+      (effects (font (size 1.27 1.27)) (justify left))
+    )
+    (property "Footprint" "Fuse:Fuseholder_Cylinder-5x20mm_Stelvio-Kontek_PTF78_Horizontal_Open" (id 2) (at 137.922 48.26 90)
+      (effects (font (size 1.27 1.27)) hide)
+    )
+    (property "Datasheet" "~" (id 3) (at 139.7 48.26 0)
+      (effects (font (size 1.27 1.27)) hide)
+    )
