File: RemoteLabs_supervisor_PCB/dc_motor_controller.kicad_sch (KiCad schematic)
At the start: 5 parts

Commit message: Schematic Work
Parts:
- added R? (x2): 470r, Resistor_SMD:R_0805_2012Metric_Pad1.20x1.40mm_HandSolder, symbol 000_Resistors_Immo:Resistor_0805
Connections:
- net INH_2 is gone; now on net INHIBIT: A?.28 (INH_2)
- net GND_D: now also R?.2, R?.2
- net I_SENSE_1: now also R?.1
- net I_SENSE_2: now also R?.1
- net INH_1 renamed INHIBIT
Other:
- note added: "Assume 6.5mA MAX V = 6.5 * 500 / 1000 V = 3.25v"
- note added: "Current sense outputs: I(load) = dk(ilis)*(I(is)-I(is_offset)) Differential Current Sense ratio dk(ilis): dk(ilis) = (I(L2)-I(L1))/((I(is))*(I(L2))-(I(is)*(I(L1)))"
- note added: "I(is_lim) @ Vs = 12v & Tj = 100degC = 5.25 mA"
- note added: "INH Pins can be joined"
- note added: "If the high side drain current is zero (ISD(HS) = 0A) the offset current IIS = IIS(offset) still will be driven. The external resistor RIS determines the voltage per IS output current. The voltage can be calculated by VIS = RIS . IIS. In case of a fault condition the status output is connected to a current source which is independent of the load current and provides IIS(lim). The maximum voltage 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"
- note added: "Must be 1% tolerance for 3.3v max"
Changed lines of the file:
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@@
 (kicad_sch (version 20211123) (generator eeschema)
   (paper "A4")
+  (junction (at 166.37 91.44) (diameter 0) (color 0 0 0 0)
+  )
+  (junction (at 72.39 111.76) (diameter 0) (color 0 0 0 0)
+  )
   (junction (at 124.46 100.33) (diameter 0) (color 0 0 0 0)
+  )
+  (junction (at 63.5 109.22) (diameter 0) (color 0 0 0 0)
   )
   (no_connect (at 152.4 127))
@@
     (stroke (width 0) (type default) (color 0 0 0 0))
   )
+  (wire (pts (xy 166.37 88.9) (xy 166.37 91.44))
+    (stroke (width 0) (type default) (color 0 0 0 0))
+  )
+  (wire (pts (xy 72.39 111.76) (xy 72.39 114.3))
+    (stroke (width 0) (type default) (color 0 0 0 0))
+  )
   (polyline (pts (xy 148.59 133.35) (xy 144.78 133.35))
     (stroke (width 0) (type default) (color 0 0 0 0))
@@
     (stroke (width 0) (type default) (color 0 0 0 0))
   )
+  (wire (pts (xy 63.5 109.22) (xy 127 109.22))
+    (stroke (width 0) (type default) (color 0 0 0 0))
+  )
+  (wire (pts (xy 63.5 113.03) (xy 64.77 113.03))
+    (stroke (width 0) (type default) (color 0 0 0 0))
+  )
   (polyline (pts (xy 148.59 127) (xy 148.59 133.35))
     (stroke (width 0) (type default) (color 0 0 0 0))
@@
     (stroke (width 0) (type default) (color 0 0 0 0))
   )
+  (wire (pts (xy 163.83 88.9) (xy 166.37 88.9))
+    (stroke (width 0) (type default) (color 0 0 0 0))
+  )
   (wire (pts (xy 144.78 148.59) (xy 144.78 151.13))
     (stroke (width 0) (type default) (color 0 0 0 0))
   )
-  (wire (pts (xy 163.83 91.44) (xy 168.91 91.44))
+  (wire (pts (xy 163.83 91.44) (xy 166.37 91.44))
     (stroke (width 0) (type default) (color 0 0 0 0))
   )
@@
     (stroke (width 0) (type default) (color 0 0 0 0))
   )
+  (wire (pts (xy 72.39 111.76) (xy 127 111.76))
+    (stroke (width 0) (type default) (color 0 0 0 0))
+  )
   (wire (pts (xy 142.24 148.59) (xy 142.24 151.13))
     (stroke (width 0) (type default) (color 0 0 0 0))
   )
+  (wire (pts (xy 63.5 110.49) (xy 64.77 110.49))
+    (stroke (width 0) (type default) (color 0 0 0 0))
+  )
   (wire (pts (xy 139.7 52.07) (xy 139.7 54.61))
     (stroke (width 0) (type default) (color 0 0 0 0))
   )
-  (wire (pts (xy 119.38 109.22) (xy 127 109.22))
+  (wire (pts (xy 72.39 121.92) (xy 72.39 124.46))
+    (stroke (width 0) (type default) (color 0 0 0 0))
+  )
+  (wire (pts (xy 63.5 113.03) (xy 63.5 114.3))
+    (stroke (width 0) (type default) (color 0 0 0 0))
+  )
+  (wire (pts (xy 166.37 91.44) (xy 168.91 91.44))
+    (stroke (width 0) (type default) (color 0 0 0 0))
+  )
+  (wire (pts (xy 63.5 109.22) (xy 63.5 110.49))
+    (stroke (width 0) (type default) (color 0 0 0 0))
+  )
+  (wire (pts (xy 52.07 109.22) (xy 63.5 109.22))
     (stroke (width 0) (type default) (color 0 0 0 0))
   )
@@
     (stroke (width 0) (type default) (color 0 0 0 0))
   )
+  (wire (pts (xy 64.77 113.03) (xy 64.77 110.49))
+    (stroke (width 0) (type default) (color 0 0 0 0))
+  )
   (wire (pts (xy 124.46 101.6) (xy 124.46 100.33))
     (stroke (width 0) (type default) (color 0 0 0 0))
@@
     (stroke (width 0) (type default) (color 0 0 0 0))
   )
+  (wire (pts (xy 63.5 121.92) (xy 63.5 124.46))
+    (stroke (width 0) (type default) (color 0 0 0 0))
+  )
   (polyline (pts (xy 142.24 137.16) (xy 142.24 143.51))
     (stroke (width 0) (type default) (color 0 0 0 0))
   )
-  (wire (pts (xy 119.38 111.76) (xy 127 111.76))
+  (wire (pts (xy 52.07 111.76) (xy 72.39 111.76))
     (stroke (width 0) (type default) (color 0 0 0 0))
   )
@@
     (stroke (width 0) (type default) (color 0 0 0 0))
   )
-  (wire (pts (xy 163.83 88.9) (xy 168.91 88.9))
-    (stroke (width 0) (type default) (color 0 0 0 0))
-  )
   (polyline (pts (xy 152.4 137.16) (xy 147.32 137.16))
     (stroke (width 0) (type default) (color 0 0 0 0))
@@
     (stroke (width 0) (type default) (color 0 0 0 0))
   )
+  (text "If the high side drain current is zero (ISD(HS) = 0A) the offset current IIS = IIS(offset) still will be driven.\nThe external resistor RIS determines the voltage per IS output current. The voltage can be calculated by\nVIS = RIS . IIS.\nIn case of a fault condition the status output is connected to a current source which is independent of the load\ncurrent and provides IIS(lim). The maximum voltage at the IS pin is determined by the choice of the external resistor\nand the supply voltage. In case of current limitation the IIS(lim) is activated for 2 * tCLS."
+    (at 48.26 157.48 0)
+    (effects (font (size 0.8 0.8)) (justify left bottom))
+  )
+  (text "Current sense outputs:\n\nI(load) = dk(ilis)*(I(is)-I(is_offset))\n\nDifferential Current Sense ratio dk(ilis):\n\ndk(ilis) = (I(L2)-I(L1))/((I(is))*(I(L2))-(I(is)*(I(L1)))"
+    (at 64.77 171.45 0)
+    (effects (font (size 0.8 0.8)) (justify left bottom))
+  )
+  (text "Assume 6.5mA MAX\n\nV = 6.5 * 500 / 1000\nV = 3.25v" (at 83.82 129.54 0)
+    (effects (font (size 1.27 1.27)) (justify left bottom))
+  )
   (text "These Pins are connected OFF BOARD\nwith wire" (at 154.94 135.89 0)
     (effects (font (size 1.27 1.27)) (justify left bottom))
   )
+  (text "Must be 1% tolerance\nfor 3.3v max" (at 31.75 127 0)
+    (effects (font (size 1.27 1.27)) (justify left bottom))
+  )
+  (text "I(is_lim) @ Vs = 12v & Tj = 100degC\n\n	= 5.25 mA" (at 82.55 120.65 0)
+    (effects (font (size 1.27 1.27)) (justify left bottom))
+  )
   (text "These Pins are connected OFF BOARD\nwith wire" (at 140.97 66.04 0)
     (effects (font (size 1.27 1.27)) (justify left bottom))
   )
+  (text "INH Pins can be joined" (at 181.61 81.28 0)
+    (effects (font (size 1.27 1.27)) (justify left bottom))
+  )
   (hierarchical_label "IN_1" (shape input) (at 168.91 115.57 0)
     (effects (font (size 1.27 1.27)) (justify left))
@@
     (effects (font (size 1.27 1.27)) (justify right))
   )
-  (hierarchical_label "I_SENSE_2" (shape output) (at 119.38 111.76 180)
-    (effects (font (size 1.27 1.27)) (justify right))
-  )
-  (hierarchical_label "INH_1" (shape input) (at 168.91 91.44 0)
+  (hierarchical_label "I_SENSE_2" (shape output) (at 52.07 111.76 180)
+    (effects (font (size 1.27 1.27)) (justify right))
+  )
+  (hierarchical_label "INHIBIT" (shape input) (at 168.91 91.44 0)
     (effects (font (size 1.27 1.27)) (justify left))
   )
@@
     (effects (font (size 1.27 1.27)) (justify left))
   )
-  (hierarchical_label "INH_2" (shape input) (at 168.91 88.9 0)
-    (effects (font (size 1.27 1.27)) (justify left))
+  (hierarchical_label "GND_D" (shape passive) (at 63.5 124.46 270)
+    (effects (font (size 1.27 1.27)) (justify right))
   )
   (hierarchical_label "12V_IN" (shape input) (at 139.7 40.64 90)
@@
     (effects (font (size 1.27 1.27)) (justify left))
   )
-  (hierarchical_label "I_SENSE_1" (shape output) (at 119.38 109.22 180)
+  (hierarchical_label "GND_D" (shape passive) (at 72.39 124.46 270)
+    (effects (font (size 1.27 1.27)) (justify right))
+  )
+  (hierarchical_label "I_SENSE_1" (shape output) (at 52.07 109.22 180)
     (effects (font (size 1.27 1.27)) (justify right))
   )
@@
     (pin "9")
   )
+  (symbol (lib_id "000_Resistors_Immo:Resistor_0805") (at 63.5 118.11 0) (unit 1)
+    (in_bom yes) (on_board yes) (fields_autoplaced)
+    (property "Reference" "R?" (id 0) (at 66.04 116.8399 0)
+      (effects (font (size 1.27 1.27)) (justify left))
+    )
+    (property "Value" "470r" (id 1) (at 66.04 119.3799 0)
+      (effects (font (size 1.27 1.27)) (justify left))
+    )
+    (property "Footprint" "Resistor_SMD:R_0805_2012Metric_Pad1.20x1.40mm_HandSolder" (id 2) (at 61.722 118.11 90)
+      (effects (font (size 1.27 1.27)) hide)
+    )
+    (property "Datasheet" "~" (id 3) (at 63.5 118.11 0)
+      (effects (font (size 1.27 1.27)) hide)
+    )
+    (pin "1")
+    (pin "2")
+  )
   (symbol (lib_id "Connector:Screw_Terminal_01x03") (at 144.78 143.51 90) (unit 1)
     (in_bom yes) (on_board yes) (fields_autoplaced)
@@
     (pin "3")
   )
+  (symbol (lib_id "000_Resistors_Immo:Resistor_0805") (at 72.39 118.11 0) (unit 1)
+    (in_bom yes) (on_board yes) (fields_autoplaced)
+    (property "Reference" "R?" (id 0) (at 74.93 116.8399 0)
+      (effects (font (size 1.27 1.27)) (justify left))
+    )
+    (property "Value" "470r" (id 1) (at 74.93 119.3799 0)
+      (effects (font (size 1.27 1.27)) (justify left))
+    )
+    (property "Footprint" "Resistor_SMD:R_0805_2012Metric_Pad1.20x1.40mm_HandSolder" (id 2) (at 70.612 118.11 90)
+      (effects (font (size 1.27 1.27)) hide)
+    )
+    (property "Datasheet" "~" (id 3) (at 72.39 118.11 0)
+      (effects (font (size 1.27 1.27)) hide)
+    )
+    (pin "1")
+    (pin "2")
+  )
   (symbol (lib_id "Connector:Screw_Terminal_01x02") (at 139.7 59.69 270) (unit 1)

Commit message: lunchtime backup
Connections:
- net INHIBIT renamed ENABLE
Other:
- note added: "INH is active low, so renamed as ENABLE"
Changed lines of the file:
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@@
+    (effects (font (size 1.27 1.27)) (justify left bottom))
+  )
+  (text "INH is active low, so renamed as ENABLE" (at 181.61 81.28 0)
     (effects (font (size 1.27 1.27)) (justify left bottom))
   )
@@
     (effects (font (size 1.27 1.27)) (justify left bottom))
   )
-  (text "INH Pins can be joined" (at 181.61 81.28 0)
+  (text "INH Pins can be joined" (at 181.61 78.74 0)
     (effects (font (size 1.27 1.27)) (justify left bottom))
   )
@@
     (effects (font (size 1.27 1.27)) (justify right))
   )
-  (hierarchical_label "INHIBIT" (shape input) (at 168.91 91.44 0)
+  (hierarchical_label "ENABLE" (shape input) (at 168.91 91.44 0)
     (effects (font (size 1.27 1.27)) (justify left))
   )

Commit message: V1.0 Circuit Design Complete
Parts:
- gave numbers to parts that had none: 7
Other:
- note added: "INH is active low, so renamed as ENABLE (Active HIGH to enable)"
- note removed: "INH is active low, so renamed as ENABLE"
Changed lines of the file:
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@@
     (effects (font (size 1.27 1.27)) (justify left bottom))
   )
-  (text "INH is active low, so renamed as ENABLE" (at 181.61 81.28 0)
+  (text "INH is active low, so renamed as ENABLE \n(Active HIGH to enable)"
+    (at 181.61 83.82 0)
     (effects (font (size 1.27 1.27)) (justify left bottom))
   )
@@
   (symbol (lib_id "000_Modules_Immo:Infineon Motor Shield Uno") (at 147.32 102.87 0) (unit 1)
     (in_bom yes) (on_board yes)
-    (property "Reference" "A?" (id 0) (at 144.78 69.85 0))
+    (property "Reference" "A3" (id 0) (at 144.78 69.85 0))
     (property "Value" "Infineon Motor Shield Uno" (id 1) (at 156.21 72.39 0))
     (property "Footprint" "Module:Arduino_UNO_R3" (id 2) (at 182.88 165.1 0)
@@
   (symbol (lib_id "000_Resistors_Immo:Resistor_0805") (at 63.5 118.11 0) (unit 1)
     (in_bom yes) (on_board yes) (fields_autoplaced)
-    (property "Reference" "R?" (id 0) (at 66.04 116.8399 0)
+    (property "Reference" "R12" (id 0) (at 66.04 116.8399 0)
       (effects (font (size 1.27 1.27)) (justify left))
     )
@@
   (symbol (lib_id "Connector:Screw_Terminal_01x03") (at 144.78 143.51 90) (unit 1)
     (in_bom yes) (on_board yes) (fields_autoplaced)
-    (property "Reference" "J?" (id 0) (at 149.86 142.2399 90)
+    (property "Reference" "J17" (id 0) (at 149.86 142.2399 90)
       (effects (font (size 1.27 1.27)) (justify right))
     )
@@
   (symbol (lib_id "000_Resistors_Immo:Resistor_0805") (at 72.39 118.11 0) (unit 1)
     (in_bom yes) (on_board yes) (fields_autoplaced)
-    (property "Reference" "R?" (id 0) (at 74.93 116.8399 0)
+    (property "Reference" "R13" (id 0) (at 74.93 116.8399 0)
       (effects (font (size 1.27 1.27)) (justify left))
     )
@@
   (symbol (lib_id "Connector:Screw_Terminal_01x02") (at 139.7 59.69 270) (unit 1)
     (in_bom yes) (on_board yes)
-    (property "Reference" "J?" (id 0) (at 118.11 57.15 90)
+    (property "Reference" "J16" (id 0) (at 118.11 57.15 90)
       (effects (font (size 1.27 1.27)) (justify left))
     )
@@
   (symbol (lib_id "Connector:Screw_Terminal_01x03") (at 144.78 156.21 270) (unit 1)
     (in_bom yes) (on_board yes)
-    (property "Reference" "J?" (id 0) (at 149.86 154.9399 90)
+    (property "Reference" "J18" (id 0) (at 149.86 154.9399 90)
       (effects (font (size 1.27 1.27)) (justify left))
     )
@@
   (symbol (lib_id "000_Protection_Immo:Fuse") (at 139.7 48.26 0) (unit 1)
     (in_bom yes) (on_board yes) (fields_autoplaced)
-    (property "Reference" "F?" (id 0) (at 142.24 46.9899 0)
+    (property "Reference" "F2" (id 0) (at 142.24 46.9899 0)
       (effects (font (size 1.27 1.27)) (justify left))
     )

Commit message: Schematic reviewed
Parts:
- J17, J18: footprint (none) -> TerminalBlock:TerminalBlock_Altech_AK300-3_P5.00mm
Changed lines of the file:
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@@
       (effects (font (size 1.27 1.27)) (justify right))
     )
-    (property "Footprint" "" (id 2) (at 144.78 143.51 0)
+    (property "Footprint" "TerminalBlock:TerminalBlock_Altech_AK300-3_P5.00mm" (id 2) (at 144.78 143.51 0)
       (effects (font (size 1.27 1.27)) hide)
     )
@@
     (pin "2")
   )
-  (symbol (lib_id "Connector:Screw_Terminal_01x03") (at 144.78 156.21 270) (unit 1)
+  (symbol (lib_name "Screw_Terminal_01x03_1") (lib_id "Connector:Screw_Terminal_01x03") (at 144.78 156.21 270) (unit 1)
     (in_bom yes) (on_board yes)
     (property "Reference" "J18" (id 0) (at 149.86 154.9399 90)
@@
       (effects (font (size 1.27 1.27)) (justify left))
     )
-    (property "Footprint" "" (id 2) (at 144.78 156.21 0)
+    (property "Footprint" "TerminalBlock:TerminalBlock_Altech_AK300-3_P5.00mm" (id 2) (at 144.78 156.21 0)
       (effects (font (size 1.27 1.27)) hide)
     )
