File: RemoteLabs_supervisor_PCB/dc_motor_controller.kicad_sch (KiCad schematic)
At the start: 7 parts, among them J16 MotorController_PWR_IP, J17 MotorController_PWR_OP, J18 Motor Output

Commit message: mbncmvbc,
Connections:
- net GND_D: now also R12.1, R13.1; no longer R12.2, R13.2
- net I_SENSE_1: now also R12.2; no longer R12.1
- net I_SENSE_2: now also R13.2; no longer R13.1
Other:
- moved on the sheet: R12, R13
Changed lines of the file:
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@@
     (pin "9")
   )
-  (symbol (lib_id "000_Resistors_Immo:Resistor_0805") (at 63.5 118.11 0) (unit 1)
+  (symbol (lib_id "000_Resistors_Immo:Resistor_0805") (at 63.5 118.11 90) (unit 1)
     (in_bom yes) (on_board yes) (fields_autoplaced)
-    (property "Reference" "R12" (id 0) (at 66.04 116.8399 0)
-      (effects (font (size 1.27 1.27)) (justify left))
+    (property "Reference" "R12" (id 0) (at 66.04 116.8399 90)
+      (effects (font (size 1.27 1.27)) (justify right))
     )
-    (property "Value" "470r" (id 1) (at 66.04 119.3799 0)
-      (effects (font (size 1.27 1.27)) (justify left))
+    (property "Value" "470r" (id 1) (at 66.04 119.3799 90)
+      (effects (font (size 1.27 1.27)) (justify right))
     )
-    (property "Footprint" "Resistor_SMD:R_0805_2012Metric_Pad1.20x1.40mm_HandSolder" (id 2) (at 61.722 118.11 90)
+    (property "Footprint" "Resistor_SMD:R_0805_2012Metric_Pad1.20x1.40mm_HandSolder" (id 2) (at 63.5 119.888 90)
       (effects (font (size 1.27 1.27)) hide)
     )
@@
     (pin "3")
   )
-  (symbol (lib_id "000_Resistors_Immo:Resistor_0805") (at 72.39 118.11 0) (unit 1)
+  (symbol (lib_id "000_Resistors_Immo:Resistor_0805") (at 72.39 118.11 90) (unit 1)
     (in_bom yes) (on_board yes) (fields_autoplaced)
-    (property "Reference" "R13" (id 0) (at 74.93 116.8399 0)
-      (effects (font (size 1.27 1.27)) (justify left))
+    (property "Reference" "R13" (id 0) (at 74.93 116.8399 90)
+      (effects (font (size 1.27 1.27)) (justify right))
     )
-    (property "Value" "470r" (id 1) (at 74.93 119.3799 0)
-      (effects (font (size 1.27 1.27)) (justify left))
+    (property "Value" "470r" (id 1) (at 74.93 119.3799 90)
+      (effects (font (size 1.27 1.27)) (justify right))
     )
-    (property "Footprint" "Resistor_SMD:R_0805_2012Metric_Pad1.20x1.40mm_HandSolder" (id 2) (at 70.612 118.11 90)
+    (property "Footprint" "Resistor_SMD:R_0805_2012Metric_Pad1.20x1.40mm_HandSolder" (id 2) (at 72.39 119.888 90)
       (effects (font (size 1.27 1.27)) hide)
     )
@@
     (pin "2")
   )
-  (symbol (lib_name "Screw_Terminal_01x03_1") (lib_id "Connector:Screw_Terminal_01x03") (at 144.78 156.21 270) (unit 1)
+  (symbol (lib_id "Connector:Screw_Terminal_01x03") (at 144.78 156.21 270) (unit 1)
     (in_bom yes) (on_board yes)
     (property "Reference" "J18" (id 0) (at 149.86 154.9399 90)

Commit message: Started PCB layout
Parts:
- A3: footprint Module:Arduino_UNO_R3 -> Module:Infineon Motor Sheild hiddenPins
- J17: value MotorController_PWR_OP -> MotorController
- J18: value Motor Output -> DC Motor Output
Connections:
- net HC3: now reaches J17.1 (Pin_1), J18.3 (Pin_3)
- net HC2: now reaches J17.2 (Pin_2), J18.2 (Pin_2)
- net HC1: now reaches J17.3 (Pin_3), J18.1 (Pin_1)
- net HC: now reaches F2.2, J16.1 (Pin_1)
Changed lines of the file:
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@@
+    (stroke (width 0) (type default) (color 0 0 0 0))
+  )
+  (wire (pts (xy 72.39 121.92) (xy 72.39 124.46))
+    (stroke (width 0) (type default) (color 0 0 0 0))
+  )
+  (wire (pts (xy 63.5 113.03) (xy 63.5 114.3))
+    (stroke (width 0) (type default) (color 0 0 0 0))
+  )
+  (wire (pts (xy 166.37 91.44) (xy 168.91 91.44))
+    (stroke (width 0) (type default) (color 0 0 0 0))
+  )
+  (wire (pts (xy 63.5 109.22) (xy 63.5 110.49))
+    (stroke (width 0) (type default) (color 0 0 0 0))
+  )
+  (wire (pts (xy 52.07 109.22) (xy 63.5 109.22))
+    (stroke (width 0) (type default) (color 0 0 0 0))
+  )
+  (wire (pts (xy 168.91 85.09) (xy 163.83 85.09))
+    (stroke (width 0) (type default) (color 0 0 0 0))
+  )
+  (polyline (pts (xy 152.4 127) (xy 152.4 137.16))
+    (stroke (width 0) (type default) (color 0 0 0 0))
+  )
+  (wire (pts (xy 124.46 99.06) (xy 127 99.06))
+    (stroke (width 0) (type default) (color 0 0 0 0))
+  )
+  (wire (pts (xy 64.77 113.03) (xy 64.77 110.49))
     (stroke (width 0) (type default) (color 0 0 0 0))
   )
   (wire (pts (xy 139.7 52.07) (xy 139.7 54.61))
-    (stroke (width 0) (type default) (color 0 0 0 0))
-  )
-  (wire (pts (xy 72.39 121.92) (xy 72.39 124.46))
-    (stroke (width 0) (type default) (color 0 0 0 0))
-  )
-  (wire (pts (xy 63.5 113.03) (xy 63.5 114.3))
-    (stroke (width 0) (type default) (color 0 0 0 0))
-  )
-  (wire (pts (xy 166.37 91.44) (xy 168.91 91.44))
-    (stroke (width 0) (type default) (color 0 0 0 0))
-  )
-  (wire (pts (xy 63.5 109.22) (xy 63.5 110.49))
-    (stroke (width 0) (type default) (color 0 0 0 0))
-  )
-  (wire (pts (xy 52.07 109.22) (xy 63.5 109.22))
-    (stroke (width 0) (type default) (color 0 0 0 0))
-  )
-  (wire (pts (xy 168.91 85.09) (xy 163.83 85.09))
-    (stroke (width 0) (type default) (color 0 0 0 0))
-  )
-  (polyline (pts (xy 152.4 127) (xy 152.4 137.16))
-    (stroke (width 0) (type default) (color 0 0 0 0))
-  )
-  (wire (pts (xy 124.46 99.06) (xy 127 99.06))
-    (stroke (width 0) (type default) (color 0 0 0 0))
-  )
-  (wire (pts (xy 64.77 113.03) (xy 64.77 110.49))
     (stroke (width 0) (type default) (color 0 0 0 0))
   )
@@
   )
   (text "INH Pins can be joined" (at 181.61 78.74 0)
+    (effects (font (size 1.27 1.27)) (justify left bottom))
+  )
+  (label "HC1" (at 147.32 151.13 90)
+    (effects (font (size 1.27 1.27)) (justify left bottom))
+  )
+  (label "HC3" (at 142.24 151.13 90)
+    (effects (font (size 1.27 1.27)) (justify left bottom))
+  )
+  (label "HC" (at 139.7 54.61 90)
+    (effects (font (size 1.27 1.27)) (justify left bottom))
+  )
+  (label "HC2" (at 144.78 151.13 90)
     (effects (font (size 1.27 1.27)) (justify left bottom))
   )
@@
     (property "Reference" "A3" (id 0) (at 144.78 69.85 0))
     (property "Value" "Infineon Motor Shield Uno" (id 1) (at 156.21 72.39 0))
-    (property "Footprint" "Module:Arduino_UNO_R3" (id 2) (at 182.88 165.1 0)
+    (property "Footprint" "Module:Infineon Motor Sheild hiddenPins" (id 2) (at 182.88 165.1 0)
       (effects (font (size 1.27 1.27) italic) hide)
     )
@@
       (effects (font (size 1.27 1.27)) (justify right))
     )
-    (property "Value" "MotorController_PWR_OP" (id 1) (at 149.86 144.7799 90)
+    (property "Value" "MotorController" (id 1) (at 149.86 144.7799 90)
       (effects (font (size 1.27 1.27)) (justify right))
     )
@@
       (effects (font (size 1.27 1.27)) (justify left))
     )
-    (property "Value" "Motor Output" (id 1) (at 149.86 157.48 90)
-      (effects (font (size 1.27 1.27)) (justify left))
-    )
+    (property "Value" "DC Motor Output" (id 1) (at 149.86 157.48 90)
+      (effects (font (size 1.27 1.27)) (justify left))
+    )

Commit message: Edited PCB design for V1.1
- Changed pin sizes for stepper motor
- Change pin sizes for DC/DC Buck module.
- In process of changing text to be readable by human beings
Parts:
- J16: value MotorController_PWR_IP -> DC Motor PWR
- J17: value MotorController -> MotorController Output
Changed lines of the file:
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@@
       (effects (font (size 1.27 1.27)) (justify right))
     )
-    (property "Value" "MotorController" (id 1) (at 149.86 144.7799 90)
+    (property "Value" "MotorController Output" (id 1) (at 149.86 144.7799 90)
       (effects (font (size 1.27 1.27)) (justify right))
     )
@@
   (symbol (lib_id "Connector:Screw_Terminal_01x02") (at 139.7 59.69 270) (unit 1)
     (in_bom yes) (on_board yes)
-    (property "Reference" "J16" (id 0) (at 118.11 57.15 90)
+    (property "Reference" "J16" (id 0) (at 127.635 57.785 90)
       (effects (font (size 1.27 1.27)) (justify left))
     )
-    (property "Value" "MotorController_PWR_IP" (id 1) (at 111.76 59.69 90)
+    (property "Value" "DC Motor PWR" (id 1) (at 121.285 60.325 90)
       (effects (font (size 1.27 1.27)) (justify left))
     )

Commit message: CHANGES
Parts:
- A3: symbol 000_Modules_Immo:Infineon Motor Shield Uno -> 000_Modules_Immo:Infineon Motor Shield MOD
Connections:
- net PENDULUM_PIN_1: now reaches A3.19 (D4)
- net PENDULUM_PIN_2: now reaches A3.20 (D5)
- net PENDULUM_PIN_3: now reaches A3.21 (D6)
- net PENDULUM_PIN_4: now reaches A3.22 (D7)
- net PENDULUM_PIN_5: now reaches A3.23 (D8)
- net 5V_IN: now reaches A3.5 (5V)
- no-connect marks 7 -> 10
Other:
- note added: "None of these pins are connected on Infineon Board, so can be used for pendulum driver"
Changed lines of the file:
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@@
   (junction (at 63.5 109.22) (diameter 0) (color 0 0 0 0)
   )
+  (no_connect (at 127 104.14))
   (no_connect (at 152.4 127))
   (no_connect (at 148.59 127))
@@
   (no_connect (at 163.83 120.65))
   (no_connect (at 163.83 123.19))
+  (no_connect (at 163.83 99.06))
+  (no_connect (at 163.83 96.52))
+  (wire (pts (xy 163.83 113.03) (xy 166.37 113.03))
+    (stroke (width 0) (type default) (color 0 0 0 0))
+  )
   (wire (pts (xy 137.16 40.64) (xy 137.16 54.61))
     (stroke (width 0) (type default) (color 0 0 0 0))
@@
     (stroke (width 0) (type default) (color 0 0 0 0))
   )
+  (wire (pts (xy 124.46 96.52) (xy 127 96.52))
+    (stroke (width 0) (type default) (color 0 0 0 0))
+  )
   (polyline (pts (xy 147.32 137.16) (xy 147.32 143.51))
     (stroke (width 0) (type default) (color 0 0 0 0))
@@
     (stroke (width 0) (type default) (color 0 0 0 0))
   )
+  (wire (pts (xy 163.83 110.49) (xy 166.37 110.49))
+    (stroke (width 0) (type default) (color 0 0 0 0))
+  )
   (wire (pts (xy 52.07 111.76) (xy 72.39 111.76))
     (stroke (width 0) (type default) (color 0 0 0 0))
   )
+  (wire (pts (xy 163.83 101.6) (xy 166.37 101.6))
+    (stroke (width 0) (type default) (color 0 0 0 0))
+  )
   (polyline (pts (xy 139.7 59.69) (xy 139.7 72.39))
     (stroke (width 0) (type default) (color 0 0 0 0))
@@
     (stroke (width 0) (type default) (color 0 0 0 0))
   )
+  (wire (pts (xy 163.83 105.41) (xy 166.37 105.41))
+    (stroke (width 0) (type default) (color 0 0 0 0))
+  )
   (polyline (pts (xy 152.4 137.16) (xy 147.32 137.16))
     (stroke (width 0) (type default) (color 0 0 0 0))
   )
   (wire (pts (xy 163.83 93.98) (xy 168.91 93.98))
+    (stroke (width 0) (type default) (color 0 0 0 0))
+  )
+  (wire (pts (xy 163.83 107.95) (xy 166.37 107.95))
     (stroke (width 0) (type default) (color 0 0 0 0))
   )
@@
     (effects (font (size 1.27 1.27)) (justify left bottom))
   )
+  (text "None of these pins are connected\n on Infineon Board, so can be used\nfor pendulum driver"
+    (at 182.88 96.52 0)
+    (effects (font (size 1.27 1.27)) (justify left bottom))
+  )
   (label "HC1" (at 147.32 151.13 90)
     (effects (font (size 1.27 1.27)) (justify left bottom))
@@
     (effects (font (size 1.27 1.27)) (justify left bottom))
   )
+  (hierarchical_label "PENDULUM_PIN_1" (shape input) (at 166.37 113.03 0)
+    (effects (font (size 1.27 1.27)) (justify left))
+  )
+  (hierarchical_label "PENDULUM_PIN_5" (shape input) (at 166.37 101.6 0)
+    (effects (font (size 1.27 1.27)) (justify left))
+  )
   (hierarchical_label "IN_1" (shape input) (at 168.91 115.57 0)
     (effects (font (size 1.27 1.27)) (justify left))
@@
     (effects (font (size 1.27 1.27)) (justify right))
   )
+  (hierarchical_label "PENDULUM_PIN_2" (shape input) (at 166.37 110.49 0)
+    (effects (font (size 1.27 1.27)) (justify left))
+  )
   (hierarchical_label "I_SENSE_2" (shape output) (at 52.07 111.76 180)
     (effects (font (size 1.27 1.27)) (justify right))
@@
     (effects (font (size 1.27 1.27)) (justify left))
   )
+  (hierarchical_label "PENDULUM_PIN_3" (shape input) (at 166.37 107.95 0)
+    (effects (font (size 1.27 1.27)) (justify left))
+  )
+  (hierarchical_label "PENDULUM_PIN_4" (shape input) (at 166.37 105.41 0)
+    (effects (font (size 1.27 1.27)) (justify left))
+  )
   (hierarchical_label "GND_PWR" (shape input) (at 137.16 40.64 90)
     (effects (font (size 1.27 1.27)) (justify left))
   )
+  (hierarchical_label "5V_IN" (shape input) (at 124.46 96.52 180)
+    (effects (font (size 1.27 1.27)) (justify right))
+  )
   (hierarchical_label "GND_D" (shape passive) (at 72.39 124.46 270)
     (effects (font (size 1.27 1.27)) (justify right))
@@
     (effects (font (size 1.27 1.27)) (justify right))
   )
-  (symbol (lib_id "000_Modules_Immo:Infineon Motor Shield Uno") (at 147.32 102.87 0) (unit 1)
+  (symbol (lib_id "000_Modules_Immo:Infineon Motor Shield MOD") (at 147.32 102.87 0) (unit 1)
     (in_bom yes) (on_board yes)
     (property "Reference" "A3" (id 0) (at 144.78 69.85 0))
     (property "Value" "Infineon Motor Shield Uno" (id 1) (at 156.21 72.39 0))
-    (property "Footprint" "Module:Infineon Motor Sheild hiddenPins" (id 2) (at 182.88 165.1 0)
+    (property "Footprint" "Module:Infineon Motor Sheild hiddenPins" (id 2) (at 171.45 158.75 0)
       (effects (font (size 1.27 1.27) italic) hide)
     )
-    (property "Datasheet" "https://docs.rs-online.com/91cb/0900766b81490d99.pdf" (id 3) (at 182.88 165.1 0)
+    (property "Datasheet" "https://docs.rs-online.com/91cb/0900766b81490d99.pdf" (id 3) (at 172.72 156.21 0)
       (effects (font (size 1.27 1.27)) hide)
     )

Commit message: Version 1.2 PCB
Connections:
- net PENDULUM_PIN_8: now reaches A3.17 (D2)
- net PENDULUM_PIN_6: now reaches A3.24 (D9)
- net PENDULUM_PIN_7: now reaches A3.25 (D10)
- no-connect marks 10 -> 8
Other:
- note added: "Pendulum Notes: Pinout: Enable Drive Pin 1 Load pin 2 STUDENT_ENABLE pin 3 Stu LED 1 pin 4 Stu LED 2 pin 5 Stu LED 3 pin 6 Sup LED 3 pin 7 Sup LED 1 pin 8 Sup LED 2 Pin 2 is enable, when supervisor enables student control HIGH is received here additionally to differentiate control of LEDs"
Changed lines of the file:
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@@
   (no_connect (at 163.83 120.65))
   (no_connect (at 163.83 123.19))
-  (no_connect (at 163.83 99.06))
-  (no_connect (at 163.83 96.52))
   (wire (pts (xy 163.83 113.03) (xy 166.37 113.03))
     (stroke (width 0) (type default) (color 0 0 0 0))
@@
     (stroke (width 0) (type default) (color 0 0 0 0))
   )
+  (wire (pts (xy 163.83 118.11) (xy 166.37 118.11))
+    (stroke (width 0) (type default) (color 0 0 0 0))
+  )
   (wire (pts (xy 144.78 148.59) (xy 144.78 151.13))
     (stroke (width 0) (type default) (color 0 0 0 0))
@@
     (stroke (width 0) (type default) (color 0 0 0 0))
   )
+  (wire (pts (xy 163.83 99.06) (xy 166.37 99.06))
+    (stroke (width 0) (type default) (color 0 0 0 0))
+  )
   (wire (pts (xy 63.5 110.49) (xy 64.77 110.49))
+    (stroke (width 0) (type default) (color 0 0 0 0))
+  )
+  (wire (pts (xy 163.83 96.52) (xy 166.37 96.52))
     (stroke (width 0) (type default) (color 0 0 0 0))
   )
@@
     (effects (font (size 0.8 0.8)) (justify left bottom))
   )
-  (text "Assume 6.5mA MAX\n\nV = 6.5 * 500 / 1000\nV = 3.25v" (at 83.82 129.54 0)
+  (text "Assume 6.5mA MAX\n\nV = 6.5 * 500 / 1000\nV = 3.25v" (at 36.83 102.87 0)
     (effects (font (size 1.27 1.27)) (justify left bottom))
   )
   (text "These Pins are connected OFF BOARD\nwith wire" (at 154.94 135.89 0)
+    (effects (font (size 1.27 1.27)) (justify left bottom))
+  )
+  (text "Pendulum Notes:\n\nPinout:\nEnable 		Drive\nPin 1		Load\npin 2		STUDENT_ENABLE\npin 3		Stu LED 1\npin 4		Stu LED 2\npin 5 		Stu LED 3\npin 6 		Sup LED 3\npin 7 		Sup LED 1\npin 8		Sup LED 2\n\nPin 2 is enable, when supervisor\nenables student control HIGH is received\nhere additionally to differentiate control of LEDs"
+    (at 208.28 126.365 0)
     (effects (font (size 1.27 1.27)) (justify left bottom))
   )
@@
     (effects (font (size 1.27 1.27)) (justify left bottom))
   )
-  (text "I(is_lim) @ Vs = 12v & Tj = 100degC\n\n	= 5.25 mA" (at 82.55 120.65 0)
+  (text "I(is_lim) @ Vs = 12v & Tj = 100degC\n\n	= 5.25 mA" (at 35.56 93.98 0)
     (effects (font (size 1.27 1.27)) (justify left bottom))
   )
@@
   )
   (text "None of these pins are connected\n on Infineon Board, so can be used\nfor pendulum driver"
-    (at 182.88 96.52 0)
+    (at 183.515 90.805 0)
     (effects (font (size 1.27 1.27)) (justify left bottom))
   )
@@
     (effects (font (size 1.27 1.27)) (justify right))
   )
+  (hierarchical_label "PENDULUM_PIN_8" (shape input) (at 166.37 118.11 0)
+    (effects (font (size 1.27 1.27)) (justify left))
+  )
   (hierarchical_label "ENABLE" (shape input) (at 168.91 91.44 0)
     (effects (font (size 1.27 1.27)) (justify left))
@@
     (effects (font (size 1.27 1.27)) (justify left))
   )
+  (hierarchical_label "PENDULUM_PIN_6" (shape input) (at 166.37 99.06 0)
+    (effects (font (size 1.27 1.27)) (justify left))
+  )
+  (hierarchical_label "PENDULUM_PIN_7" (shape input) (at 166.37 96.52 0)
+    (effects (font (size 1.27 1.27)) (justify left))
+  )
