File: RemoteLabs_supervisor_PCB/digital_signal_buffers.kicad_sch (KiCad schematic)
At the start: 30 parts

Commit message: Schematric work
Connections:
- net 5V_VCC: no longer U?.14 (VCC), U?.14 (VCC), U?.14 (VCC)
- net D_IN_B: now also U?.1; no longer U?.3
- net D_IN_C: now also U?.1; no longer U?.5
- net D_IN_D: now also U?.1; no longer U?.9
- net D_IN_E: now also U?.1; no longer U?.11
- net D_IN_F: now also U?.1; no longer U?.13
- net D_OUT_B1: now also U?.2; no longer U?.4
- net D_OUT_B2: now also U?.2; no longer U?.4
- net D_OUT_C1: now also U?.2; no longer U?.6
- net D_OUT_C2: now also U?.2; no longer U?.6
- net D_OUT_D1: now also U?.2; no longer U?.8
- net D_OUT_D2: now also U?.2; no longer U?.8
- net D_OUT_E1: now also U?.2; no longer U?.10
- net D_OUT_E2: now also U?.2; no longer U?.10
- net D_OUT_F1: now also U?.2; no longer U?.12
- net D_OUT_F2: now also U?.2; no longer U?.12
- net GND_D: no longer U?.7 (GND), U?.7 (GND), U?.7 (GND)
- new net: U?.1, U?.1, U?.2 (x5)
Changed lines of the file:
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@@
     (effects (font (size 1.27 1.27)) (justify right))
   )
-  (symbol (lib_id "000_Capacitor_Film_Immo:cap_film_0805") (at 228.6 50.8 0) (unit 1)
+  (symbol (lib_id "000_Capacitor_Film_Immo:cap_film_0805") (at 228.6 50.8 0)
     (in_bom yes) (on_board yes)
     (property "Reference" "C?" (id 0) (at 224.79 48.26 0)
@@
     (pin "2")
   )
-  (symbol (lib_id "000_Capacitor_Film_Immo:cap_film_0805") (at 200.66 50.8 0) (unit 1)
+  (symbol (lib_id "000_Capacitor_Film_Immo:cap_film_0805") (at 200.66 50.8 0)
     (in_bom yes) (on_board yes)
     (property "Reference" "C?" (id 0) (at 196.85 48.26 0)
@@
     (pin "2")
   )
-  (symbol (lib_id "74xx:74LS07") (at 144.78 156.21 0) (unit 6)
+  (symbol (lib_id "74xx:74LS07") (at 144.78 156.21 0)
     (in_bom yes) (on_board yes) (fields_autoplaced)
     (property "Reference" "U?" (id 0) (at 144.78 147.32 0))
@@
     (pin "13")
   )
-  (symbol (lib_id "74xx:74LS07") (at 144.78 41.91 0) (unit 1)
+  (symbol (lib_id "74xx:74LS07") (at 144.78 41.91 0)
     (in_bom yes) (on_board yes) (fields_autoplaced)
     (property "Reference" "U?" (id 0) (at 144.78 33.02 0))
@@
     (pin "2")
   )
-  (symbol (lib_id "74xx:74LS07") (at 107.95 41.91 0) (unit 1)
+  (symbol (lib_id "74xx:74LS07") (at 107.95 41.91 0)
     (in_bom yes) (on_board yes) (fields_autoplaced)
     (property "Reference" "U?" (id 0) (at 107.95 33.02 0))
@@
     (pin "2")
   )
-  (symbol (lib_id "74xx:74LS07") (at 209.55 50.8 0) (unit 7)
+  (symbol (lib_id "74xx:74LS07") (at 209.55 50.8 0)
     (in_bom yes) (on_board yes) (fields_autoplaced)
     (property "Reference" "U?" (id 0) (at 215.9 49.5299 0)
@@
     (pin "7")
   )
-  (symbol (lib_id "4xxx:4069") (at 58.42 177.8 0) (unit 6)
+  (symbol (lib_id "4xxx:4069") (at 58.42 177.8 0)
     (in_bom yes) (on_board yes) (fields_autoplaced)
     (property "Reference" "U?" (id 0) (at 58.42 168.91 0))
@@
     (pin "13")
   )
-  (symbol (lib_id "74xx:74LS07") (at 144.78 64.77 0) (unit 2)
+  (symbol (lib_id "74xx:74LS07") (at 144.78 64.77 0)
     (in_bom yes) (on_board yes) (fields_autoplaced)
     (property "Reference" "U?" (id 0) (at 144.78 55.88 0))
@@
     (pin "4")
   )
-  (symbol (lib_id "74xx:74LS07") (at 107.95 133.35 0) (unit 5)
+  (symbol (lib_id "74xx:74LS07") (at 107.95 133.35 0)
     (in_bom yes) (on_board yes) (fields_autoplaced)
     (property "Reference" "U?" (id 0) (at 107.95 124.46 0))
@@
     (pin "11")
   )
-  (symbol (lib_id "74xx:74LS07") (at 133.35 123.19 0) (unit 5)
+  (symbol (lib_id "74xx:74LS07") (at 133.35 123.19 0)
     (in_bom yes) (on_board yes) (fields_autoplaced)
     (property "Reference" "U?" (id 0) (at 133.35 114.3 0))
@@
     (pin "11")
   )
-  (symbol (lib_id "74xx:74LS07") (at 133.35 31.75 0) (unit 1)
+  (symbol (lib_id "74xx:74LS07") (at 133.35 31.75 0)
     (in_bom yes) (on_board yes) (fields_autoplaced)
     (property "Reference" "U?" (id 0) (at 133.35 22.86 0))
@@
     (pin "2")
   )
-  (symbol (lib_id "4xxx:4081") (at 40.64 193.04 0) (unit 4)
+  (symbol (lib_id "4xxx:4081") (at 40.64 193.04 0)
     (in_bom yes) (on_board yes)
     (property "Reference" "U?" (id 0) (at 39.37 185.42 0))
@@
     (pin "13")
   )
-  (symbol (lib_id "4xxx:4069") (at 40.64 177.8 0) (unit 5)
+  (symbol (lib_id "4xxx:4069") (at 40.64 177.8 0)
     (in_bom yes) (on_board yes) (fields_autoplaced)
     (property "Reference" "U?" (id 0) (at 40.64 168.91 0))
@@
     (pin "11")
   )
-  (symbol (lib_id "74xx:74HC86") (at 24.13 193.04 0) (unit 4)
+  (symbol (lib_id "74xx:74HC86") (at 24.13 193.04 0)
     (in_bom yes) (on_board yes) (fields_autoplaced)
     (property "Reference" "U?" (id 0) (at 23.8252 184.15 0))
@@
     (pin "13")
   )
-  (symbol (lib_id "000_Capacitor_Film_Immo:cap_film_0805") (at 256.54 50.8 0) (unit 1)
+  (symbol (lib_id "000_Capacitor_Film_Immo:cap_film_0805") (at 256.54 50.8 0)
     (in_bom yes) (on_board yes)
     (property "Reference" "C?" (id 0) (at 252.73 48.26 0)
@@
     (pin "2")
   )
-  (symbol (lib_id "74xx:74LS07") (at 144.78 133.35 0) (unit 5)
+  (symbol (lib_id "74xx:74LS07") (at 144.78 133.35 0)
     (in_bom yes) (on_board yes) (fields_autoplaced)
     (property "Reference" "U?" (id 0) (at 144.78 124.46 0))
@@
     (pin "11")
   )
-  (symbol (lib_id "74xx:74LS07") (at 144.78 87.63 0) (unit 3)
+  (symbol (lib_id "74xx:74LS07") (at 144.78 87.63 0)
     (in_bom yes) (on_board yes) (fields_autoplaced)
     (property "Reference" "U?" (id 0) (at 144.78 78.74 0))
@@
     (pin "6")
   )
-  (symbol (lib_id "74xx:74LS07") (at 107.95 110.49 0) (unit 4)
+  (symbol (lib_id "74xx:74LS07") (at 107.95 110.49 0)
     (in_bom yes) (on_board yes) (fields_autoplaced)
     (property "Reference" "U?" (id 0) (at 107.95 101.6 0))
@@
     (pin "9")
   )
-  (symbol (lib_id "74xx:74LS07") (at 107.95 64.77 0) (unit 2)
+  (symbol (lib_id "74xx:74LS07") (at 107.95 64.77 0)
     (in_bom yes) (on_board yes)
     (property "Reference" "U?" (id 0) (at 107.95 55.88 0))
@@
     (pin "4")
   )
-  (symbol (lib_id "74xx:74LS07") (at 133.35 100.33 0) (unit 4)
+  (symbol (lib_id "74xx:74LS07") (at 133.35 100.33 0)
     (in_bom yes) (on_board yes) (fields_autoplaced)
     (property "Reference" "U?" (id 0) (at 133.35 91.44 0))
@@
     (pin "9")
   )
-  (symbol (lib_id "74xx:74LS07") (at 133.35 54.61 0) (unit 2)
+  (symbol (lib_id "74xx:74LS07") (at 133.35 54.61 0)
     (in_bom yes) (on_board yes)
     (property "Reference" "U?" (id 0) (at 133.35 45.72 0))
@@
     (pin "4")
   )
-  (symbol (lib_id "74xx:74LS07") (at 265.43 50.8 0) (unit 7)
+  (symbol (lib_id "74xx:74LS07") (at 265.43 50.8 0)
     (in_bom yes) (on_board yes) (fields_autoplaced)
     (property "Reference" "U?" (id 0) (at 271.78 49.5299 0)
@@
     (pin "7")
   )
-  (symbol (lib_id "74xx:74LS07") (at 107.95 156.21 0) (unit 6)
+  (symbol (lib_id "74xx:74LS07") (at 107.95 156.21 0)
     (in_bom yes) (on_board yes) (fields_autoplaced)
     (property "Reference" "U?" (id 0) (at 107.95 147.32 0))
@@
     (pin "13")
   )
-  (symbol (lib_id "74xx:74LS07") (at 133.35 146.05 0) (unit 6)
+  (symbol (lib_id "74xx:74LS07") (at 133.35 146.05 0)
     (in_bom yes) (on_board yes) (fields_autoplaced)
     (property "Reference" "U?" (id 0) (at 133.35 137.16 0))
@@
     (pin "13")
   )
-  (symbol (lib_id "4xxx:4069") (at 22.86 177.8 0) (unit 4)
+  (symbol (lib_id "4xxx:4069") (at 22.86 177.8 0)
     (in_bom yes) (on_board yes) (fields_autoplaced)
     (property "Reference" "U?" (id 0) (at 22.86 168.91 0))
@@
     (pin "9")
   )
-  (symbol (lib_id "4xxx:4081") (at 58.42 193.04 0) (unit 3)
+  (symbol (lib_id "4xxx:4081") (at 58.42 193.04 0)
     (in_bom yes) (on_board yes) (fields_autoplaced)
     (property "Reference" "U?" (id 0) (at 58.42 184.15 0))
@@
     (pin "9")
   )
-  (symbol (lib_id "74xx:74LS07") (at 133.35 77.47 0) (unit 3)
+  (symbol (lib_id "74xx:74LS07") (at 133.35 77.47 0)
     (in_bom yes) (on_board yes) (fields_autoplaced)
     (property "Reference" "U?" (id 0) (at 133.35 68.58 0))
@@
     (pin "6")
   )
-  (symbol (lib_id "74xx:74LS07") (at 144.78 110.49 0) (unit 4)
+  (symbol (lib_id "74xx:74LS07") (at 144.78 110.49 0)
     (in_bom yes) (on_board yes) (fields_autoplaced)
     (property "Reference" "U?" (id 0) (at 144.78 101.6 0))
@@
     (pin "9")
   )
-  (symbol (lib_id "74xx:74LS07") (at 237.49 50.8 0) (unit 7)
+  (symbol (lib_id "74xx:74LS07") (at 237.49 50.8 0)
     (in_bom yes) (on_board yes)
     (property "Reference" "U?" (id 0) (at 243.84 49.5299 0)
@@
     (pin "7")
   )
-  (symbol (lib_id "74xx:74LS07") (at 107.95 87.63 0) (unit 3)
+  (symbol (lib_id "74xx:74LS07") (at 107.95 87.63 0)
     (in_bom yes) (on_board yes) (fields_autoplaced)
     (property "Reference" "U?" (id 0) (at 107.95 78.74 0))

Commit message: adding test sketch
Connections:
- net D_IN_B: now also U?.3; no longer U?.1
- net D_IN_C: now also U?.5; no longer U?.1
- net D_IN_D: now also U?.9; no longer U?.1
- net D_IN_E: now also U?.11; no longer U?.1
- net D_IN_F: now also U?.13; no longer U?.1
- net D_OUT_B1: now also U?.4; no longer U?.2
- net D_OUT_B2: now also U?.4; no longer U?.2
- net D_OUT_C1: now also U?.6; no longer U?.2
- net D_OUT_C2: now also U?.6; no longer U?.2
- net D_OUT_D1: now also U?.8; no longer U?.2
- net D_OUT_D2: now also U?.8; no longer U?.2
- net D_OUT_E1: now also U?.10; no longer U?.2
- net D_OUT_E2: now also U?.10; no longer U?.2
- net D_OUT_F1: now also U?.12; no longer U?.2
- net D_OUT_F2: now also U?.12; no longer U?.2
- net GND_D: now also U?.7 (GND), U?.7 (GND), U?.7 (GND)
- net 5V_VCC renamed VCC
- net VCC: now also U?.14 (VCC), U?.14 (VCC), U?.14 (VCC)
- new net: U?.12, U?.13, U?.13
- new net: U?.3, U?.3, U?.4
- new net: U?.10, U?.11, U?.11
- new net: U?.5, U?.5, U?.6
- new net: U?.8, U?.9, U?.9
Changed lines of the file:
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@@
     (effects (font (size 1.27 1.27)) (justify left))
   )
-  (hierarchical_label "5V_VCC" (shape input) (at 234.95 33.02 90)
+  (hierarchical_label "VCC" (shape input) (at 234.95 33.02 90)
     (effects (font (size 1.27 1.27)) (justify left))
   )
@@
     (pin "2")
   )
-  (symbol (lib_id "74xx:74LS07") (at 144.78 156.21 0) (unit 1)
+  (symbol (lib_id "74xx:74LS07") (at 144.78 156.21 0) (unit 6)
     (in_bom yes) (on_board yes) (fields_autoplaced)
     (property "Reference" "U?" (id 0) (at 144.78 147.32 0))
@@
       (effects (font (size 1.27 1.27)) hide)
     )
-    (pin "1")
-    (pin "2")
+    (pin "12")
+    (pin "13")
   )
   (symbol (lib_id "74xx:74LS07") (at 144.78 41.91 0) (unit 1)
@@
     (pin "2")
   )
-  (symbol (lib_id "74xx:74LS07") (at 209.55 50.8 0) (unit 1)
+  (symbol (lib_id "74xx:74LS07") (at 209.55 50.8 0) (unit 7)
     (in_bom yes) (on_board yes) (fields_autoplaced)
     (property "Reference" "U?" (id 0) (at 215.9 49.5299 0)
@@
       (effects (font (size 1.27 1.27)) hide)
     )
-    (pin "1")
-    (pin "2")
-  )
-  (symbol (lib_id "4xxx:4069") (at 58.42 177.8 0) (unit 1)
+    (pin "14")
+    (pin "7")
+  )
+  (symbol (lib_id "4xxx:4069") (at 58.42 177.8 0) (unit 6)
     (in_bom yes) (on_board yes) (fields_autoplaced)
     (property "Reference" "U?" (id 0) (at 58.42 168.91 0))
@@
       (effects (font (size 1.27 1.27)) hide)
     )
-    (pin "1")
-    (pin "2")
-  )
-  (symbol (lib_id "74xx:74LS07") (at 144.78 64.77 0) (unit 1)
+    (pin "12")
+    (pin "13")
+  )
+  (symbol (lib_id "74xx:74LS07") (at 144.78 64.77 0) (unit 2)
     (in_bom yes) (on_board yes) (fields_autoplaced)
     (property "Reference" "U?" (id 0) (at 144.78 55.88 0))
@@
       (effects (font (size 1.27 1.27)) hide)
     )
-    (pin "1")
-    (pin "2")
-  )
-  (symbol (lib_id "74xx:74LS07") (at 107.95 133.35 0) (unit 1)
+    (pin "3")
+    (pin "4")
+  )
+  (symbol (lib_id "74xx:74LS07") (at 107.95 133.35 0) (unit 5)
     (in_bom yes) (on_board yes) (fields_autoplaced)
     (property "Reference" "U?" (id 0) (at 107.95 124.46 0))
@@
       (effects (font (size 1.27 1.27)) hide)
     )
-    (pin "1")
-    (pin "2")
-  )
-  (symbol (lib_id "74xx:74LS07") (at 133.35 123.19 0) (unit 1)
+    (pin "10")
+    (pin "11")
+  )
+  (symbol (lib_id "74xx:74LS07") (at 133.35 123.19 0) (unit 5)
     (in_bom yes) (on_board yes) (fields_autoplaced)
     (property "Reference" "U?" (id 0) (at 133.35 114.3 0))
@@
       (effects (font (size 1.27 1.27)) hide)
     )
-    (pin "1")
-    (pin "2")
+    (pin "10")
+    (pin "11")
   )
   (symbol (lib_id "74xx:74LS07") (at 133.35 31.75 0) (unit 1)
@@
     (pin "2")
   )
-  (symbol (lib_id "4xxx:4081") (at 40.64 193.04 0) (unit 1)
+  (symbol (lib_id "4xxx:4081") (at 40.64 193.04 0) (unit 4)
     (in_bom yes) (on_board yes)
     (property "Reference" "U?" (id 0) (at 39.37 185.42 0))
@@
       (effects (font (size 1.27 1.27)) hide)
     )
-    (pin "1")
-    (pin "2")
-    (pin "3")
-  )
-  (symbol (lib_id "4xxx:4069") (at 40.64 177.8 0) (unit 1)
+    (pin "11")
+    (pin "12")
+    (pin "13")
+  )
+  (symbol (lib_id "4xxx:4069") (at 40.64 177.8 0) (unit 5)
     (in_bom yes) (on_board yes) (fields_autoplaced)
     (property "Reference" "U?" (id 0) (at 40.64 168.91 0))
@@
       (effects (font (size 1.27 1.27)) hide)
     )
-    (pin "1")
-    (pin "2")
-  )
-  (symbol (lib_id "74xx:74HC86") (at 24.13 193.04 0) (unit 1)
+    (pin "10")
+    (pin "11")
+  )
+  (symbol (lib_id "74xx:74HC86") (at 24.13 193.04 0) (unit 4)
     (in_bom yes) (on_board yes) (fields_autoplaced)
     (property "Reference" "U?" (id 0) (at 23.8252 184.15 0))
@@
       (effects (font (size 1.27 1.27)) hide)
     )
-    (pin "1")
-    (pin "2")
-    (pin "3")
+    (pin "11")
+    (pin "12")
+    (pin "13")
   )
   (symbol (lib_id "000_Capacitor_Film_Immo:cap_film_0805") (at 256.54 50.8 0) (unit 1)
@@
     (pin "2")
   )
-  (symbol (lib_id "74xx:74LS07") (at 144.78 133.35 0) (unit 1)
+  (symbol (lib_id "74xx:74LS07") (at 144.78 133.35 0) (unit 5)
     (in_bom yes) (on_board yes) (fields_autoplaced)
     (property "Reference" "U?" (id 0) (at 144.78 124.46 0))
@@
       (effects (font (size 1.27 1.27)) hide)
     )
-    (pin "1")
-    (pin "2")
-  )
-  (symbol (lib_id "74xx:74LS07") (at 144.78 87.63 0) (unit 1)
+    (pin "10")
+    (pin "11")
+  )
+  (symbol (lib_id "74xx:74LS07") (at 144.78 87.63 0) (unit 3)
     (in_bom yes) (on_board yes) (fields_autoplaced)
     (property "Reference" "U?" (id 0) (at 144.78 78.74 0))
@@
       (effects (font (size 1.27 1.27)) hide)
     )
-    (pin "1")
-    (pin "2")
-  )
-  (symbol (lib_id "74xx:74LS07") (at 107.95 110.49 0) (unit 1)
+    (pin "5")
+    (pin "6")
+  )
+  (symbol (lib_id "74xx:74LS07") (at 107.95 110.49 0) (unit 4)
     (in_bom yes) (on_board yes) (fields_autoplaced)
     (property "Reference" "U?" (id 0) (at 107.95 101.6 0))
@@
       (effects (font (size 1.27 1.27)) hide)
     )
-    (pin "1")
-    (pin "2")
-  )
-  (symbol (lib_id "74xx:74LS07") (at 107.95 64.77 0) (unit 1)
+    (pin "8")
+    (pin "9")
+  )
+  (symbol (lib_id "74xx:74LS07") (at 107.95 64.77 0) (unit 2)
     (in_bom yes) (on_board yes)
     (property "Reference" "U?" (id 0) (at 107.95 55.88 0))
@@
       (effects (font (size 1.27 1.27)) hide)
     )
-    (pin "1")
-    (pin "2")
-  )
-  (symbol (lib_id "74xx:74LS07") (at 133.35 100.33 0) (unit 1)
+    (pin "3")
+    (pin "4")
+  )
+  (symbol (lib_id "74xx:74LS07") (at 133.35 100.33 0) (unit 4)
     (in_bom yes) (on_board yes) (fields_autoplaced)
     (property "Reference" "U?" (id 0) (at 133.35 91.44 0))
@@
       (effects (font (size 1.27 1.27)) hide)
     )
-    (pin "1")
-    (pin "2")
-  )
-  (symbol (lib_id "74xx:74LS07") (at 133.35 54.61 0) (unit 1)
+    (pin "8")
+    (pin "9")
+  )
+  (symbol (lib_id "74xx:74LS07") (at 133.35 54.61 0) (unit 2)
     (in_bom yes) (on_board yes)
     (property "Reference" "U?" (id 0) (at 133.35 45.72 0))
@@
       (effects (font (size 1.27 1.27)) hide)
     )
-    (pin "1")
-    (pin "2")
-  )
-  (symbol (lib_id "74xx:74LS07") (at 265.43 50.8 0) (unit 1)
+    (pin "3")
+    (pin "4")
+  )
+  (symbol (lib_id "74xx:74LS07") (at 265.43 50.8 0) (unit 7)
     (in_bom yes) (on_board yes) (fields_autoplaced)
     (property "Reference" "U?" (id 0) (at 271.78 49.5299 0)
@@
       (effects (font (size 1.27 1.27)) hide)
     )
-    (pin "1")
-    (pin "2")
-  )
-  (symbol (lib_id "74xx:74LS07") (at 107.95 156.21 0) (unit 1)
+    (pin "14")
+    (pin "7")
+  )
+  (symbol (lib_id "74xx:74LS07") (at 107.95 156.21 0) (unit 6)
     (in_bom yes) (on_board yes) (fields_autoplaced)
     (property "Reference" "U?" (id 0) (at 107.95 147.32 0))
@@
       (effects (font (size 1.27 1.27)) hide)
     )
-    (pin "1")
-    (pin "2")
-  )
-  (symbol (lib_id "74xx:74LS07") (at 133.35 146.05 0) (unit 1)
+    (pin "12")
+    (pin "13")
+  )
+  (symbol (lib_id "74xx:74LS07") (at 133.35 146.05 0) (unit 6)
     (in_bom yes) (on_board yes) (fields_autoplaced)
     (property "Reference" "U?" (id 0) (at 133.35 137.16 0))
@@
       (effects (font (size 1.27 1.27)) hide)
     )
-    (pin "1")
-    (pin "2")
-  )
-  (symbol (lib_id "4xxx:4069") (at 22.86 177.8 0) (unit 1)
+    (pin "12")
+    (pin "13")
+  )
+  (symbol (lib_id "4xxx:4069") (at 22.86 177.8 0) (unit 4)
     (in_bom yes) (on_board yes) (fields_autoplaced)
     (property "Reference" "U?" (id 0) (at 22.86 168.91 0))
@@
       (effects (font (size 1.27 1.27)) hide)
     )
-    (pin "1")
-    (pin "2")
-  )
-  (symbol (lib_id "4xxx:4081") (at 58.42 193.04 0) (unit 1)
+    (pin "8")
+    (pin "9")
+  )
+  (symbol (lib_id "4xxx:4081") (at 58.42 193.04 0) (unit 3)
     (in_bom yes) (on_board yes) (fields_autoplaced)
     (property "Reference" "U?" (id 0) (at 58.42 184.15 0))
@@
       (effects (font (size 1.27 1.27)) hide)
     )
-    (pin "1")
-    (pin "2")
-    (pin "3")
-  )
-  (symbol (lib_id "74xx:74LS07") (at 133.35 77.47 0) (unit 1)
+    (pin "10")
+    (pin "8")
+    (pin "9")
+  )
+  (symbol (lib_id "74xx:74LS07") (at 133.35 77.47 0) (unit 3)
     (in_bom yes) (on_board yes) (fields_autoplaced)
     (property "Reference" "U?" (id 0) (at 133.35 68.58 0))
@@
       (effects (font (size 1.27 1.27)) hide)
     )
-    (pin "1")
-    (pin "2")
-  )
-  (symbol (lib_id "74xx:74LS07") (at 144.78 110.49 0) (unit 1)
+    (pin "5")
+    (pin "6")
+  )
+  (symbol (lib_id "74xx:74LS07") (at 144.78 110.49 0) (unit 4)
     (in_bom yes) (on_board yes) (fields_autoplaced)
     (property "Reference" "U?" (id 0) (at 144.78 101.6 0))
@@
       (effects (font (size 1.27 1.27)) hide)
     )
-    (pin "1")
-    (pin "2")
-  )
-  (symbol (lib_id "74xx:74LS07") (at 237.49 50.8 0) (unit 1)
+    (pin "8")
+    (pin "9")
+  )
+  (symbol (lib_id "74xx:74LS07") (at 237.49 50.8 0) (unit 7)
     (in_bom yes) (on_board yes)
     (property "Reference" "U?" (id 0) (at 243.84 49.5299 0)
@@
       (effects (font (size 1.27 1.27)) hide)
     )
-    (pin "1")
-    (pin "2")
-  )
-  (symbol (lib_id "74xx:74LS07") (at 107.95 87.63 0) (unit 1)
+    (pin "14")
+    (pin "7")
+  )
+  (symbol (lib_id "74xx:74LS07") (at 107.95 87.63 0) (unit 3)
     (in_bom yes) (on_board yes) (fields_autoplaced)
     (property "Reference" "U?" (id 0) (at 107.95 78.74 0))
@@
       (effects (font (size 1.27 1.27)) hide)
     )
-    (pin "1")
-    (pin "2")
+    (pin "5")
+    (pin "6")
   )
 )

Commit message: Circuit Design 85-90% complete
Other:
- note added: "Secondary purpose of the buffers, to stop student MCU from applying voltages to supervisor MCU either inadvertently or deliberatly."
Changed lines of the file:
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@@
+    (effects (font (size 1.27 1.27)) (justify left bottom))
+  )
+  (text "Secondary purpose of the buffers,\nto stop student MCU from applying voltages to supervisor \nMCU either inadvertently or deliberatly."
+    (at 196.85 91.44 0)
     (effects (font (size 1.27 1.27)) (justify left bottom))
   )

Commit message: V1.0 Circuit Design Complete
Parts:
- removed C? (x3): 100n, Capacitor_SMD:C_0805_2012Metric_Pad1.18x1.45mm_HandSolder, symbol 000_Capacitor_Film_Immo:cap_film_0805
- removed U? (x3): 4069, symbol 4xxx:4069
- removed U? (x2): 4081, symbol 4xxx:4081
- removed U?: 74HC86, symbol 74xx:74HC86
- added C38, C39, C40: 100n, Capacitor_SMD:C_0805_2012Metric_Pad1.18x1.45mm_HandSolder, symbol 000_Capacitor_Film_Immo:cap_film_0805
- gave numbers to parts that had none: 3
Connections:
- net GND_D: now also C38.2, C39.2, C40.2
- net VCC: now also C38.1, C39.1, C40.1
Other:
- note removed: "Spare Gates Square"

Commit message: Schematic reviewed
Parts:
- U20, U21, U22: footprint (none) -> Package_DIP:SMDIP-14_W9.53mm

Commit message: mbncmvbc,
Parts:
- added R26, R27, R28, R29, R30, R31: 1k, Resistor_SMD:R_0805_2012Metric_Pad1.20x1.40mm_HandSolder, symbol 000_Resistors_Immo:Resistor_0805
Connections:
- net D_OUT_A2: now also R27.1; no longer U22.2
- net D_OUT_B2: now also R26.1; no longer U22.4
- net D_OUT_C2: now also R28.1; no longer U22.6
- net D_OUT_D2: now also R29.1; no longer U22.8
- net D_OUT_E2: now also R31.1; no longer U22.10
- net D_OUT_F2: now also R30.1; no longer U22.12
- new net: R31.2, U22.10
- new net: R30.2, U22.12
- new net: R27.2, U22.2
- new net: R26.2, U22.4
- new net: R28.2, U22.6
- new net: R29.2, U22.8
