File: RemoteLabs_supervisor_PCB/digital_signal_buffers.kicad_sch (KiCad schematic)
At the start: 12 parts, among them U20 74LS07, U21 74LS07, U22 74LS07

Commit message: Footprint associations complete
Parts:
- U20, U21, U22: footprint Package_DIP:SMDIP-14_W9.53mm -> Package_SO:SOIC-14_3.9x8.7mm_P1.27mm
Changed lines of the file:
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@@
     (property "Reference" "U22" (id 0) (at 144.78 147.32 0))
     (property "Value" "74LS07" (id 1) (at 144.78 149.86 0))
-    (property "Footprint" "Package_DIP:SMDIP-14_W9.53mm" (id 2) (at 144.78 156.21 0)
+    (property "Footprint" "Package_SO:SOIC-14_3.9x8.7mm_P1.27mm" (id 2) (at 144.78 156.21 0)
       (effects (font (size 1.27 1.27)) hide)
     )
@@
     (property "Reference" "U22" (id 0) (at 144.78 33.02 0))
     (property "Value" "74LS07" (id 1) (at 144.78 35.56 0))
-    (property "Footprint" "Package_DIP:SMDIP-14_W9.53mm" (id 2) (at 144.78 41.91 0)
+    (property "Footprint" "Package_SO:SOIC-14_3.9x8.7mm_P1.27mm" (id 2) (at 144.78 41.91 0)
       (effects (font (size 1.27 1.27)) hide)
     )
@@
     (property "Reference" "U20" (id 0) (at 107.95 33.02 0))
     (property "Value" "74LS07" (id 1) (at 107.95 35.56 0))
-    (property "Footprint" "Package_DIP:SMDIP-14_W9.53mm" (id 2) (at 107.95 41.91 0)
+    (property "Footprint" "Package_SO:SOIC-14_3.9x8.7mm_P1.27mm" (id 2) (at 107.95 41.91 0)
       (effects (font (size 1.27 1.27)) hide)
     )
@@
       (effects (font (size 1.27 1.27)) (justify left))
     )
-    (property "Footprint" "Package_DIP:SMDIP-14_W9.53mm" (id 2) (at 209.55 50.8 0)
+    (property "Footprint" "Package_SO:SOIC-14_3.9x8.7mm_P1.27mm" (id 2) (at 209.55 50.8 0)
       (effects (font (size 1.27 1.27)) hide)
     )
@@
     (property "Reference" "U22" (id 0) (at 144.78 55.88 0))
     (property "Value" "74LS07" (id 1) (at 144.78 58.42 0))
-    (property "Footprint" "Package_DIP:SMDIP-14_W9.53mm" (id 2) (at 144.78 64.77 0)
+    (property "Footprint" "Package_SO:SOIC-14_3.9x8.7mm_P1.27mm" (id 2) (at 144.78 64.77 0)
       (effects (font (size 1.27 1.27)) hide)
     )
@@
     (property "Reference" "U20" (id 0) (at 107.95 124.46 0))
     (property "Value" "74LS07" (id 1) (at 107.95 127 0))
-    (property "Footprint" "Package_DIP:SMDIP-14_W9.53mm" (id 2) (at 107.95 133.35 0)
+    (property "Footprint" "Package_SO:SOIC-14_3.9x8.7mm_P1.27mm" (id 2) (at 107.95 133.35 0)
       (effects (font (size 1.27 1.27)) hide)
     )
@@
     (property "Reference" "U21" (id 0) (at 133.35 114.3 0))
     (property "Value" "74LS07" (id 1) (at 133.35 116.84 0))
-    (property "Footprint" "Package_DIP:SMDIP-14_W9.53mm" (id 2) (at 133.35 123.19 0)
+    (property "Footprint" "Package_SO:SOIC-14_3.9x8.7mm_P1.27mm" (id 2) (at 133.35 123.19 0)
       (effects (font (size 1.27 1.27)) hide)
     )
@@
     (property "Reference" "U21" (id 0) (at 133.35 22.86 0))
     (property "Value" "74LS07" (id 1) (at 133.35 25.4 0))
-    (property "Footprint" "Package_DIP:SMDIP-14_W9.53mm" (id 2) (at 133.35 31.75 0)
+    (property "Footprint" "Package_SO:SOIC-14_3.9x8.7mm_P1.27mm" (id 2) (at 133.35 31.75 0)
       (effects (font (size 1.27 1.27)) hide)
     )
@@
     (property "Reference" "U22" (id 0) (at 144.78 124.46 0))
     (property "Value" "74LS07" (id 1) (at 144.78 127 0))
-    (property "Footprint" "Package_DIP:SMDIP-14_W9.53mm" (id 2) (at 144.78 133.35 0)
+    (property "Footprint" "Package_SO:SOIC-14_3.9x8.7mm_P1.27mm" (id 2) (at 144.78 133.35 0)
       (effects (font (size 1.27 1.27)) hide)
     )
@@
     (property "Reference" "U22" (id 0) (at 144.78 78.74 0))
     (property "Value" "74LS07" (id 1) (at 144.78 81.28 0))
-    (property "Footprint" "Package_DIP:SMDIP-14_W9.53mm" (id 2) (at 144.78 87.63 0)
+    (property "Footprint" "Package_SO:SOIC-14_3.9x8.7mm_P1.27mm" (id 2) (at 144.78 87.63 0)
       (effects (font (size 1.27 1.27)) hide)
     )
@@
     (property "Reference" "U20" (id 0) (at 107.95 101.6 0))
     (property "Value" "74LS07" (id 1) (at 107.95 104.14 0))
-    (property "Footprint" "Package_DIP:SMDIP-14_W9.53mm" (id 2) (at 107.95 110.49 0)
+    (property "Footprint" "Package_SO:SOIC-14_3.9x8.7mm_P1.27mm" (id 2) (at 107.95 110.49 0)
       (effects (font (size 1.27 1.27)) hide)
     )
@@
     (property "Reference" "U20" (id 0) (at 107.95 55.88 0))
     (property "Value" "74LS07" (id 1) (at 107.95 58.42 0))
-    (property "Footprint" "Package_DIP:SMDIP-14_W9.53mm" (id 2) (at 107.95 64.77 0)
+    (property "Footprint" "Package_SO:SOIC-14_3.9x8.7mm_P1.27mm" (id 2) (at 107.95 64.77 0)
       (effects (font (size 1.27 1.27)) hide)
     )
@@
     (property "Reference" "U21" (id 0) (at 133.35 91.44 0))
     (property "Value" "74LS07" (id 1) (at 133.35 93.98 0))
-    (property "Footprint" "Package_DIP:SMDIP-14_W9.53mm" (id 2) (at 133.35 100.33 0)
+    (property "Footprint" "Package_SO:SOIC-14_3.9x8.7mm_P1.27mm" (id 2) (at 133.35 100.33 0)
       (effects (font (size 1.27 1.27)) hide)
     )
@@
     (property "Reference" "U21" (id 0) (at 133.35 45.72 0))
     (property "Value" "74LS07" (id 1) (at 133.35 48.26 0))
-    (property "Footprint" "Package_DIP:SMDIP-14_W9.53mm" (id 2) (at 133.35 54.61 0)
+    (property "Footprint" "Package_SO:SOIC-14_3.9x8.7mm_P1.27mm" (id 2) (at 133.35 54.61 0)
       (effects (font (size 1.27 1.27)) hide)
     )
@@
       (effects (font (size 1.27 1.27)) (justify left))
     )
-    (property "Footprint" "Package_DIP:SMDIP-14_W9.53mm" (id 2) (at 265.43 50.8 0)
+    (property "Footprint" "Package_SO:SOIC-14_3.9x8.7mm_P1.27mm" (id 2) (at 265.43 50.8 0)
       (effects (font (size 1.27 1.27)) hide)
     )
@@
     (property "Reference" "U20" (id 0) (at 107.95 147.32 0))
     (property "Value" "74LS07" (id 1) (at 107.95 149.86 0))
-    (property "Footprint" "Package_DIP:SMDIP-14_W9.53mm" (id 2) (at 107.95 156.21 0)
+    (property "Footprint" "Package_SO:SOIC-14_3.9x8.7mm_P1.27mm" (id 2) (at 107.95 156.21 0)
       (effects (font (size 1.27 1.27)) hide)
     )
@@
     (property "Reference" "U21" (id 0) (at 133.35 137.16 0))
     (property "Value" "74LS07" (id 1) (at 133.35 139.7 0))
-    (property "Footprint" "Package_DIP:SMDIP-14_W9.53mm" (id 2) (at 133.35 146.05 0)
+    (property "Footprint" "Package_SO:SOIC-14_3.9x8.7mm_P1.27mm" (id 2) (at 133.35 146.05 0)
       (effects (font (size 1.27 1.27)) hide)
     )
@@
     (property "Reference" "U21" (id 0) (at 133.35 68.58 0))
     (property "Value" "74LS07" (id 1) (at 133.35 71.12 0))
-    (property "Footprint" "Package_DIP:SMDIP-14_W9.53mm" (id 2) (at 133.35 77.47 0)
+    (property "Footprint" "Package_SO:SOIC-14_3.9x8.7mm_P1.27mm" (id 2) (at 133.35 77.47 0)
       (effects (font (size 1.27 1.27)) hide)
     )
@@
     (property "Reference" "U22" (id 0) (at 144.78 101.6 0))
     (property "Value" "74LS07" (id 1) (at 144.78 104.14 0))
-    (property "Footprint" "Package_DIP:SMDIP-14_W9.53mm" (id 2) (at 144.78 110.49 0)
+    (property "Footprint" "Package_SO:SOIC-14_3.9x8.7mm_P1.27mm" (id 2) (at 144.78 110.49 0)
       (effects (font (size 1.27 1.27)) hide)
     )
@@
       (effects (font (size 1.27 1.27)) (justify left))
     )
-    (property "Footprint" "Package_DIP:SMDIP-14_W9.53mm" (id 2) (at 237.49 50.8 0)
+    (property "Footprint" "Package_SO:SOIC-14_3.9x8.7mm_P1.27mm" (id 2) (at 237.49 50.8 0)
       (effects (font (size 1.27 1.27)) hide)
     )
@@
     (property "Reference" "U20" (id 0) (at 107.95 78.74 0))
     (property "Value" "74LS07" (id 1) (at 107.95 81.28 0))
-    (property "Footprint" "Package_DIP:SMDIP-14_W9.53mm" (id 2) (at 107.95 87.63 0)
-      (effects (font (size 1.27 1.27)) hide)
-    )
+    (property "Footprint" "Package_SO:SOIC-14_3.9x8.7mm_P1.27mm" (id 2) (at 107.95 87.63 0)
+      (effects (font (size 1.27 1.27)) hide)
+    )
