File: RemoteLabs_supervisor_PCB/output_logic.kicad_sch (KiCad schematic)
At the start: 37 parts

Commit message: Schematric work
Parts:
- added C? (x7): 100n, Capacitor_SMD:C_0805_2012Metric_Pad1.18x1.45mm_HandSolder, symbol 000_Capacitor_Film_Immo:cap_film_0805
Connections:
- net PLACEHOLDER-> LOGIC HIGH is gone; now on an unnamed net: U?.13
- net 5V_VCC: now reaches U?.14 (VCC)
- net 5V_VCC: now also U?.14 (VCC), U?.14 (VDD), U?.14 (VDD), U?.14 (VDD), U?.14 (VDD), U?.14 (VDD), C?.1, C?.1, C?.1, C?.1, C?.1, C?.1, C?.1
- net GND_D: now reaches U?.7 (GND)
- net GND_D: now also U?.7 (GND), U?.7 (VSS), U?.7 (VSS), U?.7 (VSS), U?.7 (VSS), U?.7 (VSS), C?.2, C?.2, C?.2, C?.2, C?.2, C?.2, C?.2
- net at U?.9: now also U?.11, U?.12, U?.12, U?.13, U?.13, U?.8, U?.9
- no-connect marks 0 -> 6
Other:
- note added: "Decoupling Caps"
- note added: "Spare Gates"
- note removed: "Aim: To propigate raw signals from sensors to both MCUs, to enable bare metal programming experience, but allow supervisor MCU to monitor and track hardware configurations."
- note removed: "Analog Buffers for Analog Sensors"
- note removed: "Digital Buffers for Digital Sensors"
- note removed: "Hardware Inputs"
- moved on the sheet: U?A, U?B, U?C, U?D, U?E, U?F, U?G

Commit message: adding test sketch
Connections:
- net 5V_VCC renamed VCC
Changed lines of the file:
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@@
     (effects (font (size 1.27 1.27)) (justify right))
   )
-  (hierarchical_label "5V_VCC" (shape input) (at 229.87 104.14 90)
+  (hierarchical_label "VCC" (shape input) (at 229.87 104.14 90)
     (effects (font (size 1.27 1.27)) (justify left))
   )
@@
     (effects (font (size 1.27 1.27)) (justify right))
   )
-  (hierarchical_label "5V_VCC" (shape input) (at 229.87 36.83 90)
+  (hierarchical_label "VCC" (shape input) (at 229.87 36.83 90)
     (effects (font (size 1.27 1.27)) (justify left))
   )

Commit message: lunchtime backup
Parts:
- removed U? (x4): 74HC86, symbol 74xx:74HC86
- removed U? (x4): 4081, symbol 4xxx:4081
Connections:
- net STUDENT_M_INH_2 is gone; now on an unnamed net: U?.12
- net STUDENT_M_IN_2 is gone; now on an unnamed net: U?.8
- net OUT_M_IN_1: now also U?.10
- net OUT_M_IN_2: now also U?.11
- net STUDENT_M_ENABLE: no longer U?.13, U?.6, U?.9
- net at U?.2: now also U?.6
- net STUDENT_M_INH_1 renamed SUPERVISOR_M_PWM_IN
- net STUDENT_M_IN_1 renamed STUDENT_M_PWM_IN
- new net MOTOR_DIR_A: U?.9
- new net MOTOR_DIR_B: U?.13
Other:
- note added: "PWM is assigned to either Motor driver board IN_1 or IN_2 based on 2 direction pins sent by Supervisor MCU. This would allow supervisor to drive both pins high, leading to SHOOT THROUGH. Student has the same inputs to motor driver, but direction pins are spoofed through the supervisor, so supervisor can block illegal logic (1,1) and alert the student that they have tried to do something that coul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"
- note added: "Supervisor also controls whether PWM control is enabled from student MCU"
- moved on the sheet: U?A, U?B, U?C, U?D

Commit message: Circuit Design 85-90% complete
Parts:
- added U? (x3): 74HC86, symbol 74xx:74HC86
- added U? (x4): 4081, symbol 4xxx:4081
- added U?: 4069, symbol 4xxx:4069
Connections:
- net STUDENT_STEP_ENABLE: now also U?.2
- net at U?.13, U?.6, U?.9: now also U?.2
- net at U?.8: now also U?.12, U?.11; no longer U?.3
- net at U?.2, U?.6: now also U?.13
- net at U?.10: now also U?.12
- net OUT_M_ENABLE: now reaches U?.11
- net at U?.4: now also U?.13; no longer U?.12
- net at U?.11: now also U?.13
- net OUT_M_IN_1 renamed MOTOR_OUT_1
- net OUT_M_IN_2 renamed MOTOR_OUT_2
- net STEP_OUT renamed STEPP_STEP_OUT
- net STUDENT_M_ENABLE renamed STUDENT_MOTOR_ENABLE
- net STUDENT_MOTOR_ENABLE: now also U?.9
- net STUDENT_M_PWM_IN renamed STUDENT_MOTOR_PWM
- net SUPERVISOR_M_PWM_IN renamed SUPERVISOR_MOTOR_PWM
- new net: U?.10, U?.3 (x2)
- new net: U?.3, U?.9 (x2)
- new net: U?.2, U?.6
- new net: U?.11, U?.13, U?.9
- new net: U?.12, U?.3
- new net PIXEL_DATA_OUT: U?.8
- new net STEP_EN_OUT: U?.8
- new net STUDENT_MOTOR_EN: U?.8
- new net STUDENT_PIXEL_DATA: U?.1
- new net STUDENT_PIXEL_ENABLE: U?.2, U?.5
- new net STUDENT_STEP_EN: U?.1
- new net SUPERVISOR_MOTOR_EN: U?.12
- new net SUPERVISOR_PIXEL_DATA: U?.1
- new net SUPERVISOR_STEP_EN: U?.1
- no-connect marks 6 -> 2
Other:
- note added: "Pixel Output"
- moved on the sheet: U?A, U?B, U?C, U?D, U?E, U?F

Commit message: V1.0 Circuit Design Complete
Parts:
- removed U? (x2): 4069, symbol 4xxx:4069
- removed U?: 74HC86, symbol 74xx:74HC86
- removed U? (x2): 4081, symbol 4xxx:4081
- added unit 3 of U12
- added unit 4 of U12
- added unit 3 of U14
- added unit 4 of U14
- added unit 7 of U8
- gave numbers to parts that had none: 14
Connections:
- net DIRECTION_OUT: now also U13.8; no longer U13.6
- net GND_D: now also U8.11, U8.13, U8.9, U14.12, U14.13, U8.7 (VSS)
- net MOTOR_DIR_A: now also U11.2; no longer U11.9
- net MOTOR_DIR_B: now also U11.6; no longer U11.13
- net MOTOR_OUT_1: now also U11.3; no longer U11.10
- net MOTOR_OUT_2: now also U11.4; no longer U11.11
- net OUT_M_ENABLE: now also U13.6; no longer U13.11
- net PIXEL_DATA_OUT: now also U14.6; no longer U14.8
- net STEPP_STEP_OUT: now also U13.11; no longer U13.8
- net STEP_EN_OUT: now also U14.3; no longer U14.8
- net STUDENT_STEP_EN: now also U11.8; no longer U11.1
- net STUDENT_STEP_ENABLE: now also U11.9, U8.3, U12.9; no longer U11.2, U8.5
- net SUPERVISOR_PIXEL_DATA: now also U12.5; no longer U12.1
- net SUPERVISOR_STEP_EN: now also U11.12; no longer U11.1
- net VCC: now also U8.14 (VDD)
- net at U10.10: now also U13.10; no longer U13.5
- net at U10.13, U10.9: now also U11.13, U8.4, U12.13; no longer U11.2, U8.6
- net at U12.3: now also U14.4; no longer U14.9
- net at U8.6: now also U12.6; no longer U12.2
- net at U10.4: now also U13.12; no longer U13.9
- net at U9.3: now also U13.1; no longer U13.12
- net at U9.10: now also U13.4; no longer U13.12
- net at U10.3: now also U13.9; no longer U13.4
- net at U9.11: now also U13.5; no longer U13.13
- net at U10.11: now also U13.13; no longer U13.10
- net at U9.4: now also U13.2; no longer U13.13
- new net: U12.4, U14.5
- new net: U11.1, U11.5, U13.3
- new net: U12.11, U14.10
- new net: U12.10, U14.9
- new net: U11.11, U14.2
- new net: U11.10, U14.1
- new net STEP_RST_OUT: U14.8
- new net STUDENT_STEP_RST: U12.8
- new net SUPERVISOR_STEP_RST: U12.12
- no-connect marks 2 -> 4
Other:
- note removed: "Servo Motor Outputs"
- moved on the sheet: C24, C25, C26, C27, C28, C29, C30, U10A, U10B, U10C, U10D, U10E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

Commit message: Schematic reviewed
Parts:
- U10, U11, U12, U13, U14, U8, U9: footprint (none) -> Package_DIP:SMDIP-14_W9.53mm
Connections:
- net STUDENT_MOTOR_ENABLE renamed MCU_MOTOR_SELECT
- net STUDENT_PIXEL_ENABLE renamed MCU_PIXEL_SELECT
- net STUDENT_STEP_ENABLE renamed MCU_STEP_SELECT
