File: RemoteLabs_supervisor_PCB/output_logic.kicad_sch (KiCad schematic)
At the start: 14 parts, among them U10 4081, U11 4081, U12 4081, U13 74HC86, U14 74HC86, U8 4069, U9 4081

Commit message: Footprint associations complete
Parts:
- U10, U11, U12, U13, U14, U8, U9: footprint Package_DIP:SMDIP-14_W9.53mm -> Package_SO:SOIC-14_3.9x8.7mm_P1.27mm

Commit message: routing board layout 2.0
Parts:
- renumbered U11 to U10, U12 to U10, U10 to U11, U12 to U11, U9 to U12, U14 to U13, U13 to U14, U11 to U9
Connections:
- net DIRECTION_OUT: now also U13.3; no longer U13.8
- net MCU_MOTOR_SELECT: now also U12.6; no longer U12.9
- net MCU_PIXEL_SELECT: now also U12.9; no longer U12.2
- net MCU_STEP_SELECT: now also U10.13; no longer U10.9
- net MOTOR_DIR_B: now also U9.9; no longer U9.6
- net MOTOR_OUT_2: now also U9.10; no longer U9.4
- net PIXEL_DATA_OUT: now also U14.8; no longer U14.6
- net STEPP_STEP_OUT: now also U13.6; no longer U13.11
- net STEP_EN_OUT: now also U13.8; no longer U13.3
- net STEP_RST_OUT: now also U13.11; no longer U13.8
- net STUDENT_MOTOR_EN: now also U12.5; no longer U12.8
- net STUDENT_PIXEL_DATA: now also U12.8; no longer U12.1
- net STUDENT_STEP_RST: now also U10.12; no longer U10.8
- net SUPERVISOR_DIRECTION: now also U11.1; no longer U11.8
- net SUPERVISOR_PIXEL_DATA: now also U12.12; no longer U12.5
- net SUPERVISOR_STEP: now also U11.5; no longer U11.12
- net SUPERVISOR_STEP_EN: now also U11.8; no longer U11.12
- net at U8.6: now also U12.13; no longer U12.6
- net at U14.3, U9.1: now also U9.8; no longer U9.5
- net at U11.11: now also U13.13; no longer U13.10
- net at U10.4: now also U13.4; no longer U13.12
- net at U14.4: now also U12.4; no longer U12.10
- net at U10.3: now also U13.1; no longer U13.9
- net at U10.10: now also U13.9; no longer U13.1
- new net: U11.13, U11.2, U11.6, U11.9, U8.4
- new net: U11.3, U13.2
- new net: U12.11, U14.10
- new net: U12.10, U14.9
- new net: U10.11, U13.12
- new net: U11.10, U13.10
- new net: U11.4, U13.5

Commit message: Ahhhhhhhhhhhhhhh
Connections:
- net STEP_EN_OUT renamed STEP_SLP_OUT
- net STUDENT_STEP_EN renamed STUDENT_STEP_SLP
- net SUPERVISOR_STEP_EN renamed SUPERVISOR_STEP_SLP
Changed lines of the file:
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@@
     (effects (font (size 1.27 1.27)) (justify right))
   )
-  (hierarchical_label "STUDENT_STEP_EN" (shape input) (at 37.465 116.84 180)
+  (hierarchical_label "STUDENT_STEP_SLP" (shape input) (at 37.465 116.84 180)
     (effects (font (size 1.27 1.27)) (justify right))
   )
@@
     (effects (font (size 1.27 1.27)) (justify left))
   )
-  (hierarchical_label "SUPERVISOR_STEP_EN" (shape input) (at 99.695 129.54 180)
+  (hierarchical_label "SUPERVISOR_STEP_SLP" (shape input) (at 99.695 129.54 180)
     (effects (font (size 1.27 1.27)) (justify right))
   )
-  (hierarchical_label "STEP_EN_OUT" (shape output) (at 155.575 129.54 0)
+  (hierarchical_label "STEP_SLP_OUT" (shape output) (at 155.575 129.54 0)
     (effects (font (size 1.27 1.27)) (justify left))
   )
