File: RemoteLabs_supervisor_PCB/servo_control.kicad_sch (KiCad schematic)
At the start: 0 parts

Commit message: Schematric work
Parts:
- added J?: Servo_A, symbol Connector:Conn_01x03_Male
- added J?: Servo_B, symbol Connector:Conn_01x03_Male
Connections:
- new net 5V_VCC: J?.2 (Pin_2), J?.2 (Pin_2)
- new net GND_P: J?.3 (Pin_3)
- new net GND_p: J?.3 (Pin_3)
- new net SERVO_A: J?.1 (Pin_1)
- new net SERVO_B: J?.1 (Pin_1)
Changed lines of the file:
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@@
 (kicad_sch (version 20211123) (generator eeschema)
   (paper "A4")
+  (wire (pts (xy 143.51 82.55) (xy 151.13 82.55))
+    (stroke (width 0) (type default) (color 0 0 0 0))
+  )
+  (wire (pts (xy 143.51 87.63) (xy 151.13 87.63))
+    (stroke (width 0) (type default) (color 0 0 0 0))
+  )
+  (wire (pts (xy 143.51 67.31) (xy 151.13 67.31))
+    (stroke (width 0) (type default) (color 0 0 0 0))
+  )
+  (wire (pts (xy 143.51 62.23) (xy 151.13 62.23))
+    (stroke (width 0) (type default) (color 0 0 0 0))
+  )
+  (wire (pts (xy 143.51 64.77) (xy 151.13 64.77))
+    (stroke (width 0) (type default) (color 0 0 0 0))
+  )
+  (wire (pts (xy 143.51 85.09) (xy 151.13 85.09))
+    (stroke (width 0) (type default) (color 0 0 0 0))
+  )
+  (hierarchical_label "GND_P" (shape passive) (at 151.13 67.31 0)
+    (effects (font (size 1.27 1.27)) (justify left))
+  )
+  (hierarchical_label "5V_VCC" (shape input) (at 151.13 64.77 0)
+    (effects (font (size 1.27 1.27)) (justify left))
+  )
+  (hierarchical_label "GND_p" (shape passive) (at 151.13 87.63 0)
+    (effects (font (size 1.27 1.27)) (justify left))
+  )
+  (hierarchical_label "SERVO_A" (shape input) (at 151.13 62.23 0)
+    (effects (font (size 1.27 1.27)) (justify left))
+  )
+  (hierarchical_label "SERVO_B" (shape input) (at 151.13 82.55 0)
+    (effects (font (size 1.27 1.27)) (justify left))
+  )
+  (hierarchical_label "5V_VCC" (shape input) (at 151.13 85.09 0)
+    (effects (font (size 1.27 1.27)) (justify left))
+  )
+  (symbol (lib_id "Connector:Conn_01x03_Male") (at 138.43 64.77 0) (unit 1)
+    (in_bom yes) (on_board yes) (fields_autoplaced)
+    (property "Reference" "J?" (id 0) (at 139.065 57.15 0))
+    (property "Value" "Servo_A" (id 1) (at 139.065 59.69 0))
+    (property "Footprint" "" (id 2) (at 138.43 64.77 0)
+      (effects (font (size 1.27 1.27)) hide)
+    )
+    (property "Datasheet" "~" (id 3) (at 138.43 64.77 0)
+      (effects (font (size 1.27 1.27)) hide)
+    )
+    (pin "1")
+    (pin "2")
+    (pin "3")
+  )
+  (symbol (lib_id "Connector:Conn_01x03_Male") (at 138.43 85.09 0) (unit 1)
+    (in_bom yes) (on_board yes) (fields_autoplaced)
+    (property "Reference" "J?" (id 0) (at 139.065 77.47 0))
+    (property "Value" "Servo_B" (id 1) (at 139.065 80.01 0))
+    (property "Footprint" "" (id 2) (at 138.43 85.09 0)
+      (effects (font (size 1.27 1.27)) hide)
+    )
+    (property "Datasheet" "~" (id 3) (at 138.43 85.09 0)
+      (effects (font (size 1.27 1.27)) hide)
+    )
+    (pin "1")
+    (pin "2")
+    (pin "3")
+  )
 )

Commit message: V1.0 Circuit Design Complete
Parts:
- gave numbers to parts that had none: 2
Changed lines of the file:
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@@
   (symbol (lib_id "Connector:Conn_01x03_Male") (at 138.43 64.77 0) (unit 1)
     (in_bom yes) (on_board yes) (fields_autoplaced)
-    (property "Reference" "J?" (id 0) (at 139.065 57.15 0))
+    (property "Reference" "J20" (id 0) (at 139.065 57.15 0))
     (property "Value" "Servo_A" (id 1) (at 139.065 59.69 0))
     (property "Footprint" "" (id 2) (at 138.43 64.77 0)
@@
   (symbol (lib_id "Connector:Conn_01x03_Male") (at 138.43 85.09 0) (unit 1)
     (in_bom yes) (on_board yes) (fields_autoplaced)
-    (property "Reference" "J?" (id 0) (at 139.065 77.47 0))
+    (property "Reference" "J21" (id 0) (at 139.065 77.47 0))
     (property "Value" "Servo_B" (id 1) (at 139.065 80.01 0))
     (property "Footprint" "" (id 2) (at 138.43 85.09 0)

Commit message: ERC checks run
Connections:
- net GND_p is gone; now on net GND_P: J21.3 (Pin_3)
Changed lines of the file:
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@@
     (effects (font (size 1.27 1.27)) (justify left))
   )
-  (hierarchical_label "GND_p" (shape passive) (at 151.13 87.63 0)
+  (hierarchical_label "GND_P" (shape passive) (at 151.13 87.63 0)
     (effects (font (size 1.27 1.27)) (justify left))
   )

Commit message: Schematic reviewed
Parts:
- J20, J21: footprint (none) -> Connector_PinHeader_2.54mm:PinHeader_1x03_P2.54mm_Vertical
Changed lines of the file:
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@@
     (effects (font (size 1.27 1.27)) (justify left))
   )
-  (symbol (lib_id "Connector:Conn_01x03_Male") (at 138.43 64.77 0) (unit 1)
+  (symbol (lib_name "Conn_01x03_Male_1") (lib_id "Connector:Conn_01x03_Male") (at 138.43 64.77 0) (unit 1)
     (in_bom yes) (on_board yes) (fields_autoplaced)
     (property "Reference" "J20" (id 0) (at 139.065 57.15 0))
     (property "Value" "Servo_A" (id 1) (at 139.065 59.69 0))
-    (property "Footprint" "" (id 2) (at 138.43 64.77 0)
+    (property "Footprint" "Connector_PinHeader_2.54mm:PinHeader_1x03_P2.54mm_Vertical" (id 2) (at 138.43 64.77 0)
       (effects (font (size 1.27 1.27)) hide)
     )
@@
     (property "Reference" "J21" (id 0) (at 139.065 77.47 0))
     (property "Value" "Servo_B" (id 1) (at 139.065 80.01 0))
-    (property "Footprint" "" (id 2) (at 138.43 85.09 0)
+    (property "Footprint" "Connector_PinHeader_2.54mm:PinHeader_1x03_P2.54mm_Vertical" (id 2) (at 138.43 85.09 0)
       (effects (font (size 1.27 1.27)) hide)
     )
