File: RemoteLabs_supervisor_PCB/power_distribution.kicad_sch (KiCad schematic)
At the start: 0 parts

Commit message: update
Parts:
- added D?: BZV55B9V1, Diode_SMD:D_MiniMELF, symbol Diode:BZV55B9V1
- added D?: BZV55B18, Diode_SMD:D_MiniMELF_Handsoldering, symbol Diode:BZV55B18
- added F?: 20A, Fuse:Fuseholder_Cylinder-5x20mm_Stelvio-Kontek_PTF78_Horizontal_Open, symbol 000_Protection_Immo:Fuse
- added J?: XT60_connector_DC_60A_male, Connector_AMASS:AMASS_XT60PW-M, symbol 000_Connectors_Immo:XT60_connector_DC_60A_male
- added Q?: IRF5305_PBF, Package_TO_SOT_SMD:TO-263-2, symbol 000_MOSFET_Immo:IRF5305_PBF
- added R?: 330r, Resistor_SMD:R_0805_2012Metric_Pad1.20x1.40mm_HandSolder, symbol 000_Resistors_Immo:Resistor_0805
- added TP?: 12V_DC, TestPoint:TestPoint_Pad_D1.5mm, symbol Connector:TestPoint
- added U? (x3): LM2596S DC-DC Module, Package_TO_SOT_SMD:TO-263-5_TabPin3, symbol 000_Modules_Immo:LM2596S DC-DC Module
Connections:
- new net: D?.2 (A), Q?.1 (G), R?.1
- new net: F?.2, Q?.2 (D)
- new net 12V_DC: F?.1, J?.2 (V+)
- new net 12V_DC_OUT: D?.1 (K), Q?.3 (S), TP?.1, U?.2 (IN+), U?.2 (IN+), U?.2 (IN+)
- new net 5V_DC_MCU: U?.4 (Out+)
- new net 5V_DC_RPI: U?.4 (Out+)
- new net 5V_DC_SERVO: U?.4 (Out+)
- new net GND_P: J?.1 (V-), R?.2, U?.1 (IN-), U?.1 (IN-), U?.1 (IN-), U?.3 (OUT-), U?.3 (OUT-), U?.3 (OUT-)
- no-connect marks 0 -> 2
Other:
- note added: "Reverse Voltage protection"
- note added: "Using ratio of Vcc to Zener Voltage on previous PCB New Zener voltage ~9v?"

Commit message: adding test sketch
Parts:
- added C? (x2): 10u, Capacitor_SMD:CP_Elec_6.3x5.9, symbol 000_Capacitor_Electrolytic_Immo:22u
- added J?: USB_A, symbol Connector:USB_A
- added TP?: 5V_SERVO, TestPoint:TestPoint_Pad_D1.5mm, symbol Connector:TestPoint
- added TP?: 3V3_MCU, TestPoint:TestPoint_Pad_D1.5mm, symbol Connector:TestPoint
- added TP?: 5V_MCU, TestPoint:TestPoint_Pad_D1.5mm, symbol Connector:TestPoint
- added TP?: 5V_RPI, TestPoint:TestPoint_Pad_D1.5mm, symbol Connector:TestPoint
- added U?: AMS1117-3.3, Package_TO_SOT_SMD:TO-263-5_TabPin3, symbol Regulator_Linear:AMS1117-3.3
Connections:
- net 12V_DC_OUT: now also C?.1, U?.3 (VI)
- net 5V_DC_MCU: now also TP?.1
- net 5V_DC_RPI: now also J?.1 (VBUS), TP?.1
- net 5V_DC_SERVO: now also TP?.1
- net GND_P: now also C?.2, C?.2, J?.4 (GND), J?.5 (Shield), U?.1 (GND)
- new net 3V3_DC_MCU: C?.1, TP?.1, U?.2 (VO)
- no-connect marks 2 -> 4

Commit message: sdf
Parts:
- added J?: Strip Lighting, Connector_PinHeader_1.27mm:PinHeader_1x02_P1.27mm_Vertical, symbol 000_Pin_Headers_Immo:Conn_01x02_Male
Connections:
- net 12V_DC_OUT: now also J?.2 (Pin_2)
- net GND_P: now also J?.1 (Pin_1)
Changed lines of the file:
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@@
   (junction (at 116.84 46.99) (diameter 0) (color 0 0 0 0)
+  )
+  (junction (at 185.42 46.99) (diameter 0) (color 0 0 0 0)
   )
   (junction (at 116.84 83.82) (diameter 0) (color 0 0 0 0)
@@
     (stroke (width 0) (type default) (color 0 0 0 0))
   )
-  (wire (pts (xy 116.84 46.99) (xy 160.02 46.99))
+  (wire (pts (xy 185.42 46.99) (xy 190.5 46.99))
+    (stroke (width 0) (type default) (color 0 0 0 0))
+  )
+  (wire (pts (xy 116.84 46.99) (xy 185.42 46.99))
     (stroke (width 0) (type default) (color 0 0 0 0))
   )
@@
     (stroke (width 0) (type default) (color 0 0 0 0))
   )
+  (wire (pts (xy 190.5 50.8) (xy 185.42 50.8))
+    (stroke (width 0) (type default) (color 0 0 0 0))
+  )
   (wire (pts (xy 152.4 139.7) (xy 152.4 140.97))
     (stroke (width 0) (type default) (color 0 0 0 0))
@@
     (stroke (width 0) (type default) (color 0 0 0 0))
   )
+  (wire (pts (xy 186.69 53.34) (xy 190.5 53.34))
+    (stroke (width 0) (type default) (color 0 0 0 0))
+  )
   (wire (pts (xy 157.48 71.12) (xy 160.02 71.12))
     (stroke (width 0) (type default) (color 0 0 0 0))
@@
   )
   (wire (pts (xy 157.48 106.68) (xy 160.02 106.68))
+    (stroke (width 0) (type default) (color 0 0 0 0))
+  )
+  (wire (pts (xy 185.42 50.8) (xy 185.42 46.99))
     (stroke (width 0) (type default) (color 0 0 0 0))
   )
@@
     (effects (font (size 1.27 1.27)) (justify left))
   )
-  (hierarchical_label "12V_DC_OUT" (shape output) (at 160.02 46.99 0)
+  (hierarchical_label "12V_DC_OUT" (shape output) (at 190.5 46.99 0)
     (effects (font (size 1.27 1.27)) (justify left))
   )
   (hierarchical_label "GND_P" (shape passive) (at 160.02 106.68 0)
     (effects (font (size 1.27 1.27)) (justify left))
+  )
+  (hierarchical_label "GND_P" (shape passive) (at 186.69 53.34 180)
+    (effects (font (size 1.27 1.27)) (justify right))
   )
   (hierarchical_label "5V_DC_MCU" (shape output) (at 190.5 66.04 0)
@@
       (effects (font (size 1.27 1.27)) hide)
     )
+    (pin "1")
+    (pin "2")
+  )
+  (symbol (lib_id "000_Pin_Headers_Immo:Conn_01x02_Male") (at 195.58 53.34 180) (unit 1)
+    (in_bom yes) (on_board yes)
+    (property "Reference" "J?" (id 0) (at 196.85 50.7999 0)
+      (effects (font (size 1.27 1.27)) (justify right))
+    )
+    (property "Value" "Strip Lighting" (id 1) (at 189.23 55.88 0)
+      (effects (font (size 1.27 1.27)) (justify right))
+    )
+    (property "Footprint" "Connector_PinHeader_1.27mm:PinHeader_1x02_P1.27mm_Vertical" (id 2) (at 195.58 53.34 0)
+      (effects (font (size 1.27 1.27)) hide)
+    )
+    (property "Datasheet" "~" (id 3) (at 195.58 53.34 0)
+      (effects (font (size 1.27 1.27)) hide)
+    )

Commit message: V1.0 Circuit Design Complete
Parts:
- removed TP?: 5V_MCU, TestPoint:TestPoint_Pad_D1.5mm, symbol Connector:TestPoint
- removed U?: LM2596S DC-DC Module, Package_TO_SOT_SMD:TO-263-5_TabPin3, symbol 000_Modules_Immo:LM2596S DC-DC Module
- added J6: USB_A, symbol Connector:USB_A
- added JP1: 3V3 PWR SRC, symbol 000_Connectors_Immo:Jumper_3_Bridged12
- gave numbers to parts that had none: 17
Connections:
- net 12V_DC_OUT: no longer C1.1, U3.3 (VI)
- net 5V_DC_RPI: now also J6.1 (VBUS), JP1.1 (A)
- net GND_P: now also J6.4 (GND), J6.5 (Shield)
- new net: C1.1, JP1.2 (C), U3.3 (VI)
- new net USP_PWR_IN: JP1.3 (B)
- no-connect marks 4 -> 6
Other:
- moved on the sheet: C1, C2, J5, TP4, TP5, U2, U3

Commit message: ERC checks run
Changed lines of the file:
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@@
+    (stroke (width 0) (type default) (color 0 0 0 0))
+  )
+  (wire (pts (xy 198.755 104.775) (xy 198.755 107.315))
     (stroke (width 0) (type default) (color 0 0 0 0))
   )
@@
     (stroke (width 0) (type default) (color 0 0 0 0))
   )
-  (wire (pts (xy 186.69 53.34) (xy 190.5 53.34))
+  (wire (pts (xy 186.055 53.34) (xy 190.5 53.34))
     (stroke (width 0) (type default) (color 0 0 0 0))
   )
@@
     (effects (font (size 1.27 1.27)) (justify left))
   )
-  (hierarchical_label "GND_P" (shape passive) (at 186.69 53.34 180)
+  (hierarchical_label "GND_P" (shape passive) (at 186.055 53.34 180)
     (effects (font (size 1.27 1.27)) (justify right))
   )
@@
     (effects (font (size 1.27 1.27)) (justify right))
   )
+  (symbol (lib_id "power:PWR_FLAG") (at 198.755 104.775 0) (unit 1)
+    (in_bom yes) (on_board yes) (fields_autoplaced)
+    (property "Reference" "#FLG0101" (id 0) (at 198.755 102.87 0)
+      (effects (font (size 1.27 1.27)) hide)
+    )
+    (property "Value" "PWR_FLAG" (id 1) (at 198.755 99.06 0))
+    (property "Footprint" "" (id 2) (at 198.755 104.775 0)
+      (effects (font (size 1.27 1.27)) hide)
+    )
+    (property "Datasheet" "~" (id 3) (at 198.755 104.775 0)
+      (effects (font (size 1.27 1.27)) hide)
+    )
+    (pin "1")
+  )
   (symbol (lib_id "000_Capacitor_Electrolytic_Immo:22u") (at 229.235 112.395 0) (unit 1)

Commit message: Schematic reviewed
Parts:
- removed D2: BZV55B18, Diode_SMD:D_MiniMELF_Handsoldering, symbol Diode:BZV55B18
- added C? (x2): 100u, Capacitor_SMD:CP_Elec_10x10, symbol 000_Capacitor_Electrolytic_Immo:100u
- added J29: 3V3 PWR SRC, Connector_PinHeader_2.54mm:PinHeader_1x03_P2.54mm_Vertical, symbol Connector:Conn_01x03_Male
- added J30: 12V_DC, TerminalBlock:TerminalBlock_Altech_AK300-2_P5.00mm, symbol Connector:Screw_Terminal_01x02
- added J31: 5V_DC, TerminalBlock:TerminalBlock_Altech_AK300-2_P5.00mm, symbol Connector:Screw_Terminal_01x02
- J5, J6: footprint (none) -> Connector_USB:USB_A_Molex_67643_Horizontal
- JP1: footprint (none) -> Jumper:SolderJumper-3_P1.3mm_Bridged12_RoundedPad1.0x1.5mm
Connections:
- net 12V_DC_OUT: now also C?.2, J30.2 (Pin_2)
- net 5V_DC_RPI: now also J29.1 (Pin_1), J31.2 (Pin_2)
- net 5V_DC_SERVO: now also C?.2
- net GND_P: now also C?.1, C?.1, J30.1 (Pin_1), J31.1 (Pin_1)
- net USP_PWR_IN: now also J29.3 (Pin_3)
- net at C1.1, JP1.2 (C), U3.3 (VI): now also J29.2 (Pin_2)
- no-connect marks 6 -> 5

Commit message: mbncmvbc,
Parts:
- added D6: 12V Power, symbol Device:LED
- added D7: 3V3 Power, symbol Device:LED
- added J32: GND_BUS, Connector_PinHeader_1.27mm:PinHeader_1x10_P1.27mm_Vertical, symbol Connector:Conn_01x10_Male
- added J33: 12V_BUS, Connector_PinHeader_2.54mm:PinHeader_1x05_P2.54mm_Vertical, symbol 000_Pin_Headers_Immo:Conn_01x05_Male
- added J34: 5V_P_BUS, Connector_PinHeader_2.54mm:PinHeader_1x05_P2.54mm_Vertical, symbol 000_Pin_Headers_Immo:Conn_01x05_Male
- added J35: 5V_D_BUS, Connector_PinHeader_2.54mm:PinHeader_1x05_P2.54mm_Vertical, symbol 000_Pin_Headers_Immo:Conn_01x05_Male
- added J36: 3V3_BUS, Connector_PinHeader_2.54mm:PinHeader_1x05_P2.54mm_Vertical, symbol 000_Pin_Headers_Immo:Conn_01x05_Male
- added R36: 1k, Resistor_SMD:R_0805_2012Metric_Pad1.20x1.40mm_HandSolder, symbol 000_Resistors_Immo:Resistor_0805
- added R37: 330r, Resistor_SMD:R_0805_2012Metric_Pad1.20x1.40mm_HandSolder, symbol 000_Resistors_Immo:Resistor_0805
- gave numbers to parts that had none: 2
Connections:
- net 12V_DC_OUT: now also D6.1 (K), J33.1 (Pin_1), J33.2 (Pin_2), J33.3 (Pin_3), J33.4 (Pin_4), J33.5 (Pin_5)
- net 3V3_DC_MCU: now also D7.1 (K), J36.1 (Pin_1), J36.2 (Pin_2), J36.3 (Pin_3), J36.4 (Pin_4), J36.5 (Pin_5)
- net 5V_DC_RPI: now also J35.1 (Pin_1), J35.2 (Pin_2), J35.3 (Pin_3), J35.4 (Pin_4), J35.5 (Pin_5)
- net 5V_DC_SERVO: now also J34.1 (Pin_1), J34.2 (Pin_2), J34.3 (Pin_3), J34.4 (Pin_4), J34.5 (Pin_5)
- net GND_P: now also R6.1, J32.1 (Pin_1), J32.10 (Pin_10), J32.2 (Pin_2), J32.3 (Pin_3), J32.4 (Pin_4), J32.5 (Pin_5), J32.6 (Pin_6), J32.7 (Pin_7), J32.8 (Pin_8), J32.9 (Pin_9), R36.1, R37.1; no longer R6.2
- net at D1.2 (A), Q1.1 (G): now also R6.2; no longer R6.1
- new net: D6.2 (A), R36.2
- new net: D7.2 (A), R37.2
- no-connect marks 5 -> 4
Other:
- moved on the sheet: R6

Commit message: Footprint Association Underway
Parts:
- removed J5, J6: USB_A, Connector_USB:USB_A_Molex_67643_Horizontal, symbol Connector:USB_A
- added J5: USB_A_Stacked, symbol Connector:USB_A_Stacked
- Q1: footprint Package_TO_SOT_SMD:TO-263-2 -> Package_TO_SOT_THT:TO-220-3_Vertical
- U3: footprint Package_TO_SOT_SMD:TO-263-5_TabPin3 -> Package_TO_SOT_SMD:SOT-223-3_TabPin2
- renumbered C1 to EC1, C45 to EC10, C2 to EC2, C44 to EC9
Connections:
- net 12V_DC_OUT: now also EC9.1; no longer EC9.2
- net 5V_DC_RPI: now also J5.1 (VBUS1), J5.5 (VBUS2)
- net GND_P: now also EC9.2, J5.4 (GND1), J5.8 (GND2), J5.9 (Shield); no longer EC9.1
Other:
- moved on the sheet: EC9, J31
