File: RemoteLabs_supervisor_PCB/power_distribution.kicad_sch (KiCad schematic)
At the start: 34 parts, among them J29 3V3 PWR SRC, J3 XT60_60A_male, J30 12V_DC, J31 5V_DC_RPI, J32 GND_BUS, J33 12V_BUS, J34 5V_P_BUS, J35 5V_D_BUS, J36 3V3_BUS, J4 Strip Lighting, J5 USB_A_Stacked, J6 5V_DC_LED, Q1 IRF5305_PBF, U1 R-78C5.0-1.0, U18 R-78C5.0-1.0, U3 AMS1117-3.3

Commit message: Version 2 PCB Layout
Parts:
- added NT4: NetTie_2, NetTie:NetTie-2_SMD_Pad2.0mm, symbol Device:NetTie_2
Connections:
- net GND_D: no longer C1.2, C10.2, C2.2, C6.2, EC12.2, J6.1 (Pin_1), U1.2 (GND), U18.2 (GND)
- net GND_P: now also J6.1 (Pin_1), NT4.1
- new net GND_PB: C1.2, C10.2, C2.2, C6.2, U1.2 (GND), U18.2 (GND)
- new net PGND0: EC12.2, NT4.2
Changed lines of the file:
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@@
-    (stroke (width 0) (type default) (color 0 0 0 0))
-  )
-  (wire (pts (xy 130.81 126.365) (xy 130.81 128.905))
     (stroke (width 0) (type default) (color 0 0 0 0))
   )
@@
     (stroke (width 0) (type default) (color 0 0 0 0))
   )
-  (wire (pts (xy 174.625 123.19) (xy 177.165 123.19))
-    (stroke (width 0) (type default) (color 0 0 0 0))
-  )
   (wire (pts (xy 218.44 31.75) (xy 218.44 41.91))
     (stroke (width 0) (type default) (color 0 0 0 0))
@@
     (stroke (width 0) (type default) (color 0 0 0 0))
   )
-  (wire (pts (xy 154.305 123.19) (xy 154.305 127.635))
-    (stroke (width 0) (type default) (color 0 0 0 0))
-  )
   (wire (pts (xy 160.655 113.665) (xy 163.83 113.665))
     (stroke (width 0) (type default) (color 0 0 0 0))
@@
     (stroke (width 0) (type default) (color 0 0 0 0))
   )
+  (wire (pts (xy 207.645 97.155) (xy 207.645 99.695))
+    (stroke (width 0) (type default) (color 0 0 0 0))
+  )
   (wire (pts (xy 248.285 86.995) (xy 248.285 88.9))
     (stroke (width 0) (type default) (color 0 0 0 0))
@@
     (stroke (width 0) (type default) (color 0 0 0 0))
   )
+  (wire (pts (xy 154.305 131.445) (xy 154.305 133.35))
+    (stroke (width 0) (type default) (color 0 0 0 0))
+  )
   (wire (pts (xy 118.11 123.825) (xy 118.11 126.365))
     (stroke (width 0) (type default) (color 0 0 0 0))
@@
     (stroke (width 0) (type default) (color 0 0 0 0))
   )
+  (wire (pts (xy 154.305 123.19) (xy 154.305 126.365))
+    (stroke (width 0) (type default) (color 0 0 0 0))
+  )
+  (wire (pts (xy 255.27 106.68) (xy 255.27 107.95))
+    (stroke (width 0) (type default) (color 0 0 0 0))
+  )
   (wire (pts (xy 143.51 153.035) (xy 143.51 155.575))
     (stroke (width 0) (type default) (color 0 0 0 0))
@@
     (stroke (width 0) (type default) (color 0 0 0 0))
   )
-  (wire (pts (xy 255.27 106.68) (xy 255.27 108.585))
-    (stroke (width 0) (type default) (color 0 0 0 0))
-  )
   (wire (pts (xy 65.405 103.505) (xy 67.945 103.505))
     (stroke (width 0) (type default) (color 0 0 0 0))
@@
     (stroke (width 0) (type default) (color 0 0 0 0))
   )
+  (wire (pts (xy 130.81 126.365) (xy 130.81 128.27))
+    (stroke (width 0) (type default) (color 0 0 0 0))
+  )
   (wire (pts (xy 221.615 95.885) (xy 221.615 97.155))
     (stroke (width 0) (type default) (color 0 0 0 0))
@@
     (stroke (width 0) (type default) (color 0 0 0 0))
   )
-  (wire (pts (xy 207.645 97.155) (xy 207.645 99.06))
-    (stroke (width 0) (type default) (color 0 0 0 0))
-  )
   (wire (pts (xy 153.67 24.13) (xy 153.67 26.67))
     (stroke (width 0) (type default) (color 0 0 0 0))
   )
   (wire (pts (xy 138.43 113.665) (xy 143.51 113.665))
+    (stroke (width 0) (type default) (color 0 0 0 0))
+  )
+  (wire (pts (xy 175.895 123.19) (xy 177.165 123.19))
     (stroke (width 0) (type default) (color 0 0 0 0))
   )
@@
     (effects (font (size 1.27 1.27)) (justify left bottom))
   )
+  (label "PGND0" (at 154.305 123.825 270)
+    (effects (font (size 1.27 1.27)) (justify right bottom))
+  )
   (label "01" (at 62.23 43.18 0)
     (effects (font (size 1.27 1.27)) (justify left bottom))
@@
     (effects (font (size 1.27 1.27)) (justify left bottom))
   )
-  (hierarchical_label "GND_D" (shape passive) (at 130.81 128.905 270)
-    (effects (font (size 1.27 1.27)) (justify right))
-  )
-  (hierarchical_label "GND_D" (shape passive) (at 255.27 108.585 270)
-    (effects (font (size 1.27 1.27)) (justify right))
-  )
-  (hierarchical_label "GND_D" (shape passive) (at 168.91 168.275 270)
+  (hierarchical_label "GND_D" (shape passive) (at 255.27 107.95 270)
     (effects (font (size 1.27 1.27)) (justify right))
   )
@@
     (effects (font (size 1.27 1.27)) (justify left))
   )
-  (hierarchical_label "GND_D" (shape passive) (at 174.625 123.19 180)
-    (effects (font (size 1.27 1.27)) (justify right))
-  )
   (hierarchical_label "5V_DC_RPI" (shape output) (at 184.15 63.5 0)
     (effects (font (size 1.27 1.27)) (justify left))
@@
     (effects (font (size 1.27 1.27)) (justify left))
   )
-  (hierarchical_label "GND_D" (shape passive) (at 207.645 99.06 270)
+  (hierarchical_label "GND_PB" (shape passive) (at 130.81 168.275 270)
+    (effects (font (size 1.27 1.27)) (justify right))
+  )
+  (hierarchical_label "GND_D" (shape passive) (at 168.91 168.275 270)
     (effects (font (size 1.27 1.27)) (justify right))
   )
@@
     (effects (font (size 1.27 1.27)) (justify right))
   )
-  (hierarchical_label "GND_D" (shape passive) (at 154.305 127.635 270)
+  (hierarchical_label "GND_P" (shape passive) (at 154.305 133.35 270)
     (effects (font (size 1.27 1.27)) (justify right))
   )
   (hierarchical_label "GND_P" (shape passive) (at 222.25 29.21 180)
-    (effects (font (size 1.27 1.27)) (justify right))
-  )
-  (hierarchical_label "GND_D" (shape passive) (at 130.81 168.275 270)
     (effects (font (size 1.27 1.27)) (justify right))
   )
@@
     (effects (font (size 1.27 1.27)) (justify left))
   )
+  (hierarchical_label "GND_D" (shape passive) (at 207.645 99.695 270)
+    (effects (font (size 1.27 1.27)) (justify right))
+  )
   (hierarchical_label "GND_P" (shape passive) (at 176.53 33.02 180)
     (effects (font (size 1.27 1.27)) (justify right))
@@
   )
   (hierarchical_label "USP_PWR_IN" (shape input) (at 180.34 92.71 270)
+    (effects (font (size 1.27 1.27)) (justify right))
+  )
+  (hierarchical_label "GND_P" (shape passive) (at 175.895 123.19 180)
     (effects (font (size 1.27 1.27)) (justify right))
   )
   (hierarchical_label "5V_DC_LED" (shape output) (at 167.64 113.665 0)
     (effects (font (size 1.27 1.27)) (justify left))
+  )
+  (hierarchical_label "GND_PB" (shape passive) (at 130.81 128.27 270)
+    (effects (font (size 1.27 1.27)) (justify right))
   )
   (symbol (lib_id "000_Pin_Headers_Immo:Conn_01x05_Male") (at 151.13 19.05 270) (unit 1)
@@
       (effects (font (size 1.27 1.27)) hide)
     )
+    (pin "1")
+    (pin "2")
+  )
+  (symbol (lib_id "Device:NetTie_2") (at 154.305 128.905 270) (mirror x) (unit 1)
+    (in_bom yes) (on_board yes) (fields_autoplaced)
+    (property "Reference" "NT4" (id 0) (at 156.21 127.6349 90)
+      (effects (font (size 1.27 1.27)) (justify left))
+    )
+    (property "Value" "NetTie_2" (id 1) (at 156.21 130.1749 90)
+      (effects (font (size 1.27 1.27)) (justify left))
+    )
+    (property "Footprint" "NetTie:NetTie-2_SMD_Pad2.0mm" (id 2) (at 154.305 128.905 0)
+      (effects (font (size 1.27 1.27)) hide)
+    )
+    (property "Datasheet" "~" (id 3) (at 154.305 128.905 0)
+      (effects (font (size 1.27 1.27)) hide)
+    )
