File: RemoteLabs_supervisor_PCB/MCU_student.kicad_sch (KiCad schematic)
At the start: 0 parts

Commit message: nearing circut deisng complete
Parts:
- added A?: Arduino_Nano_33_IoT, Module:Arduino_Nano, symbol MCU_Module:Arduino_Nano_33_IoT
- added C1A?: 100p, Capacitor_SMD:C_0805_2012Metric_Pad1.18x1.45mm_HandSolder, symbol 000_Capacitor_Film_Immo:cap_film_0805
- added C1B?, C? (x4): 100n, Capacitor_SMD:C_0805_2012Metric_Pad1.18x1.45mm_HandSolder, symbol 000_Capacitor_Film_Immo:cap_film_0805
- added C? (x2): 10u, Capacitor_SMD:CP_Elec_6.3x5.9, symbol 000_Capacitor_Electrolytic_Immo:22u
- added C?: 1u, Capacitor_SMD:C_0805_2012Metric_Pad1.18x1.45mm_HandSolder, symbol 000_Capacitor_Film_Immo:cap_film_0805
- added J?: MCU_Header, symbol Connector:Conn_01x08_Male
- added J?: ShiftReg_Header, symbol Connector:Conn_01x08_Male
- added J?: SPI Header, symbol Connector:Conn_01x03_Male
- added JP?: 5Vsup, symbol 000_Connectors_Immo:Jumper_3_Bridged12
- added JP?: 3V3_prog, symbol 000_Connectors_Immo:Jumper_3_Bridged12
- added L?: 10uH, symbol pspice:INDUCTOR
- added R?: 2k2, Resistor_SMD:R_0805_2012Metric_Pad1.20x1.40mm_HandSolder, symbol 000_Resistors_Immo:Resistor_0805
- added R?: 330r, Resistor_SMD:R_0805_2012Metric_Pad1.20x1.40mm_HandSolder, symbol 000_Resistors_Immo:Resistor_0805
- added U?: 4094, symbol 000_Logic_IC_Immo:4094
- added U?: ATSAMD21G18A-M, Package_DFN_QFN:QFN-48-1EP_7x7mm_P0.5mm_EP5.15x5.15mm, symbol MCU_Microchip_SAMD:ATSAMD21G18A-M
Connections:
- new net: A?.17 (3V3), JP?.3 (B)
- new net: A?.30 (VIN), JP?.1 (A)
- new net: J?.1 (Pin_1), U?.13 (PA08)
- new net: J?.2 (Pin_2), U?.24 (PA15)
- new net: J?.3 (Pin_3), U?.32 (PA23)
- new net: J?.4 (Pin_4), U?.34 (PA25)
- new net: J?.5 (Pin_5), U?.39 (PA27)
- new net: J?.6 (Pin_6), U?.41 (PA28)
- new net: J?.7 (Pin_7), U?.45 (PA30)
- new net: J?.8 (Pin_8), U?.46 (PA31)
- new net: C?.1, C?.2, L?.2, U?.6 (VDDANA)
- new net: C?.1, U?.43 (VDDCORE)
- new net 3V3_DC_IN: C1A?.1, C?.1, C?.1, C?.1, C?.2, JP?.2 (C), L?.1, R?.1, U?.15 (OE), U?.16 (VCC), U?.17 (VDDIO), U?.36 (VDDIO), U?.44 (VDDIN)
- new net 5V_DC_IN: JP?.2 (C)
- new net DC_MOTOR_DIR1: A?.15 (D12), U?.28 (PA19)
- new net DC_MOTOR_DIR2: A?.10 (D7), U?.11 (PA06)
- new net DC_MOTOR_EN: J?.1 (Pin_1), U?.4 (Q0)
- new net DC_MOTOR_IS1: A?.26 (A7), U?.48 (PB03)
- new net DC_MOTOR_IS2: A?.25 (A6), U?.14 (PA09)
- new net DC_MOTOR_PWM: A?.13 (D10), U?.30 (PA21)
- new net ENCODER_A: A?.6 (D3), U?.20 (PB11)
- new net ENCODER_B: A?.5 (D2), U?.19 (PB10)
- new net ENCODER_INDEX: A?.7 (D4), U?.12 (PA07)
- new net GND_D: A?.29 (GND), A?.4 (GND), C1A?.2, C1B?.1, C1B?.2, C?.1, C?.1, C?.2, C?.2, C?.2, C?.2, C?.2, R?.2, R?.2, U?.18 (GND), U?.35 (GND), U?.40 (~{RESET}), U?.42 (GND), U?.5 (GNDANA), U?.8 (GND)
- new net LATCH: A?.11 (D8), J?.3 (Pin_3), U?.1 (STROBE), U?.27 (PA18)
- new net LIMIT_1: A?.23 (A4), U?.7 (PB08)
- new net LIMIT_2: U?.31 (PA22)
- new net MCU_RESET: A?.28 (~{RESET}), A?.3 (~{RESET}), R?.1
- new net MOSI: A?.14 (D11), J?.1 (Pin_1), U?.2 (DATA), U?.25 (PA16)
- new net PIXEL_DATA: A?.8 (D5), U?.10 (PA05)
- new net PROG_RX: A?.2 (D0/RX), U?.38 (PB23)
- new net PROG_TX: A?.1 (D1/TX), U?.37 (PB22)
- new net SCK: A?.16 (D13), J?.2 (Pin_2), U?.26 (PA17), U?.3 (CLOCK)
- new net SERVO_1: A?.12 (D9), U?.29 (PA20)
- new net SERVO_2: U?.33 (PA24)
- new net STEPP_DIR: J?.6 (Pin_6), U?.13 (Q5)
- new net STEPP_EN: J?.7 (Pin_7), U?.12 (Q6)
- new net STEPP_FLT: A?.24 (A5), U?.8 (PB09)
- new net STEPP_RST: J?.8 (Pin_8), U?.11 (Q7)
- new net STEPP_STEP: A?.9 (D6), U?.9 (PA04)
- new net THERMO: A?.22 (A3), U?.15 (PA10)
Other:
- note added: "A4 & A5 Internal pull up for I2C Bus Avoid analogRead"
- note added: "Additional Ferrite Bead here?"
- note added: "Arduino Nano IoT 33 Devboard Slot"
- note added: "C1A or C1B IF C1B -> R1 = 10k"
- note added: "Functions Available on Raw MCU Removed for IoT Board to free pins"
- note added: "Main Differences: No need for "Student Enable pins" as this is a supervisor only function No need for any pins that detect input from student No Mode Pins"
- note added: "PCB Laid out for Either: - Arduino Nano 33 IoT OR - SAMD21 MCU Only components for 1 of these options should be populated, the other left emtpty Connectors in the middle are shared by both options and should always be populated"
- note added: "SAMD21 BareMetal MCU Slot"
- note added: "Shift Register to Expand Number of Output Pins"
- note added: "Should be low ESR"
- note added: "Student MCU"
- note added: "https://ww1.microchip.com/downloads/en/DeviceDoc/SAM_D21_DA1_Family_DataSheet_DS40001882F.pdf"

Commit message: V1.0 Circuit Design Complete
Parts:
- removed JP?: 5Vsup, symbol 000_Connectors_Immo:Jumper_3_Bridged12
- added C3: 4n7, Capacitor_SMD:C_0805_2012Metric_Pad1.18x1.45mm_HandSolder, symbol 000_Capacitor_Film_Immo:cap_film_0805
- added C4, C5: 9pF, Capacitor_SMD:C_0805_2012Metric_Pad1.18x1.45mm_HandSolder, symbol 000_Capacitor_Film_Immo:cap_film_0805_mini
- added D3: PRTR5V0U2X, Package_TO_SOT_SMD:SOT-143, symbol Power_Protection:PRTR5V0U2X_smaller
- added J7: USB_B_Mini, Connector_USB:USB_Mini-B_Lumberg_2486_01_Horizontal, symbol Connector:USB_B_Mini
- added J9: Spare Student GPIOs, symbol Connector:Conn_01x04_Male
- added R7: 1M, Resistor_SMD:R_0805_2012Metric_Pad1.20x1.40mm_HandSolder, symbol 000_Resistors_Immo:Resistor_0805
- added Y1: 32.768 kHz, symbol Device:Crystal_Small
- gave numbers to parts that had none: 19
Connections:
- net GND_D: now also C4.1, C5.1, J7.5 (GND)
- net SERVO_2: now also U4.16 (PA11); no longer U4.33 (PA24)
- net STEPP_DIR: now also J10.5 (Pin_5), U5.14 (Q4); no longer J10.6 (Pin_6), U5.13 (Q5)
- net STEPP_EN: now also J10.6 (Pin_6), U5.13 (Q5); no longer J10.7 (Pin_7), U5.12 (Q6)
- net STEPP_RST: now also J10.7 (Pin_7), U5.12 (Q6); no longer J10.8 (Pin_8), U5.11 (Q7)
- net at A1.17 (3V3): now also JP2.1 (A); no longer JP2.3 (B)
- net at J8.4 (Pin_4): now also U4.39 (PA27); no longer U4.34 (PA25)
- net at J8.5 (Pin_5): now also U4.41 (PA28); no longer U4.39 (PA27)
- net at J8.6 (Pin_6): now also U4.45 (PA30); no longer U4.41 (PA28)
- net at J8.7 (Pin_7): now also U4.46 (PA31); no longer U4.45 (PA30)
- net MODE_2: now reaches J8.8 (Pin_8)
- net MODE_2: now also U4.23 (PA14); no longer U4.46 (PA31)
- net at U4.1 (PA00): now also C4.2, Y1.2
- net at U4.2 (PA01): now also C5.2, Y1.1
- net SPARE_2: now reaches U4.21 (PA12)
- net SPARE_2: now also J9.3 (Pin_3)
- net SPARE_3: now reaches U4.22 (PA13)
- net SPARE_3: now also J9.4 (Pin_4)
- net SPARE_0: now reaches U4.3 (PA02)
- net SPARE_0: now also J9.1 (Pin_1)
- net SPARE_1: now reaches U4.4 (PA03)
- net SPARE_1: now also J9.2 (Pin_2)
- new net: C3.1, D3.1 (GND), J7.6 (Shield), R7.1
- new net: C3.2, R7.2
- new net USB_N: D3.3 (I/O2), J7.2 (D-), U4.33 (PA24)
- new net USB_P: D3.2 (I/O1), J7.3 (D+), U4.34 (PA25)
- new net V_USB: D3.4 (VCC), J7.1 (VBUS)
Other:
- note added: "C2A or C2B IF C2B -> R3 = 10k"
- note added: "SAMD21 BareMetal USB I/F"
- note removed: "C1A or C1B IF C1B -> R1 = 10k"
- moved on the sheet: C2A1, C2B1, J10, J11, J8, R3, R4

Commit message: ERC checks run
Parts:
- removed JP2: 3V3_prog, symbol 000_Connectors_Immo:Jumper_3_Bridged12
- added J28: student_PA03, Connector_PinHeader_1.27mm:PinHeader_1x01_P1.27mm_Vertical, symbol 000_Pin_Headers_Immo:Conn_01x01_Male
- J11: value SPI Header -> SPI Student
Connections:
- net 3V3_DC_IN: now also A1.17 (3V3)
- net GND_D: now also C3.2, R7.2, U4.49 (EP)
- net SERVO_2: now also U4.21 (PA12); no longer U4.16 (PA11)
- net SPARE_0: now also A1.19 (A0)
- net SPARE_1: now also A1.20 (A1), U4.47 (PB02); no longer U4.4 (PA03)
- net SPARE_2: now also A1.21 (A2), U4.16 (PA11); no longer U4.21 (PA12)
- net SHIFT_7: now reaches U5.11 (Q7)
- net SHIFT_7: now also J10.8 (Pin_8)
- net SHIFT_1: now reaches U5.5 (Q1)
- net SHIFT_1: now also J10.2 (Pin_2)
- net SHIFT_2: now reaches U5.6 (Q2)
- net SHIFT_2: now also J10.3 (Pin_3)
- net SHIFT_3: now reaches U5.7 (Q3)
- net SHIFT_3: now also J10.4 (Pin_4)
- new net: J28.1 (Pin_1), U4.4 (PA03)
- no-connect marks 0 -> 5

Commit message: Schematic reviewed
Parts:
- J10, J8: footprint (none) -> Connector_PinHeader_2.54mm:PinHeader_1x08_P2.54mm_Vertical
- J11: footprint (none) -> Connector_PinHeader_2.54mm:PinHeader_1x03_P2.54mm_Vertical
- J9: footprint (none) -> Connector_PinHeader_2.54mm:PinHeader_1x04_P2.54mm_Vertical
- L1: footprint (none) -> Inductor_SMD:L_0805_2012Metric_Pad1.15x1.40mm_HandSolder
- U5: footprint (none) -> Package_DIP:SMDIP-18_W9.53mm
- Y1: footprint (none) -> Crystal:Crystal_SMD_SeikoEpson_MC405-2Pin_9.6x4.1mm_HandSoldering
Other:
- moved on the sheet: J10, J11
Changed lines of the file:
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@@
     (stroke (width 0) (type default) (color 0 0 0 0))
   )
-  (wire (pts (xy 160.02 153.67) (xy 170.815 153.67))
+  (wire (pts (xy 154.94 153.67) (xy 165.735 153.67))
     (stroke (width 0) (type default) (color 0 0 0 0))
   )
@@
     (stroke (width 0) (type default) (color 0 0 0 0))
   )
-  (wire (pts (xy 157.48 127) (xy 161.29 127))
+  (wire (pts (xy 154.94 126.365) (xy 158.75 126.365))
     (stroke (width 0) (type default) (color 0 0 0 0))
   )
@@
     (stroke (width 0) (type default) (color 0 0 0 0))
   )
-  (wire (pts (xy 160.02 148.59) (xy 170.815 148.59))
+  (wire (pts (xy 154.94 148.59) (xy 165.735 148.59))
     (stroke (width 0) (type default) (color 0 0 0 0))
   )
@@
     (stroke (width 0) (type default) (color 0 0 0 0))
   )
-  (wire (pts (xy 157.48 119.38) (xy 168.275 119.38))
+  (wire (pts (xy 154.94 118.745) (xy 165.735 118.745))
     (stroke (width 0) (type default) (color 0 0 0 0))
   )
@@
     (stroke (width 0) (type default) (color 0 0 0 0))
   )
-  (wire (pts (xy 157.48 132.08) (xy 168.275 132.08))
+  (wire (pts (xy 154.94 131.445) (xy 165.735 131.445))
     (stroke (width 0) (type default) (color 0 0 0 0))
   )
@@
     (stroke (width 0) (type default) (color 0 0 0 0))
   )
-  (wire (pts (xy 160.02 151.13) (xy 170.815 151.13))
+  (wire (pts (xy 154.94 151.13) (xy 165.735 151.13))
     (stroke (width 0) (type default) (color 0 0 0 0))
   )
@@
     (stroke (width 0) (type default) (color 0 0 0 0))
   )
-  (wire (pts (xy 157.48 116.84) (xy 168.275 116.84))
+  (wire (pts (xy 154.94 116.205) (xy 165.735 116.205))
     (stroke (width 0) (type default) (color 0 0 0 0))
   )
@@
     (stroke (width 0) (type default) (color 0 0 0 0))
   )
-  (wire (pts (xy 157.48 129.54) (xy 161.29 129.54))
+  (wire (pts (xy 154.94 128.905) (xy 158.75 128.905))
     (stroke (width 0) (type default) (color 0 0 0 0))
   )
@@
     (stroke (width 0) (type default) (color 0 0 0 0))
   )
-  (wire (pts (xy 157.48 124.46) (xy 161.29 124.46))
+  (wire (pts (xy 154.94 123.825) (xy 158.75 123.825))
     (stroke (width 0) (type default) (color 0 0 0 0))
   )
@@
     (stroke (width 0) (type default) (color 0 0 0 0))
   )
-  (wire (pts (xy 161.29 114.3) (xy 157.48 114.3))
+  (wire (pts (xy 158.75 113.665) (xy 154.94 113.665))
     (stroke (width 0) (type default) (color 0 0 0 0))
   )
@@
     (stroke (width 0) (type default) (color 0 0 0 0))
   )
-  (wire (pts (xy 157.48 121.92) (xy 168.275 121.92))
+  (wire (pts (xy 154.94 121.285) (xy 165.735 121.285))
     (stroke (width 0) (type default) (color 0 0 0 0))
   )
@@
     (effects (font (size 1.27 1.27)) (justify right bottom))
   )
-  (label "SCK" (at 170.815 151.13 180)
+  (label "SCK" (at 165.735 151.13 180)
     (effects (font (size 1.27 1.27)) (justify right bottom))
   )
@@
     (effects (font (size 1.27 1.27)) (justify left bottom))
   )
-  (label "MOSI" (at 170.815 148.59 180)
+  (label "MOSI" (at 165.735 148.59 180)
     (effects (font (size 1.27 1.27)) (justify right bottom))
   )
@@
     (effects (font (size 1.27 1.27)) (justify left bottom))
   )
-  (label "SHIFT_7" (at 168.275 132.08 180)
+  (label "SHIFT_7" (at 165.735 131.445 180)
     (effects (font (size 1.27 1.27)) (justify right bottom))
   )
@@
     (effects (font (size 1.27 1.27)) (justify left bottom))
   )
-  (label "SHIFT_1" (at 168.275 116.84 180)
+  (label "SHIFT_1" (at 165.735 116.205 180)
     (effects (font (size 1.27 1.27)) (justify right bottom))
   )
@@
     (effects (font (size 1.27 1.27)) (justify left bottom))
   )
-  (label "SHIFT_2" (at 168.275 119.38 180)
+  (label "SHIFT_2" (at 165.735 118.745 180)
     (effects (font (size 1.27 1.27)) (justify right bottom))
   )
@@
     (effects (font (size 1.27 1.27)) (justify right bottom))
   )
-  (label "SHIFT_3" (at 168.275 121.92 180)
+  (label "SHIFT_3" (at 165.735 121.285 180)
     (effects (font (size 1.27 1.27)) (justify right bottom))
   )
@@
     (effects (font (size 1.27 1.27)) (justify left bottom))
   )
-  (label "LATCH" (at 170.815 153.67 180)
+  (label "LATCH" (at 165.735 153.67 180)
     (effects (font (size 1.27 1.27)) (justify right bottom))
   )
@@
     (effects (font (size 1.27 1.27)) (justify right))
   )
-  (hierarchical_label "STEPP_EN" (shape output) (at 161.29 127 0)
+  (hierarchical_label "STEPP_EN" (shape output) (at 158.75 126.365 0)
     (effects (font (size 1.27 1.27)) (justify left))
   )
@@
     (effects (font (size 1.27 1.27)) (justify right))
   )
-  (hierarchical_label "DC_MOTOR_EN" (shape output) (at 161.29 114.3 0)
+  (hierarchical_label "DC_MOTOR_EN" (shape output) (at 158.75 113.665 0)
     (effects (font (size 1.27 1.27)) (justify left))
   )
@@
     (effects (font (size 1.27 1.27)) (justify right))
   )
-  (hierarchical_label "STEPP_RST" (shape output) (at 161.29 129.54 0)
+  (hierarchical_label "STEPP_RST" (shape output) (at 158.75 128.905 0)
     (effects (font (size 1.27 1.27)) (justify left))
   )
@@
     (effects (font (size 1.27 1.27)) (justify right))
   )
-  (hierarchical_label "STEPP_DIR" (shape output) (at 161.29 124.46 0)
+  (hierarchical_label "STEPP_DIR" (shape output) (at 158.75 123.825 0)
     (effects (font (size 1.27 1.27)) (justify left))
   )
@@
     (property "Reference" "J9" (id 0) (at 150.495 160.02 0))
     (property "Value" "Spare Student GPIOs" (id 1) (at 150.495 162.56 0))
-    (property "Footprint" "" (id 2) (at 149.86 167.64 0)
+    (property "Footprint" "Connector_PinHeader_2.54mm:PinHeader_1x04_P2.54mm_Vertical" (id 2) (at 149.86 167.64 0)
       (effects (font (size 1.27 1.27)) hide)
     )
@@
       (effects (font (size 1.27 1.27)) (justify left))
     )
-    (property "Footprint" "" (id 2) (at 219.71 137.16 0)
+    (property "Footprint" "Package_DIP:SMDIP-18_W9.53mm" (id 2) (at 219.71 137.16 0)
       (effects (font (size 1.27 1.27)) hide)
     )
@@
     (property "Reference" "J8" (id 0) (at 28.575 102.87 0))
     (property "Value" "MCU_Header" (id 1) (at 28.575 105.41 0))
-    (property "Footprint" "" (id 2) (at 27.94 115.57 0)
+    (property "Footprint" "Connector_PinHeader_2.54mm:PinHeader_1x08_P2.54mm_Vertical" (id 2) (at 27.94 115.57 0)
       (effects (font (size 1.27 1.27)) hide)
     )
@@
     (pin "2")
   )
-  (symbol (lib_id "Connector:Conn_01x08_Male") (at 152.4 121.92 0) (unit 1)
-    (in_bom yes) (on_board yes) (fields_autoplaced)
-    (property "Reference" "J10" (id 0) (at 147.32 123.19 90))
-    (property "Value" "ShiftReg_Header" (id 1) (at 149.86 123.19 90))
-    (property "Footprint" "" (id 2) (at 152.4 121.92 0)
-      (effects (font (size 1.27 1.27)) hide)
-    )
-    (property "Datasheet" "~" (id 3) (at 152.4 121.92 0)
+  (symbol (lib_name "Conn_01x08_Male_1") (lib_id "Connector:Conn_01x08_Male") (at 149.86 121.285 0) (unit 1)
+    (in_bom yes) (on_board yes) (fields_autoplaced)
+    (property "Reference" "J10" (id 0) (at 144.78 122.555 90))
+    (property "Value" "ShiftReg_Header" (id 1) (at 147.32 122.555 90))
+    (property "Footprint" "Connector_PinHeader_2.54mm:PinHeader_1x08_P2.54mm_Vertical" (id 2) (at 149.86 121.285 0)
+      (effects (font (size 1.27 1.27)) hide)
+    )
+    (property "Datasheet" "~" (id 3) (at 149.86 121.285 0)
       (effects (font (size 1.27 1.27)) hide)
     )
@@
       (effects (font (size 1.27 1.27)) (justify left))
     )
-    (property "Footprint" "" (id 2) (at 69.85 82.55 0)
+    (property "Footprint" "Crystal:Crystal_SMD_SeikoEpson_MC405-2Pin_9.6x4.1mm_HandSoldering" (id 2) (at 69.85 82.55 0)
       (effects (font (size 1.27 1.27)) hide)
     )
@@
     (pin "2")
   )
-  (symbol (lib_id "Connector:Conn_01x03_Male") (at 154.94 151.13 0) (unit 1)
-    (in_bom yes) (on_board yes) (fields_autoplaced)
-    (property "Reference" "J11" (id 0) (at 155.575 143.51 0))
-    (property "Value" "SPI Student" (id 1) (at 155.575 146.05 0))
-    (property "Footprint" "" (id 2) (at 154.94 151.13 0)
-      (effects (font (size 1.27 1.27)) hide)
-    )
-    (property "Datasheet" "~" (id 3) (at 154.94 151.13 0)
+  (symbol (lib_id "Connector:Conn_01x03_Male") (at 149.86 151.13 0) (unit 1)
+    (in_bom yes) (on_board yes) (fields_autoplaced)
+    (property "Reference" "J11" (id 0) (at 150.495 143.51 0))
+    (property "Value" "SPI Student" (id 1) (at 150.495 146.05 0))
+    (property "Footprint" "Connector_PinHeader_2.54mm:PinHeader_1x03_P2.54mm_Vertical" (id 2) (at 149.86 151.13 0)
+      (effects (font (size 1.27 1.27)) hide)
+    )
+    (property "Datasheet" "~" (id 3) (at 149.86 151.13 0)
       (effects (font (size 1.27 1.27)) hide)
     )
@@
     (property "Reference" "L1" (id 0) (at 99.06 52.07 0))
     (property "Value" "10uH" (id 1) (at 99.06 54.61 0))
-    (property "Footprint" "" (id 2) (at 99.06 57.15 0)
-      (effects (font (size 1.27 1.27)) hide)
-    )
+    (property "Footprint" "Inductor_SMD:L_0805_2012Metric_Pad1.15x1.40mm_HandSolder" (id 2) (at 99.06 57.15 0)
+      (effects (font (size 1.27 1.27)) hide)
+    )

Commit message: mbncmvbc,
Parts:
- removed L1: 10uH, Inductor_SMD:L_0805_2012Metric_Pad1.15x1.40mm_HandSolder, symbol pspice:INDUCTOR
- added D2: PMEG6020ER, Diode_SMD:Nexperia_CFP3_SOD-123W, symbol Diode:PMEG6020ER
- added FB1: BLM18PG471, Inductor_SMD:L_0805_2012Metric_Pad1.05x1.20mm_HandSolder, symbol Device:FerriteBead_Small
- added SW2: Student Reset, symbol 000_Switches_Immo:pushbutton_tactile_2pin_SMD
Connections:
- net 3V3_DC_IN: now also R3.2, FB1.1; no longer R3.1
- net GND_D: now also R3.1, R4.1, R7.1, SW2.1; no longer R3.2, R4.2, R7.2
- net MCU_RESET: now also R4.2, SW2.2; no longer R4.1
- net V_USB: now also D2.1 (K); no longer D3.4 (VCC), J7.1 (VBUS)
- net at C3.1, D3.1 (GND), J7.6 (Shield): now also R7.2; no longer R7.1
- net at C10.1, C11.2, U4.6 (VDDANA): now also FB1.2
- new net: D2.2 (A), D3.4 (VCC), J7.1 (VBUS)
Other:
- moved on the sheet: R3, R4, R7
