File: RemoteLabs_supervisor_PCB/MCU_student.kicad_sch (KiCad schematic)
At the start: 29 parts, among them J10 ShiftReg_Header, J11 SPI Student, J28 student_PA03, J7 USB_B_Mini, J8 MCU_Header, J9 Spare Student GPIOs, SW2 Student Reset, U4 ATSAMD21G18A-M, U5 4094, Y1 32.768 kHz

Commit message: Finished BOM and purchasing
Parts:
- added D?: Yellow, symbol Device:LED
- added R?: 330r, Resistor_SMD:R_0805_2012Metric_Pad1.20x1.40mm_HandSolder, symbol 000_Resistors_Immo:Resistor_0805
Connections:
- net GND_D: now also D?.1 (K)
- net SCK: now also R?.2
- new net: D?.2 (A), R?.1
Other:
- note added: "Replicates LED_BUILTIN on Arduino Pin: D13"
- moved on the sheet: J11, J9
Changed lines of the file:
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@@
   (junction (at 69.85 80.01) (diameter 0) (color 0 0 0 0)
+  )
+  (junction (at 157.48 160.02) (diameter 0) (color 0 0 0 0)
   )
   (junction (at 91.44 48.26) (diameter 0) (color 0 0 0 0)
@@
     (stroke (width 0) (type default) (color 0 0 0 0))
   )
+  (wire (pts (xy 157.48 170.815) (xy 157.48 173.355))
+    (stroke (width 0) (type default) (color 0 0 0 0))
+  )
   (wire (pts (xy 93.98 171.45) (xy 93.98 177.8))
     (stroke (width 0) (type default) (color 0 0 0 0))
   )
+  (wire (pts (xy 157.48 160.02) (xy 157.48 163.195))
+    (stroke (width 0) (type default) (color 0 0 0 0))
+  )
   (wire (pts (xy 60.96 80.01) (xy 64.77 80.01))
     (stroke (width 0) (type default) (color 0 0 0 0))
@@
     (stroke (width 0) (type default) (color 0 0 0 0))
   )
-  (wire (pts (xy 154.94 153.67) (xy 165.735 153.67))
+  (wire (pts (xy 141.605 162.56) (xy 152.4 162.56))
     (stroke (width 0) (type default) (color 0 0 0 0))
   )
@@
     (stroke (width 0) (type default) (color 0 0 0 0))
   )
-  (wire (pts (xy 154.94 148.59) (xy 165.735 148.59))
+  (wire (pts (xy 141.605 157.48) (xy 152.4 157.48))
     (stroke (width 0) (type default) (color 0 0 0 0))
   )
@@
     (stroke (width 0) (type default) (color 0 0 0 0))
   )
+  (wire (pts (xy 157.48 160.02) (xy 165.1 160.02))
+    (stroke (width 0) (type default) (color 0 0 0 0))
+  )
   (wire (pts (xy 116.84 35.56) (xy 116.84 48.26))
     (stroke (width 0) (type default) (color 0 0 0 0))
@@
     (stroke (width 0) (type default) (color 0 0 0 0))
   )
+  (wire (pts (xy 157.48 180.975) (xy 157.48 182.88))
+    (stroke (width 0) (type default) (color 0 0 0 0))
+  )
   (wire (pts (xy 50.8 49.53) (xy 59.69 49.53))
     (stroke (width 0) (type default) (color 0 0 0 0))
@@
     (stroke (width 0) (type default) (color 0 0 0 0))
   )
-  (wire (pts (xy 154.94 151.13) (xy 165.735 151.13))
+  (wire (pts (xy 141.605 160.02) (xy 157.48 160.02))
     (stroke (width 0) (type default) (color 0 0 0 0))
   )
@@
     (stroke (width 0) (type default) (color 0 0 0 0))
   )
-  (wire (pts (xy 154.94 170.18) (xy 165.735 170.18))
-    (stroke (width 0) (type default) (color 0 0 0 0))
-  )
-  (wire (pts (xy 154.94 165.1) (xy 165.735 165.1))
+  (wire (pts (xy 154.94 144.78) (xy 165.735 144.78))
+    (stroke (width 0) (type default) (color 0 0 0 0))
+  )
+  (wire (pts (xy 154.94 139.7) (xy 165.735 139.7))
     (stroke (width 0) (type default) (color 0 0 0 0))
   )
@@
     (stroke (width 0) (type default) (color 0 0 0 0))
   )
-  (wire (pts (xy 154.94 167.64) (xy 165.735 167.64))
+  (wire (pts (xy 154.94 142.24) (xy 165.735 142.24))
     (stroke (width 0) (type default) (color 0 0 0 0))
   )
@@
     (stroke (width 0) (type default) (color 0 0 0 0))
   )
-  (wire (pts (xy 154.94 172.72) (xy 165.735 172.72))
+  (wire (pts (xy 154.94 147.32) (xy 165.735 147.32))
     (stroke (width 0) (type default) (color 0 0 0 0))
   )
@@
     (effects (font (size 1.27 1.27)) (justify left bottom))
   )
-  (label "SPARE_0" (at 165.735 165.1 180)
-    (effects (font (size 1.27 1.27)) (justify right bottom))
-  )
-  (label "SPARE_1" (at 165.735 167.64 180)
+  (text "Replicates LED_BUILTIN\non Arduino Pin: D13" (at 132.08 175.26 0)
+    (effects (font (size 1.27 1.27)) (justify left bottom))
+  )
+  (label "SPARE_0" (at 165.735 139.7 180)
+    (effects (font (size 1.27 1.27)) (justify right bottom))
+  )
+  (label "SPARE_1" (at 165.735 142.24 180)
     (effects (font (size 1.27 1.27)) (justify right bottom))
   )
@@
     (effects (font (size 1.27 1.27)) (justify right bottom))
   )
-  (label "SPARE_3" (at 165.735 172.72 180)
-    (effects (font (size 1.27 1.27)) (justify right bottom))
-  )
-  (label "SCK" (at 165.735 151.13 180)
+  (label "SPARE_3" (at 165.735 147.32 180)
+    (effects (font (size 1.27 1.27)) (justify right bottom))
+  )
+  (label "SCK" (at 165.1 160.02 180)
     (effects (font (size 1.27 1.27)) (justify right bottom))
   )
@@
     (effects (font (size 1.27 1.27)) (justify left bottom))
   )
-  (label "MOSI" (at 165.735 148.59 180)
+  (label "MOSI" (at 152.4 157.48 180)
     (effects (font (size 1.27 1.27)) (justify right bottom))
   )
@@
     (effects (font (size 1.27 1.27)) (justify right bottom))
   )
-  (label "SPARE_2" (at 165.735 170.18 180)
+  (label "SPARE_2" (at 165.735 144.78 180)
     (effects (font (size 1.27 1.27)) (justify right bottom))
   )
@@
     (effects (font (size 1.27 1.27)) (justify left bottom))
   )
-  (label "LATCH" (at 165.735 153.67 180)
+  (label "LATCH" (at 152.4 162.56 180)
     (effects (font (size 1.27 1.27)) (justify right bottom))
   )
@@
   (hierarchical_label "DC_MOTOR_PWM" (shape output) (at 247.65 55.88 0)
     (effects (font (size 1.27 1.27)) (justify left))
+  )
+  (hierarchical_label "GND_D" (shape passive) (at 157.48 182.88 270)
+    (effects (font (size 1.27 1.27)) (justify right))
   )
   (hierarchical_label "DC_MOTOR_IS2" (shape input) (at 204.47 50.8 180)
@@
     (pin "2")
   )
-  (symbol (lib_id "Connector:Conn_01x04_Male") (at 149.86 167.64 0) (unit 1)
+  (symbol (lib_id "Connector:Conn_01x04_Male") (at 149.86 142.24 0) (unit 1)
     (in_bom yes) (on_board yes) (fields_autoplaced)
-    (property "Reference" "J9" (id 0) (at 150.495 160.02 0))
-    (property "Value" "Spare Student GPIOs" (id 1) (at 150.495 162.56 0))
-    (property "Footprint" "Connector_PinHeader_2.54mm:PinHeader_1x04_P2.54mm_Vertical" (id 2) (at 149.86 167.64 0)
-      (effects (font (size 1.27 1.27)) hide)
-    )
-    (property "Datasheet" "~" (id 3) (at 149.86 167.64 0)
+    (property "Reference" "J9" (id 0) (at 150.495 134.62 0))
+    (property "Value" "Spare Student GPIOs" (id 1) (at 150.495 137.16 0))
+    (property "Footprint" "Connector_PinHeader_2.54mm:PinHeader_1x04_P2.54mm_Vertical" (id 2) (at 149.86 142.24 0)
+      (effects (font (size 1.27 1.27)) hide)
+    )
+    (property "Datasheet" "~" (id 3) (at 149.86 142.24 0)
       (effects (font (size 1.27 1.27)) hide)
     )
@@
     (pin "2")
   )
+  (symbol (lib_id "Device:LED") (at 157.48 177.165 90) (unit 1)
+    (in_bom yes) (on_board yes) (fields_autoplaced)
+    (property "Reference" "D?" (id 0) (at 161.29 177.4824 90)
+      (effects (font (size 1.27 1.27)) (justify right))
+    )
+    (property "Value" "Yellow" (id 1) (at 161.29 180.0224 90)
+      (effects (font (size 1.27 1.27)) (justify right))
+    )
+    (property "Footprint" "" (id 2) (at 157.48 177.165 0)
+      (effects (font (size 1.27 1.27)) hide)
+    )
+    (property "Datasheet" "~" (id 3) (at 157.48 177.165 0)
+      (effects (font (size 1.27 1.27)) hide)
+    )
+    (pin "1")
+    (pin "2")
+  )
   (symbol (lib_id "000_Pin_Headers_Immo:Conn_01x01_Male") (at 38.1 90.17 0) (unit 1)
     (in_bom yes) (on_board yes)
@@
     (pin "2")
   )
-  (symbol (lib_id "Connector:Conn_01x03_Male") (at 149.86 151.13 0) (unit 1)
+  (symbol (lib_id "000_Resistors_Immo:Resistor_0805") (at 157.48 167.005 90) (unit 1)
     (in_bom yes) (on_board yes) (fields_autoplaced)
-    (property "Reference" "J11" (id 0) (at 150.495 143.51 0))
-    (property "Value" "SPI Student" (id 1) (at 150.495 146.05 0))
-    (property "Footprint" "Connector_PinHeader_2.54mm:PinHeader_1x03_P2.54mm_Vertical" (id 2) (at 149.86 151.13 0)
-      (effects (font (size 1.27 1.27)) hide)
-    )
-    (property "Datasheet" "~" (id 3) (at 149.86 151.13 0)
-      (effects (font (size 1.27 1.27)) hide)
-    )
+    (property "Reference" "R?" (id 0) (at 160.02 165.7349 90)
+      (effects (font (size 1.27 1.27)) (justify right))
+    )
+    (property "Value" "330r" (id 1) (at 160.02 168.2749 90)
+      (effects (font (size 1.27 1.27)) (justify right))
+    )
+    (property "Footprint" "Resistor_SMD:R_0805_2012Metric_Pad1.20x1.40mm_HandSolder" (id 2) (at 157.48 168.783 90)
+      (effects (font (size 1.27 1.27)) hide)
+    )
+    (property "Datasheet" "~" (id 3) (at 157.48 167.005 0)
+      (effects (font (size 1.27 1.27)) hide)
+    )
+    (pin "1")
+    (pin "2")
+  )
+  (symbol (lib_id "Connector:Conn_01x03_Male") (at 136.525 160.02 0) (unit 1)
+    (in_bom yes) (on_board yes) (fields_autoplaced)
+    (property "Reference" "J11" (id 0) (at 137.16 152.4 0))
+    (property "Value" "SPI Student" (id 1) (at 137.16 154.94 0))
+    (property "Footprint" "Connector_PinHeader_2.54mm:PinHeader_1x03_P2.54mm_Vertical" (id 2) (at 136.525 160.02 0)
+      (effects (font (size 1.27 1.27)) hide)
+    )
+    (property "Datasheet" "~" (id 3) (at 136.525 160.02 0)
+      (effects (font (size 1.27 1.27)) hide)
+    )

Commit message: Footprint Association Underway
Parts:
- gave numbers to parts that had none: 2
- renumbered C6 to EC3, C10 to EC4
Changed lines of the file:
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@@
   (symbol (lib_id "000_Capacitor_Electrolytic_Immo:22u") (at 80.01 48.26 270) (unit 1)
     (in_bom yes) (on_board yes) (fields_autoplaced)
-    (property "Reference" "C6" (id 0) (at 80.899 40.64 90))
+    (property "Reference" "EC3" (id 0) (at 80.899 40.64 90))
     (property "Value" "10u" (id 1) (at 80.899 43.18 90))
     (property "Footprint" "Capacitor_SMD:CP_Elec_6.3x5.9" (id 2) (at 76.2 49.2252 0)
@@
   (symbol (lib_id "000_Capacitor_Electrolytic_Immo:22u") (at 111.76 57.15 90) (unit 1)
     (in_bom yes) (on_board yes) (fields_autoplaced)
-    (property "Reference" "C10" (id 0) (at 110.871 49.53 90))
+    (property "Reference" "EC4" (id 0) (at 110.871 49.53 90))
     (property "Value" "10u" (id 1) (at 110.871 52.07 90))
     (property "Footprint" "Capacitor_SMD:CP_Elec_6.3x5.9" (id 2) (at 115.57 56.1848 0)
@@
   (symbol (lib_id "Device:LED") (at 157.48 177.165 90) (unit 1)
     (in_bom yes) (on_board yes) (fields_autoplaced)
-    (property "Reference" "D?" (id 0) (at 161.29 177.4824 90)
+    (property "Reference" "D8" (id 0) (at 161.29 177.4824 90)
       (effects (font (size 1.27 1.27)) (justify right))
     )
@@
   (symbol (lib_id "000_Resistors_Immo:Resistor_0805") (at 157.48 167.005 90) (unit 1)
     (in_bom yes) (on_board yes) (fields_autoplaced)
-    (property "Reference" "R?" (id 0) (at 160.02 165.7349 90)
-      (effects (font (size 1.27 1.27)) (justify right))
-    )
+    (property "Reference" "R38" (id 0) (at 160.02 165.7349 90)
+      (effects (font (size 1.27 1.27)) (justify right))
+    )
