File: RemoteLabs_supervisor_PCB/stepper_controller.kicad_sch (KiCad schematic)
At the start: 0 parts

Commit message: started working on schematic
Parts:
- added A?: DRV8825 High Current Stepper Motor Driver Module, Module:Arduino_UNO_R3, symbol 000_Modules_Immo:DRV8825 High Current Stepper Motor Driver Module
- added C?: 100u, Capacitor_SMD:CP_Elec_10x10, symbol 000_Capacitor_Electrolytic_Immo:100u
- added J?: Stepper Motor Output, symbol Connector:Conn_01x04_Male
Connections:
- new net: A?.11 (2A), J?.4 (Pin_4)
- new net: A?.12 (1A), J?.3 (Pin_3)
- new net: A?.13 (1B), J?.2 (Pin_2)
- new net: A?.14 (2B), J?.1 (Pin_1)
- new net DIRECTION: A?.8 (DIR)
- new net DISABLE: A?.1 (EN)
- new net ENABLE: A?.5 (~{RESET}), A?.6 (~{SLEEP})
- new net FAULT_OUT: A?.10 (FAULT)
- new net GND_D: A?.9 (GND_D)
- new net MODE_0: A?.2 (MODE_0)
- new net MODE_1: A?.3 (MODE_1)
- new net MODE_2: A?.4 (MODE_2)
- new net STEP: A?.7 (STEP)
- new net STEPPER_PGND: A?.15 (GND_P), C?.2
- new net STEPPER_VSUP: A?.16 (VMOT), C?.1
Other:
- note added: "M"

Commit message: Schematic Work
Connections:
- net DISABLE is gone; now on net ENABLE: A?.1 (EN)
- net ENABLE: no longer A?.5 (~{RESET}), A?.6 (~{SLEEP})
- new net RESET: A?.5 (~{RESET})
- new net SLEEP: A?.6 (~{SLEEP})
Changed lines of the file:
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@@
 (kicad_sch (version 20211123) (generator eeschema)
   (paper "A4")
-  (junction (at 105.41 107.95) (diameter 0) (color 0 0 0 0)
-  )
   (junction (at 162.56 93.98) (diameter 0) (color 0 0 0 0)
   )
@@
     (stroke (width 0) (type default) (color 0 0 0 0))
   )
+  (wire (pts (xy 102.87 105.41) (xy 107.95 105.41))
+    (stroke (width 0) (type default) (color 0 0 0 0))
+  )
   (wire (pts (xy 148.59 100.33) (xy 152.4 100.33))
+    (stroke (width 0) (type default) (color 0 0 0 0))
+  )
+  (wire (pts (xy 102.87 109.22) (xy 107.95 109.22))
     (stroke (width 0) (type default) (color 0 0 0 0))
   )
@@
     (stroke (width 0) (type default) (color 0 0 0 0))
   )
-  (wire (pts (xy 105.41 109.22) (xy 105.41 107.95))
-    (stroke (width 0) (type default) (color 0 0 0 0))
-  )
   (wire (pts (xy 142.24 90.17) (xy 154.94 90.17))
     (stroke (width 0) (type default) (color 0 0 0 0))
@@
   )
   (wire (pts (xy 102.87 93.98) (xy 107.95 93.98))
-    (stroke (width 0) (type default) (color 0 0 0 0))
-  )
-  (wire (pts (xy 105.41 107.95) (xy 105.41 105.41))
     (stroke (width 0) (type default) (color 0 0 0 0))
   )
@@
     (stroke (width 0) (type default) (color 0 0 0 0))
   )
-  (wire (pts (xy 107.95 109.22) (xy 105.41 109.22))
-    (stroke (width 0) (type default) (color 0 0 0 0))
-  )
   (wire (pts (xy 154.94 90.17) (xy 154.94 83.82))
     (stroke (width 0) (type default) (color 0 0 0 0))
   )
-  (wire (pts (xy 105.41 105.41) (xy 107.95 105.41))
-    (stroke (width 0) (type default) (color 0 0 0 0))
-  )
   (wire (pts (xy 148.59 109.22) (xy 142.24 109.22))
-    (stroke (width 0) (type default) (color 0 0 0 0))
-  )
-  (wire (pts (xy 102.87 107.95) (xy 105.41 107.95))
     (stroke (width 0) (type default) (color 0 0 0 0))
   )
@@
     (effects (font (size 1.27 1.27)) (justify left bottom))
   )
-  (hierarchical_label "DISABLE" (shape input) (at 102.87 90.17 180)
+  (hierarchical_label "ENABLE" (shape input) (at 102.87 90.17 180)
     (effects (font (size 1.27 1.27)) (justify right))
   )
@@
     (effects (font (size 1.27 1.27)) (justify left))
   )
-  (hierarchical_label "ENABLE" (shape input) (at 102.87 107.95 180)
+  (hierarchical_label "SLEEP" (shape input) (at 102.87 109.22 180)
     (effects (font (size 1.27 1.27)) (justify right))
   )
@@
     (effects (font (size 1.27 1.27)) (justify right))
   )
+  (hierarchical_label "RESET" (shape input) (at 102.87 105.41 180)
+    (effects (font (size 1.27 1.27)) (justify right))
+  )

Commit message: V1.0 Circuit Design Complete
Parts:
- gave numbers to parts that had none: 3
Changed lines of the file:
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@@
   (symbol (lib_id "000_Modules_Immo:DRV8825 High Current Stepper Motor Driver Module") (at 125.73 102.87 0) (unit 1)
     (in_bom yes) (on_board yes) (fields_autoplaced)
-    (property "Reference" "A?" (id 0) (at 125.095 77.47 0))
+    (property "Reference" "A4" (id 0) (at 125.095 77.47 0))
     (property "Value" "DRV8825 High Current Stepper Motor Driver Module" (id 1) (at 125.095 80.01 0))
     (property "Footprint" "Module:Arduino_UNO_R3" (id 2) (at 129.54 134.62 0)
@@
   (symbol (lib_id "000_Capacitor_Electrolytic_Immo:100u") (at 162.56 88.9 0) (unit 1)
     (in_bom yes) (on_board yes) (fields_autoplaced)
-    (property "Reference" "C?" (id 0) (at 166.37 86.7409 0)
+    (property "Reference" "C23" (id 0) (at 166.37 86.7409 0)
       (effects (font (size 1.27 1.27)) (justify left))
     )
@@
   (symbol (lib_id "Connector:Conn_01x04_Male") (at 157.48 102.87 0) (mirror y) (unit 1)
     (in_bom yes) (on_board yes)
-    (property "Reference" "J?" (id 0) (at 153.67 96.52 0)
+    (property "Reference" "J19" (id 0) (at 153.67 96.52 0)
       (effects (font (size 1.27 1.27)) (justify right))
     )

Commit message: Schematic reviewed
Parts:
- J19: footprint (none) -> Connector_PinHeader_2.54mm:PinHeader_1x04_P2.54mm_Vertical
Changed lines of the file:
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@@
       (effects (font (size 1.27 1.27)) (justify right))
     )
-    (property "Footprint" "" (id 2) (at 157.48 102.87 0)
+    (property "Footprint" "Connector_PinHeader_2.54mm:PinHeader_1x04_P2.54mm_Vertical" (id 2) (at 157.48 102.87 0)
       (effects (font (size 1.27 1.27)) hide)
     )

Commit message: Footprint Association Underway
Parts:
- renumbered C23 to EC11
Changed lines of the file:
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@@
   (symbol (lib_id "000_Capacitor_Electrolytic_Immo:100u") (at 162.56 88.9 0) (unit 1)
     (in_bom yes) (on_board yes) (fields_autoplaced)
-    (property "Reference" "C23" (id 0) (at 166.37 86.7409 0)
+    (property "Reference" "EC11" (id 0) (at 166.37 86.7409 0)
       (effects (font (size 1.27 1.27)) (justify left))
     )

Commit message: Footprint associations complete
Parts:
- EC11: footprint Capacitor_SMD:CP_Elec_10x10 -> Capacitor_SMD:CP_Elec_6.3x7.7
Changed lines of the file:
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@@
       (effects (font (size 1.27 1.27)) (justify left))
     )
-    (property "Footprint" "Capacitor_SMD:CP_Elec_10x10" (id 2) (at 163.5252 92.71 0)
+    (property "Footprint" "Capacitor_SMD:CP_Elec_6.3x7.7" (id 2) (at 163.5252 92.71 0)
       (effects (font (size 1.27 1.27)) hide)
     )

Commit message: Started PCB layout
Parts:
- A4: value DRV8825 High Current Stepper Motor Driver Module -> DRV8825 Stepper Driver; footprint Module:Arduino_UNO_R3 -> Module:DRV8825 Stepper Motor Module
Changed lines of the file:
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@@
     (in_bom yes) (on_board yes) (fields_autoplaced)
     (property "Reference" "A4" (id 0) (at 125.095 77.47 0))
-    (property "Value" "DRV8825 High Current Stepper Motor Driver Module" (id 1) (at 125.095 80.01 0))
-    (property "Footprint" "Module:Arduino_UNO_R3" (id 2) (at 129.54 134.62 0)
+    (property "Value" "DRV8825 Stepper Driver" (id 1) (at 125.095 80.01 0))
+    (property "Footprint" "Module:DRV8825 Stepper Motor Module" (id 2) (at 129.54 134.62 0)
       (effects (font (size 1.27 1.27) italic) hide)
     )

Commit message: PCB layout
Parts:
- J19: footprint Connector_PinHeader_2.54mm:PinHeader_1x04_P2.54mm_Vertical -> Connector_JST:JST_XH_B4B-XH-A_1x04_P2.50mm_Vertical; symbol Connector:Conn_01x04_Male -> 000_Connectors_Immo:4_pin_JST_XH_male
Changed lines of the file:
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@@
     (pin "2")
   )
-  (symbol (lib_id "Connector:Conn_01x04_Male") (at 157.48 102.87 0) (mirror y) (unit 1)
+  (symbol (lib_id "000_Connectors_Immo:4_pin_JST_XH_male") (at 157.48 102.87 0) (mirror y) (unit 1)
     (in_bom yes) (on_board yes)
     (property "Reference" "J19" (id 0) (at 153.67 96.52 0)
@@
       (effects (font (size 1.27 1.27)) (justify right))
     )
-    (property "Footprint" "Connector_PinHeader_2.54mm:PinHeader_1x04_P2.54mm_Vertical" (id 2) (at 157.48 102.87 0)
+    (property "Footprint" "Connector_JST:JST_XH_B4B-XH-A_1x04_P2.50mm_Vertical" (id 2) (at 154.94 113.665 0)
       (effects (font (size 1.27 1.27)) hide)
     )
