File: RemoteLabs_supervisor_PCB/MCU_supervisor.kicad_sch (KiCad schematic)
At the start: 33 parts, among them J12 MCU_Header, J13 USB_B_Mini, J14 ShiftReg_Header, J15 SPI Supervisor, SW1 Stepper_Mode, SW3 Supervisor Reset, U6 ATSAMD21G18A-M, U7 4094, Y2 32.768 kHz

Commit message: Footprint associations complete
Parts:
- D9: footprint (none) -> Diode_SMD:D_0805_2012Metric_Pad1.15x1.40mm_HandSolder
- EC5, EC6: footprint Capacitor_SMD:CP_Elec_6.3x5.9 -> Capacitor_SMD:CP_Elec_4x5.4
- SW3: footprint (none) -> Button_Switch_SMD:SW_Push_1P1T_NO_CK_KSC6xxJ
- U7: footprint Package_DIP:SMDIP-18_W9.53mm -> Package_SO:SOIC-16_3.9x9.9mm_P1.27mm
Changed lines of the file:
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@@
       (effects (font (size 1.27 1.27)) (justify right))
     )
-    (property "Footprint" "" (id 2) (at 38.1 175.895 0)
+    (property "Footprint" "Button_Switch_SMD:SW_Push_1P1T_NO_CK_KSC6xxJ" (id 2) (at 38.1 175.895 0)
       (effects (font (size 1.27 1.27)) hide)
     )
@@
       (effects (font (size 1.27 1.27)) (justify right))
     )
-    (property "Footprint" "" (id 2) (at 161.925 173.99 0)
+    (property "Footprint" "Diode_SMD:D_0805_2012Metric_Pad1.15x1.40mm_HandSolder" (id 2) (at 161.925 173.99 0)
       (effects (font (size 1.27 1.27)) hide)
     )
@@
     (property "Reference" "EC5" (id 0) (at 83.439 39.37 90))
     (property "Value" "10u" (id 1) (at 83.439 41.91 90))
-    (property "Footprint" "Capacitor_SMD:CP_Elec_6.3x5.9" (id 2) (at 78.74 47.9552 0)
+    (property "Footprint" "Capacitor_SMD:CP_Elec_4x5.4" (id 2) (at 78.74 47.9552 0)
       (effects (font (size 1.27 1.27)) hide)
     )
@@
       (effects (font (size 1.27 1.27)) (justify left))
     )
-    (property "Footprint" "Package_DIP:SMDIP-18_W9.53mm" (id 2) (at 222.25 135.89 0)
+    (property "Footprint" "Package_SO:SOIC-16_3.9x9.9mm_P1.27mm" (id 2) (at 222.25 135.89 0)
       (effects (font (size 1.27 1.27)) hide)
     )
@@
     (property "Reference" "EC6" (id 0) (at 113.411 48.26 90))
     (property "Value" "10u" (id 1) (at 113.411 50.8 90))
-    (property "Footprint" "Capacitor_SMD:CP_Elec_6.3x5.9" (id 2) (at 118.11 54.9148 0)
-      (effects (font (size 1.27 1.27)) hide)
-    )
+    (property "Footprint" "Capacitor_SMD:CP_Elec_4x5.4" (id 2) (at 118.11 54.9148 0)
+      (effects (font (size 1.27 1.27)) hide)
+    )

Commit message: Started PCB layout
Parts:
- removed C14, C15: 9pF, Capacitor_SMD:C_0805_2012Metric_Pad1.18x1.45mm_HandSolder, symbol 000_Capacitor_Film_Immo:cap_film_0805_mini
- removed Y2: 32.768 kHz, Crystal:Crystal_SMD_SeikoEpson_MC405-2Pin_9.6x4.1mm_HandSoldering, symbol Device:Crystal_Small
- added C16: 100n, Capacitor_SMD:C_0805_2012Metric_Pad1.18x1.45mm_HandSolder, symbol 000_Capacitor_Film_Immo:cap_film_0805
- added C20: 10n, Capacitor_SMD:C_0805_2012Metric_Pad1.18x1.45mm_HandSolder, symbol 000_Capacitor_Film_Immo:cap_film_0805_mini
- added C23, C36: 12p, Capacitor_SMD:C_0805_2012Metric_Pad1.18x1.45mm_HandSolder, symbol 000_Capacitor_Film_Immo:cap_film_0805_mini
- added JP6, JP7, JP8: Xtal/IC, 000_Connectors_Immo:SolderJumper-3_P1.3mm_Bridged12_RoundedPad1.0x1.5mm_NumberLabels, symbol Jumper:SolderJumper_3_Bridged12
- added JP9: Reset Jumper, 000_Connectors_Immo:SolderJumper-2_P1.3mm_Open_Pad1.0x1.5mm, symbol Jumper:SolderJumper_2_Open
- added R41: 0r, Resistor_SMD:R_0805_2012Metric_Pad1.20x1.40mm_HandSolder, symbol 000_Resistors_Immo:Resistor_0805
- added U23: TCYSH14F, Package_TO_SOT_SMD:SOT-23-5_HandSoldering, symbol 74xGxx:SN74LVC1G14DBV
- added X2: ASEK-xxxMHz, Oscillator:Oscillator_SMD_Abracon_ASE-4Pin_3.2x2.5mm, symbol 000_Oscillator_Immo:ASEK-xxxMHz
Connections:
- net 3V3_DC_IN: now also C16.1, JP7.1 (A), U23.5 (VCC)
- net GND_D: now also C16.2, C20.2, C23.2, C36.2, JP7.3 (B), JP9.1 (A), U23.3 (GND), X2.2 (GND); no longer C1A1.2, C1B1.1, R1.1, R2.1, U6.40 (~{RESET})
- net HSE_OUT: now reaches U6.2 (PA01)
- net HSE_OUT: now also R41.2
- net HSE_IN: now reaches U6.1 (PA00)
- net HSE_IN: now also C23.1, JP6.3 (B), U23.4
- new net: C1A1.2, C1B1.1, JP9.2 (B), R1.1, R2.1, U6.40 (~{RESET})
- new net: JP8.1 (A), U23.2
- new net: JP8.2 (C), X2.3 (OUT)
- new net: C36.1, JP8.3 (B), R41.1
- new net: C20.1, JP6.1 (A), JP7.2 (C), X2.4 (Vdd)
- new net: JP6.2 (C), X2.1 (TRI)
Other:
- note added: "External Clock Package IC"
- note added: "For Osc IC - R? Unpopulated - C? & C? Unpopulated - C? ~ 10n - All Jumpers 2 - 1 For Xtal - R? = 0ohm to 47ohm - C? & C? Value = 2 *(Cxtal -Cstray) - All Jumpers 2 - 3 TCYSH14F - No Idea, probably omit for Xtal"
- note removed: "https://ww1.microchip.com/downloads/en/DeviceDoc/SAM_D21_DA1_Family_DataSheet_DS40001882F.pdf"
- moved on the sheet: A2, C13, C22, D4, D5, D9, J13, J14, J15, R10, R11, R39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

Commit message: PCB layout
Parts:
- removed JP8: Xtal/IC, 000_Connectors_Immo:SolderJumper-3_P1.3mm_Bridged12_RoundedPad1.0x1.5mm_NumberLabels, symbol Jumper:SolderJumper_3_Bridged12
- C17: footprint Capacitor_SMD:C_0805_2012Metric_Pad1.18x1.45mm_HandSolder -> Capacitor_Tantalum_SMD:CP_EIA-2012-12_Kemet-R_Pad1.30x1.05mm_HandSolder; symbol 000_Capacitor_Film_Immo:cap_film_0805 -> 000_Capacitor_Film_Immo:tantalum
Connections:
- net HSE_IN: no longer C23.1
- net at U23.2: now also C36.1, R41.1, X2.3 (OUT)
- net at JP6.2 (C), X2.1 (TRI): now also C23.1
Other:
- note added: "For Osc IC - R? Unpopulated - C? & C? Unpopulated - C? ~ 10n - All Jumpers 2 - 1 For Xtal - R? = 0ohm to 47ohm - C? & C? Value = 2 *(Cxtal -Cstray) - Omit C20 - All Jumpers 2 - 3 - TCYSH14F - No Idea, probably omit for Xtal"
- note removed: "For Osc IC - R? Unpopulated - C? & C? Unpopulated - C? ~ 10n - All Jumpers 2 - 1 For Xtal - R? = 0ohm to 47ohm - C? & C? Value = 2 *(Cxtal -Cstray) - All Jumpers 2 - 3 TCYSH14F - No Idea, probably omit for Xtal"
- moved on the sheet: C16, C23, JP6

Commit message: Edited PCB design for V1.1
- Changed pin sizes for stepper motor
- Change pin sizes for DC/DC Buck module.
- In process of changing text to be readable by human beings
Parts:
- JP9: value Reset Jumper -> Reset GND
- X2: value ASEK-xxxMHz -> 32.768kHz
Changed lines of the file:
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@@
       (effects (font (size 1.27 1.27)) (justify right))
     )
-    (property "Value" "Reset Jumper" (id 1) (at 49.53 183.515 90)
+    (property "Value" "Reset GND" (id 1) (at 49.53 183.515 90)
       (effects (font (size 1.27 1.27)) (justify right))
     )
@@
     (in_bom yes) (on_board yes)
     (property "Reference" "X2" (id 0) (at 170.815 76.835 0))
-    (property "Value" "ASEK-xxxMHz" (id 1) (at 175.895 74.295 0))
+    (property "Value" "32.768kHz" (id 1) (at 175.895 74.295 0))
     (property "Footprint" "Oscillator:Oscillator_SMD_Abracon_ASE-4Pin_3.2x2.5mm" (id 2) (at 184.15 106.045 0)
       (effects (font (size 1.27 1.27)) hide)

Commit message: Ahhhhhhhhhhhhhhh
Connections:
- net 3V3_DC_IN: now also R10.1, R11.1, R9.1; no longer SW1.4, SW1.5, SW1.6
- net GND_D: now also SW1.4, SW1.5, SW1.6; no longer R10.1, R11.1, R9.1
- net SHIFT_REG_7: no longer U7.11 (Q7)
- net STEPP_EN: now also U7.11 (Q7); no longer J14.6 (Pin_6), U7.13 (Q5)
- new net STEPP_SLP: J14.6 (Pin_6), U7.13 (Q5)
Other:
- note added: "DIGITAL IN"
Changed lines of the file:
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@@
   (junction (at 176.53 130.175) (diameter 0) (color 0 0 0 0)
   )
+  (junction (at 93.98 181.61) (diameter 0) (color 0 0 0 0)
+  )
   (junction (at 217.17 125.095) (diameter 0) (color 0 0 0 0)
-  )
-  (junction (at 93.98 181.61) (diameter 0) (color 0 0 0 0)
   )
   (junction (at 241.3 116.205) (diameter 0) (color 0 0 0 0)
@@
     (stroke (width 0) (type default) (color 0 0 0 0))
   )
+  (wire (pts (xy 182.88 139.065) (xy 182.88 140.335))
+    (stroke (width 0) (type default) (color 0 0 0 0))
+  )
   (wire (pts (xy 63.5 137.16) (xy 76.2 137.16))
     (stroke (width 0) (type default) (color 0 0 0 0))
@@
     (stroke (width 0) (type default) (color 0 0 0 0))
   )
+  (wire (pts (xy 217.17 122.555) (xy 217.17 125.095))
+    (stroke (width 0) (type default) (color 0 0 0 0))
+  )
   (wire (pts (xy 175.26 81.915) (xy 180.975 81.915))
     (stroke (width 0) (type default) (color 0 0 0 0))
@@
     (stroke (width 0) (type default) (color 0 0 0 0))
   )
+  (wire (pts (xy 182.88 140.335) (xy 182.88 142.24))
+    (stroke (width 0) (type default) (color 0 0 0 0))
+  )
   (wire (pts (xy 182.88 127.635) (xy 187.96 127.635))
     (stroke (width 0) (type default) (color 0 0 0 0))
@@
     (stroke (width 0) (type default) (color 0 0 0 0))
   )
-  (wire (pts (xy 182.88 139.065) (xy 182.88 140.335))
-    (stroke (width 0) (type default) (color 0 0 0 0))
-  )
   (wire (pts (xy 212.09 127.635) (xy 217.17 127.635))
     (stroke (width 0) (type default) (color 0 0 0 0))
@@
     (stroke (width 0) (type default) (color 0 0 0 0))
   )
-  (wire (pts (xy 182.88 140.335) (xy 182.88 142.875))
-    (stroke (width 0) (type default) (color 0 0 0 0))
-  )
   (polyline (pts (xy 168.91 95.885) (xy 193.04 95.885))
     (stroke (width 0) (type default) (color 0 0 0 0))
@@
     (stroke (width 0) (type default) (color 0 0 0 0))
   )
-  (wire (pts (xy 254 146.685) (xy 266.7 146.685))
-    (stroke (width 0) (type default) (color 0 0 0 0))
-  )
   (wire (pts (xy 32.385 20.955) (xy 32.385 22.225))
     (stroke (width 0) (type default) (color 0 0 0 0))
@@
     (stroke (width 0) (type default) (color 0 0 0 0))
   )
+  (wire (pts (xy 254 146.685) (xy 255.905 146.685))
+    (stroke (width 0) (type default) (color 0 0 0 0))
+  )
   (wire (pts (xy 180.975 75.565) (xy 188.595 75.565))
     (stroke (width 0) (type default) (color 0 0 0 0))
@@
   )
   (wire (pts (xy 93.98 71.12) (xy 93.98 73.66))
-    (stroke (width 0) (type default) (color 0 0 0 0))
-  )
-  (wire (pts (xy 223.52 125.095) (xy 217.17 125.095))
     (stroke (width 0) (type default) (color 0 0 0 0))
   )
@@
     (effects (font (size 1.27 1.27)) (justify left bottom))
   )
+  (text "DIGITAL IN" (at 201.93 58.42 180)
+    (effects (font (size 1.27 1.27)) (justify right bottom))
+  )
   (text "External Clock Package IC" (at 158.75 60.96 0)
     (effects (font (size 1.27 1.27)) (justify left bottom))
@@
     (effects (font (size 0.8 0.8)) (justify left bottom))
   )
+  (text "DIGITAL IN" (at 201.93 55.88 180)
+    (effects (font (size 1.27 1.27)) (justify right bottom))
+  )
   (text "SAMD21 BareMetal USB I/F" (at 21.59 18.415 0)
     (effects (font (size 1.27 1.27)) (justify left bottom))
+  )
+  (text "DIGITAL IN" (at 201.93 48.895 180)
+    (effects (font (size 1.27 1.27)) (justify right bottom))
   )
   (text "Replicates LED_BUILTIN\non Arduino Pin: D13" (at 173.355 163.195 0)
@@
     (effects (font (size 1.27 1.27)) (justify left bottom))
   )
+  (text "DIGITAL IN" (at 201.93 45.72 180)
+    (effects (font (size 1.27 1.27)) (justify right bottom))
+  )
   (text "place shiftreg header\nand MCU header together \n- Shorting the pins\nCH by CH avoids the need\nfor shift register if using\nraw MCU."
     (at 121.92 196.85 0)
@@
     (effects (font (size 1.27 1.27)) (justify left bottom))
   )
-  (label "SHIFT_REG_7" (at 266.7 146.685 180)
-    (effects (font (size 1.27 1.27)) (justify right bottom))
-  )
   (label "MOSI" (at 225.425 131.445 0)
     (effects (font (size 1.27 1.27)) (justify left bottom))
@@
     (effects (font (size 1.27 1.27)) (justify right))
   )
-  (hierarchical_label "STEPP_EN" (shape output) (at 132.715 178.435 0)
+  (hierarchical_label "STEPP_SLP" (shape output) (at 132.715 178.435 0)
     (effects (font (size 1.27 1.27)) (justify left))
   )
@@
     (effects (font (size 1.27 1.27)) (justify right))
   )
-  (hierarchical_label "GND_D" (shape passive) (at 182.88 142.875 270)
-    (effects (font (size 1.27 1.27)) (justify right))
+  (hierarchical_label "GND_D" (shape passive) (at 217.17 122.555 90)
+    (effects (font (size 1.27 1.27)) (justify left))
   )
   (hierarchical_label "MODE_2" (shape output) (at 173.99 130.175 180)
@@
     (effects (font (size 1.27 1.27)) (justify right))
   )
+  (hierarchical_label "STEPP_EN" (shape output) (at 255.905 146.685 0)
+    (effects (font (size 1.27 1.27)) (justify left))
+  )
   (hierarchical_label "PROG_TX" (shape output) (at 266.7 70.485 0)
     (effects (font (size 1.27 1.27)) (justify left))
@@
     (effects (font (size 1.27 1.27)) (justify right))
   )
-  (hierarchical_label "3V3_DC_IN" (shape input) (at 223.52 125.095 90)
-    (effects (font (size 1.27 1.27)) (justify left))
+  (hierarchical_label "3V3_DC_IN" (shape input) (at 182.88 142.24 270)
+    (effects (font (size 1.27 1.27)) (justify right))
   )
   (hierarchical_label "STEPP_FLT" (shape input) (at 223.52 45.085 180)
     (effects (font (size 1.27 1.27)) (justify right))
   )
-  (hierarchical_label "STEPP_EN" (shape output) (at 255.905 141.605 0)
-    (effects (font (size 1.27 1.27)) (justify left))
-  )
+  (hierarchical_label "STEPP_SLP" (shape output) (at 255.905 141.605 0)
+    (effects (font (size 1.27 1.27)) (justify left))
+  )

Commit message: Version 1.2 PCB
Parts:
- added N1: Net_Tie, NetTie:NetTie-2_SMD_Pad0.5mm, symbol 000_Utility_Immo:Net_Tie
Connections:
- net SHIFT_REG_7 is gone; now on net STEPP_EN: J14.8 (Pin_8)
- net GND_D: no longer SW1.4, SW1.5, SW1.6
- new net: N1.1 (A), SW1.4, SW1.5, SW1.6
- new net GND_P: N1.2 (C)
Other:
- moved on the sheet: C22, U7

Commit message: Everything
Other:
- note added: "For Osc IC - R41 Unpopulated - C23 & C36 Unpopulated - C20 ~ 10n - All Jumpers 2 - 1 For Xtal - R? = 0ohm to 47ohm - C? & C? Value = 2 *(Cxtal -Cstray) - Omit C20 - All Jumpers 2 - 3 - TCYSH14F - No Idea, probably omit for Xtal"
- note removed: "For Osc IC - R? Unpopulated - C? & C? Unpopulated - C? ~ 10n - All Jumpers 2 - 1 For Xtal - R? = 0ohm to 47ohm - C? & C? Value = 2 *(Cxtal -Cstray) - Omit C20 - All Jumpers 2 - 3 - TCYSH14F - No Idea, probably omit for Xtal"
Changed lines of the file:
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@@
     (effects (font (size 1.27 1.27)) (justify left bottom))
   )
-  (text "For Osc IC\n- R? Unpopulated\n- C? & C? Unpopulated\n- C? ~ 10n\n- All Jumpers 2 - 1\n\nFor Xtal\n- R? = 0ohm to 47ohm \n- C? & C? Value = 2 *(Cxtal -Cstray)\n- Omit C20\n- All Jumpers 2 - 3\n- TCYSH14F - No Idea, probably omit for Xtal"
+  (text "For Osc IC\n- R41 Unpopulated\n- C23 & C36 Unpopulated\n- C20 ~ 10n\n- All Jumpers 2 - 1\n\nFor Xtal\n- R? = 0ohm to 47ohm \n- C? & C? Value = 2 *(Cxtal -Cstray)\n- Omit C20\n- All Jumpers 2 - 3\n- TCYSH14F - No Idea, probably omit for Xtal"
     (at 172.72 113.03 0)
     (effects (font (size 0.8 0.8)) (justify left bottom))
