File: RemoteLabs_supervisor_PCB/analog_signal_buffers.kicad_sch (KiCad schematic)
At the start: 18 parts

Commit message: adding test sketch
Connections:
- net 5V_VCC renamed VCC
Changed lines of the file:
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@@
     (effects (font (size 1.27 1.27)) (justify left bottom))
   )
-  (hierarchical_label "5V_VCC" (shape input) (at 241.3 33.02 90)
+  (hierarchical_label "VCC" (shape input) (at 241.3 33.02 90)
     (effects (font (size 1.27 1.27)) (justify left))
   )

Commit message: sdf
Connections:
- net GND_D renamed GND_A
Changed lines of the file:
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@@
     (effects (font (size 1.27 1.27)) (justify left))
   )
-  (hierarchical_label "GND_D" (shape input) (at 241.3 59.69 270)
+  (hierarchical_label "GND_A" (shape passive) (at 241.3 59.69 270)
     (effects (font (size 1.27 1.27)) (justify right))
   )

Commit message: V1.0 Circuit Design Complete
Parts:
- gave numbers to parts that had none: 6
Connections:
- net A_IN_B: now also U23.5 (+); no longer U23.12 (+)
- net A_IN_D: now also U23.12 (+); no longer U23.5 (+)
- net A_OUT_A1: now also U24.1, U24.2 (-); no longer U24.6 (-), U24.7
- net A_OUT_A2: now also U24.6 (-), U24.7; no longer U24.8, U24.9 (-)
- net A_OUT_B1: now also U24.8, U24.9 (-); no longer U24.1, U24.2 (-)
- net A_OUT_B2: now also U24.13 (-), U24.14; no longer U24.6 (-), U24.7
- net A_OUT_C1: now also U25.1, U25.2 (-); no longer U25.13 (-), U25.14
- net A_OUT_C2: now also U25.6 (-), U25.7; no longer U25.1, U25.2 (-)
- net at U23.8, U23.9 (-): now also U25.3 (+), U25.5 (+); no longer U25.12 (+), U25.3 (+)
- net at U23.1, U23.2 (-): now also U24.3 (+), U24.5 (+); no longer U24.10 (+), U24.5 (+)
- net at U25.10 (+), U25.12 (+): now also U23.13 (-), U23.14; no longer U23.6 (-), U23.7
- new net: U23.6 (-), U23.7, U24.10 (+), U24.12 (+)

Commit message: Schematic reviewed
Parts:
- U23, U24, U25: footprint (none) -> Package_DIP:SMDIP-14_W9.53mm
Changed lines of the file:
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@@
     (pin "2")
   )
-  (symbol (lib_id "Amplifier_Operational:TL074") (at 110.49 119.38 0) (unit 1)
+  (symbol (lib_name "TL074_6") (lib_id "Amplifier_Operational:TL074") (at 110.49 119.38 0) (unit 1)
     (in_bom yes) (on_board yes)
     (property "Reference" "U25" (id 0) (at 110.49 109.22 0))
     (property "Value" "TL074" (id 1) (at 110.49 111.76 0))
-    (property "Footprint" "" (id 2) (at 109.22 116.84 0)
+    (property "Footprint" "Package_DIP:SMDIP-14_W9.53mm" (id 2) (at 109.22 116.84 0)
       (effects (font (size 1.27 1.27)) hide)
     )
@@
     (pin "3")
   )
-  (symbol (lib_id "Amplifier_Operational:TL074") (at 110.49 138.43 0) (unit 2)
+  (symbol (lib_name "TL074_4") (lib_id "Amplifier_Operational:TL074") (at 110.49 138.43 0) (unit 2)
     (in_bom yes) (on_board yes) (fields_autoplaced)
     (property "Reference" "U25" (id 0) (at 110.49 128.27 0))
     (property "Value" "TL074" (id 1) (at 110.49 130.81 0))
-    (property "Footprint" "" (id 2) (at 109.22 135.89 0)
+    (property "Footprint" "Package_DIP:SMDIP-14_W9.53mm" (id 2) (at 109.22 135.89 0)
       (effects (font (size 1.27 1.27)) hide)
     )
@@
     (property "Reference" "U24" (id 0) (at 109.22 21.59 0))
     (property "Value" "TL074" (id 1) (at 110.49 24.13 0))
-    (property "Footprint" "" (id 2) (at 109.22 29.21 0)
+    (property "Footprint" "Package_DIP:SMDIP-14_W9.53mm" (id 2) (at 109.22 29.21 0)
       (effects (font (size 1.27 1.27)) hide)
     )
@@
     (pin "3")
   )
-  (symbol (lib_id "Amplifier_Operational:TL074") (at 77.47 39.37 0) (unit 1)
+  (symbol (lib_name "TL074_9") (lib_id "Amplifier_Operational:TL074") (at 77.47 39.37 0) (unit 1)
     (in_bom yes) (on_board yes) (fields_autoplaced)
     (property "Reference" "U23" (id 0) (at 77.47 29.21 0))
     (property "Value" "TL074" (id 1) (at 77.47 31.75 0))
-    (property "Footprint" "" (id 2) (at 76.2 36.83 0)
+    (property "Footprint" "Package_DIP:SMDIP-14_W9.53mm" (id 2) (at 76.2 36.83 0)
       (effects (font (size 1.27 1.27)) hide)
     )
@@
     (pin "3")
   )
-  (symbol (lib_id "Amplifier_Operational:TL074") (at 110.49 50.8 0) (unit 2)
+  (symbol (lib_name "TL074_12") (lib_id "Amplifier_Operational:TL074") (at 110.49 50.8 0) (unit 2)
     (in_bom yes) (on_board yes) (fields_autoplaced)
     (property "Reference" "U24" (id 0) (at 110.49 40.64 0))
     (property "Value" "TL074" (id 1) (at 110.49 43.18 0))
-    (property "Footprint" "" (id 2) (at 109.22 48.26 0)
+    (property "Footprint" "Package_DIP:SMDIP-14_W9.53mm" (id 2) (at 109.22 48.26 0)
       (effects (font (size 1.27 1.27)) hide)
     )
@@
     (pin "7")
   )
-  (symbol (lib_id "Amplifier_Operational:TL074") (at 227.33 46.99 0) (unit 5)
+  (symbol (lib_name "TL074_3") (lib_id "Amplifier_Operational:TL074") (at 227.33 46.99 0) (unit 5)
     (in_bom yes) (on_board yes) (fields_autoplaced)
     (property "Reference" "U23" (id 0) (at 226.06 45.7199 0)
@@
       (effects (font (size 1.27 1.27)) (justify left))
     )
-    (property "Footprint" "" (id 2) (at 226.06 44.45 0)
+    (property "Footprint" "Package_DIP:SMDIP-14_W9.53mm" (id 2) (at 226.06 44.45 0)
       (effects (font (size 1.27 1.27)) hide)
     )
@@
     (pin "4")
   )
-  (symbol (lib_id "Amplifier_Operational:TL074") (at 77.47 168.91 0) (unit 4)
+  (symbol (lib_name "TL074_13") (lib_id "Amplifier_Operational:TL074") (at 77.47 168.91 0) (unit 4)
     (in_bom yes) (on_board yes) (fields_autoplaced)
     (property "Reference" "U23" (id 0) (at 77.47 158.75 0))
     (property "Value" "TL074" (id 1) (at 77.47 161.29 0))
-    (property "Footprint" "" (id 2) (at 76.2 166.37 0)
+    (property "Footprint" "Package_DIP:SMDIP-14_W9.53mm" (id 2) (at 76.2 166.37 0)
       (effects (font (size 1.27 1.27)) hide)
     )
@@
     (pin "14")
   )
-  (symbol (lib_id "Amplifier_Operational:TL074") (at 246.38 46.99 0) (unit 5)
+  (symbol (lib_name "TL074_1") (lib_id "Amplifier_Operational:TL074") (at 246.38 46.99 0) (unit 5)
     (in_bom yes) (on_board yes) (fields_autoplaced)
     (property "Reference" "U24" (id 0) (at 245.11 45.7199 0)
@@
       (effects (font (size 1.27 1.27)) (justify left))
     )
-    (property "Footprint" "" (id 2) (at 245.11 44.45 0)
+    (property "Footprint" "Package_DIP:SMDIP-14_W9.53mm" (id 2) (at 245.11 44.45 0)
       (effects (font (size 1.27 1.27)) hide)
     )
@@
     (pin "4")
   )
-  (symbol (lib_id "Amplifier_Operational:TL074") (at 77.47 82.55 0) (unit 2)
+  (symbol (lib_name "TL074_11") (lib_id "Amplifier_Operational:TL074") (at 77.47 82.55 0) (unit 2)
     (in_bom yes) (on_board yes) (fields_autoplaced)
     (property "Reference" "U23" (id 0) (at 77.47 72.39 0))
     (property "Value" "TL074" (id 1) (at 77.47 74.93 0))
-    (property "Footprint" "" (id 2) (at 76.2 80.01 0)
+    (property "Footprint" "Package_DIP:SMDIP-14_W9.53mm" (id 2) (at 76.2 80.01 0)
       (effects (font (size 1.27 1.27)) hide)
     )
@@
     (pin "7")
   )
-  (symbol (lib_id "Amplifier_Operational:TL074") (at 110.49 161.29 0) (unit 3)
+  (symbol (lib_name "TL074_5") (lib_id "Amplifier_Operational:TL074") (at 110.49 161.29 0) (unit 3)
     (in_bom yes) (on_board yes) (fields_autoplaced)
     (property "Reference" "U25" (id 0) (at 110.49 151.13 0))
     (property "Value" "TL074" (id 1) (at 110.49 153.67 0))
-    (property "Footprint" "" (id 2) (at 109.22 158.75 0)
+    (property "Footprint" "Package_DIP:SMDIP-14_W9.53mm" (id 2) (at 109.22 158.75 0)
       (effects (font (size 1.27 1.27)) hide)
     )
@@
     (pin "2")
   )
-  (symbol (lib_id "Amplifier_Operational:TL074") (at 77.47 127 0) (unit 3)
+  (symbol (lib_name "TL074_7") (lib_id "Amplifier_Operational:TL074") (at 77.47 127 0) (unit 3)
     (in_bom yes) (on_board yes) (fields_autoplaced)
     (property "Reference" "U23" (id 0) (at 77.47 116.84 0))
     (property "Value" "TL074" (id 1) (at 77.47 119.38 0))
-    (property "Footprint" "" (id 2) (at 76.2 124.46 0)
+    (property "Footprint" "Package_DIP:SMDIP-14_W9.53mm" (id 2) (at 76.2 124.46 0)
       (effects (font (size 1.27 1.27)) hide)
     )
@@
     (pin "9")
   )
-  (symbol (lib_id "Amplifier_Operational:TL074") (at 265.43 46.99 0) (unit 5)
+  (symbol (lib_name "TL074_2") (lib_id "Amplifier_Operational:TL074") (at 265.43 46.99 0) (unit 5)
     (in_bom yes) (on_board yes) (fields_autoplaced)
     (property "Reference" "U25" (id 0) (at 264.16 45.7199 0)
@@
       (effects (font (size 1.27 1.27)) (justify left))
     )
-    (property "Footprint" "" (id 2) (at 264.16 44.45 0)
+    (property "Footprint" "Package_DIP:SMDIP-14_W9.53mm" (id 2) (at 264.16 44.45 0)
       (effects (font (size 1.27 1.27)) hide)
     )
@@
     (pin "4")
   )
-  (symbol (lib_id "Amplifier_Operational:TL074") (at 110.49 93.98 0) (unit 4)
+  (symbol (lib_name "TL074_8") (lib_id "Amplifier_Operational:TL074") (at 110.49 93.98 0) (unit 4)
     (in_bom yes) (on_board yes) (fields_autoplaced)
     (property "Reference" "U24" (id 0) (at 110.49 83.82 0))
     (property "Value" "TL074" (id 1) (at 110.49 86.36 0))
-    (property "Footprint" "" (id 2) (at 109.22 91.44 0)
+    (property "Footprint" "Package_DIP:SMDIP-14_W9.53mm" (id 2) (at 109.22 91.44 0)
       (effects (font (size 1.27 1.27)) hide)
     )
@@
     (pin "14")
   )
-  (symbol (lib_id "Amplifier_Operational:TL074") (at 110.49 180.34 0) (unit 4)
+  (symbol (lib_name "TL074_14") (lib_id "Amplifier_Operational:TL074") (at 110.49 180.34 0) (unit 4)
     (in_bom yes) (on_board yes) (fields_autoplaced)
     (property "Reference" "U25" (id 0) (at 110.49 170.18 0))
     (property "Value" "TL074" (id 1) (at 110.49 172.72 0))
-    (property "Footprint" "" (id 2) (at 109.22 177.8 0)
+    (property "Footprint" "Package_DIP:SMDIP-14_W9.53mm" (id 2) (at 109.22 177.8 0)
       (effects (font (size 1.27 1.27)) hide)
     )
@@
     (pin "14")
   )
-  (symbol (lib_id "Amplifier_Operational:TL074") (at 110.49 74.93 0) (unit 3)
+  (symbol (lib_name "TL074_10") (lib_id "Amplifier_Operational:TL074") (at 110.49 74.93 0) (unit 3)
     (in_bom yes) (on_board yes) (fields_autoplaced)
     (property "Reference" "U24" (id 0) (at 110.49 64.77 0))
     (property "Value" "TL074" (id 1) (at 110.49 67.31 0))
-    (property "Footprint" "" (id 2) (at 109.22 72.39 0)
-      (effects (font (size 1.27 1.27)) hide)
-    )
+    (property "Footprint" "Package_DIP:SMDIP-14_W9.53mm" (id 2) (at 109.22 72.39 0)
+      (effects (font (size 1.27 1.27)) hide)
+    )

Commit message: mbncmvbc,
Parts:
- removed U23, U24, U25: TL074, Package_DIP:SMDIP-14_W9.53mm, symbol Amplifier_Operational:TL074
- added R32, R33, R34, R35: 1k, Resistor_SMD:R_0805_2012Metric_Pad1.20x1.40mm_HandSolder, symbol 000_Resistors_Immo:Resistor_0805
- added U15, U16, U17: NCS20074D, Package_SO:SOIC-14_3.9x8.7mm_P1.27mm, symbol Amplifier_Operational:NCS20074D
Connections:
- net A_IN_A: now also U15.3 (+)
- net A_IN_B: now also U15.5 (+)
- net A_IN_C: now also U15.10 (+)
- net A_IN_D: now also U15.12 (+)
- net A_OUT_A1: now also U16.1, U16.2 (-)
- net A_OUT_A2: now also R34.1
- net A_OUT_B1: now also U16.6 (-), U16.7
- net A_OUT_B2: now also R32.1
- net A_OUT_C1: now also U16.8, U16.9 (-)
- net A_OUT_C2: now also R35.1
- net A_OUT_D1: now also U16.13 (-), U16.14
- net A_OUT_D2: now also R33.1
- net GND_A: now also U15.11 (V-), U16.11 (V-), U17.11 (V-)
- net VCC: now also U15.4 (V+), U16.4 (V+), U17.4 (V+)
- new net: U15.6 (-), U15.7, U16.5 (+), U17.5 (+)
- new net: U15.13 (-), U15.14, U16.12 (+), U17.12 (+)
- new net: R32.2, U17.6 (-), U17.7
- new net: U15.1, U15.2 (-), U16.3 (+), U17.3 (+)
- new net: U15.8, U15.9 (-), U16.10 (+), U17.10 (+)
- new net: R34.2, U17.1, U17.2 (-)
- new net: R33.2, U17.13 (-), U17.14
- new net: R35.2, U17.8, U17.9 (-)

Commit message: Footprint associations complete
Connections:
- net DB2: now reaches U15.6 (-), U15.7, U16.5 (+), U17.5 (+)
- net DB4: now reaches U15.13 (-), U15.14, U16.12 (+), U17.12 (+)
- net DB2B: now reaches R32.2, U17.6 (-), U17.7
- net DB1: now reaches U15.1, U15.2 (-), U16.3 (+), U17.3 (+)
- net DB3: now reaches U15.8, U15.9 (-), U16.10 (+), U17.10 (+)
- net DB1B: now reaches R34.2, U17.1, U17.2 (-)
- net DB4B: now reaches R33.2, U17.13 (-), U17.14
- net DB3B: now reaches R35.2, U17.8, U17.9 (-)
Changed lines of the file:
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@@
+    (effects (font (size 1.27 1.27)) (justify left bottom))
+  )
+  (label "DB1B" (at 113.665 58.42 0)
+    (effects (font (size 1.27 1.27)) (justify left bottom))
+  )
+  (label "DB4" (at 92.71 158.75 0)
+    (effects (font (size 1.27 1.27)) (justify left bottom))
+  )
+  (label "DB2" (at 91.44 72.39 0)
+    (effects (font (size 1.27 1.27)) (justify left bottom))
+  )
+  (label "DB3" (at 92.71 116.84 0)
+    (effects (font (size 1.27 1.27)) (justify left bottom))
+  )
+  (label "DB3B" (at 113.03 146.05 0)
+    (effects (font (size 1.27 1.27)) (justify left bottom))
+  )
+  (label "DB2B" (at 114.3 101.6 0)
+    (effects (font (size 1.27 1.27)) (justify left bottom))
+  )
+  (label "DB4B" (at 113.665 189.23 0)
+    (effects (font (size 1.27 1.27)) (justify left bottom))
+  )
+  (label "DB1" (at 92.075 29.21 0)
     (effects (font (size 1.27 1.27)) (justify left bottom))
   )
