File: pendulum_daughterboard/Driver PCB/LED_Circuit.kicad_sch (KiCad schematic)
At the start: 15 parts, among them IC1 AND GATES, IC2 NAND (Used as AND), IC3 NAND (Used as Inverter), IC4 OR, J4 Conn_01x04

Commit message: Today's Progress on the PCB
22/06/22
Connections:
- net ENABLE is gone; now on net STUDENT_ENABLE: IC1.13 (4B)
- net GND: now also J4.1 (Pin_1); no longer J4.4 (Pin_4)
- net OR_OUT_1: now also J4.4 (Pin_4); no longer J4.1 (Pin_1)
- net OR_OUT_2: now also J4.3 (Pin_3); no longer J4.2 (Pin_2)
- net OR_OUT_3: now also J4.2 (Pin_2); no longer J4.3 (Pin_3)
Other:
- moved on the sheet: D1, D2, D3, J4, R1, R2, R3
