File: pendulum_daughterboard/Driver PCB/Microcontroller_Circuit_sch.kicad_sch (KiCad schematic)
At the start: 11 parts, among them J1 AVR-ISP-6, J2 Conn_01x02_Female, Q1 BC557, Q2 BC547, SW1 SW_Push, U10 ATtiny85-20S

Commit message: Today's Progress on the PCB
22/06/22
Parts:
- removed D4: D, Diode_SMD:D_0603_1608Metric_Pad1.05x0.95mm_HandSolder, symbol Simulation_SPICE:DIODE
- removed J2: Conn_01x02_Female, Connector_PinHeader_2.00mm:PinHeader_1x02_P2.00mm_Horizontal, symbol Connector:Conn_01x02_Female
- removed Q1: BC557, Package_TO_SOT_SMD:SOT-523, symbol Transistor_BJT:BC557
- removed Q2: BC547, Package_TO_SOT_SMD:SOT-523, symbol Transistor_BJT:BC547
- removed R4, R5: 2k2, Resistor_SMD:R_0805_2012Metric_Pad1.20x1.40mm_HandSolder, symbol Device:R
Connections:
- net DRIVE_ENABLE renamed DRIVE
Other:
- moved on the sheet: C8, J1, R6, SW1, U10

Commit message: changes
11.50
Parts:
- removed SW1: SW_Push, Button_Switch_SMD:Panasonic_EVQPUK_EVQPUB, symbol Switch:SW_Push
- added SW1: SW_Push, Button_Switch_SMD:13019319, symbol Switch:SW_Push_Dual
Connections:
- net GND: now also SW1.1, SW1.2
- net at J1.5 (~{RST}), R6.1, U10.1 (~{RESET}/PB5): now also SW1.3, SW1.4
Changed lines of the file:
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@@
   (junction (at 146.05 82.55) (diameter 0) (color 0 0 0 0)
   )
+  (junction (at 128.27 113.03) (diameter 0) (color 0 0 0 0)
+  )
   (junction (at 146.05 50.8) (diameter 0) (color 0 0 0 0)
   )
-  (junction (at 143.51 125.73) (diameter 0) (color 0 0 0 0)
+  (junction (at 113.03 113.03) (diameter 0) (color 0 0 0 0)
+  )
+  (junction (at 143.51 151.13) (diameter 0) (color 0 0 0 0)
   )
   (junction (at 137.16 101.6) (diameter 0) (color 0 0 0 0)
@@
     (stroke (width 0) (type default) (color 0 0 0 0))
   )
+  (wire (pts (xy 104.14 104.14) (xy 104.14 113.03))
+    (stroke (width 0) (type default) (color 0 0 0 0))
+  )
+  (wire (pts (xy 190.5 102.87) (xy 190.5 151.13))
+    (stroke (width 0) (type default) (color 0 0 0 0))
+  )
   (wire (pts (xy 151.13 85.09) (xy 175.26 85.09))
     (stroke (width 0) (type default) (color 0 0 0 0))
@@
     (stroke (width 0) (type default) (color 0 0 0 0))
   )
-  (wire (pts (xy 143.51 125.73) (xy 190.5 125.73))
+  (wire (pts (xy 137.16 113.03) (xy 144.78 113.03))
+    (stroke (width 0) (type default) (color 0 0 0 0))
+  )
+  (wire (pts (xy 143.51 151.13) (xy 190.5 151.13))
+    (stroke (width 0) (type default) (color 0 0 0 0))
+  )
+  (wire (pts (xy 128.27 107.95) (xy 128.27 113.03))
     (stroke (width 0) (type default) (color 0 0 0 0))
   )
@@
     (stroke (width 0) (type default) (color 0 0 0 0))
   )
-  (wire (pts (xy 100.33 100.33) (xy 100.33 125.73))
+  (wire (pts (xy 128.27 113.03) (xy 128.27 118.11))
+    (stroke (width 0) (type default) (color 0 0 0 0))
+  )
+  (wire (pts (xy 100.33 100.33) (xy 100.33 151.13))
     (stroke (width 0) (type default) (color 0 0 0 0))
   )
@@
     (stroke (width 0) (type default) (color 0 0 0 0))
   )
+  (wire (pts (xy 113.03 118.11) (xy 119.38 118.11))
+    (stroke (width 0) (type default) (color 0 0 0 0))
+  )
+  (wire (pts (xy 113.03 107.95) (xy 119.38 107.95))
+    (stroke (width 0) (type default) (color 0 0 0 0))
+  )
+  (wire (pts (xy 113.03 113.03) (xy 113.03 118.11))
+    (stroke (width 0) (type default) (color 0 0 0 0))
+  )
   (wire (pts (xy 100.33 77.47) (xy 100.33 50.8))
     (stroke (width 0) (type default) (color 0 0 0 0))
@@
     (stroke (width 0) (type default) (color 0 0 0 0))
   )
+  (wire (pts (xy 124.46 107.95) (xy 128.27 107.95))
+    (stroke (width 0) (type default) (color 0 0 0 0))
+  )
   (wire (pts (xy 137.16 101.6) (xy 175.26 101.6))
     (stroke (width 0) (type default) (color 0 0 0 0))
   )
-  (wire (pts (xy 190.5 125.73) (xy 190.5 102.87))
-    (stroke (width 0) (type default) (color 0 0 0 0))
-  )
-  (wire (pts (xy 143.51 125.73) (xy 143.51 128.27))
+  (wire (pts (xy 143.51 151.13) (xy 143.51 153.67))
     (stroke (width 0) (type default) (color 0 0 0 0))
   )
@@
     (stroke (width 0) (type default) (color 0 0 0 0))
   )
+  (wire (pts (xy 128.27 118.11) (xy 124.46 118.11))
+    (stroke (width 0) (type default) (color 0 0 0 0))
+  )
+  (wire (pts (xy 104.14 113.03) (xy 113.03 113.03))
+    (stroke (width 0) (type default) (color 0 0 0 0))
+  )
   (wire (pts (xy 152.4 113.03) (xy 158.75 113.03))
     (stroke (width 0) (type default) (color 0 0 0 0))
   )
+  (wire (pts (xy 128.27 113.03) (xy 137.16 113.03))
+    (stroke (width 0) (type default) (color 0 0 0 0))
+  )
   (wire (pts (xy 146.05 63.5) (xy 146.05 66.04))
     (stroke (width 0) (type default) (color 0 0 0 0))
@@
     (stroke (width 0) (type default) (color 0 0 0 0))
   )
+  (wire (pts (xy 113.03 113.03) (xy 113.03 107.95))
+    (stroke (width 0) (type default) (color 0 0 0 0))
+  )
   (wire (pts (xy 124.46 85.09) (xy 124.46 82.55))
     (stroke (width 0) (type default) (color 0 0 0 0))
   )
-  (wire (pts (xy 137.16 113.03) (xy 144.78 113.03))
-    (stroke (width 0) (type default) (color 0 0 0 0))
-  )
   (wire (pts (xy 146.05 80.01) (xy 146.05 82.55))
     (stroke (width 0) (type default) (color 0 0 0 0))
@@
     (stroke (width 0) (type default) (color 0 0 0 0))
   )
-  (wire (pts (xy 123.19 113.03) (xy 124.46 113.03))
-    (stroke (width 0) (type default) (color 0 0 0 0))
-  )
-  (wire (pts (xy 134.62 113.03) (xy 137.16 113.03))
-    (stroke (width 0) (type default) (color 0 0 0 0))
-  )
   (wire (pts (xy 137.16 101.6) (xy 137.16 113.03))
     (stroke (width 0) (type default) (color 0 0 0 0))
@@
     (stroke (width 0) (type default) (color 0 0 0 0))
   )
-  (wire (pts (xy 100.33 125.73) (xy 143.51 125.73))
-    (stroke (width 0) (type default) (color 0 0 0 0))
-  )
-  (hierarchical_label "GND" (shape input) (at 123.19 113.03 180)
-    (effects (font (size 1.27 1.27)) (justify right))
+  (wire (pts (xy 100.33 151.13) (xy 143.51 151.13))
+    (stroke (width 0) (type default) (color 0 0 0 0))
+  )
+  (hierarchical_label "GND" (shape input) (at 104.14 104.14 90)
+    (effects (font (size 1.27 1.27)) (justify left))
   )
   (hierarchical_label "DRIVE_MCU" (shape output) (at 168.91 90.17 180)
     (effects (font (size 1.27 1.27)) (justify right))
   )
-  (hierarchical_label "GND" (shape input) (at 143.51 128.27 270)
+  (hierarchical_label "GND" (shape input) (at 143.51 153.67 270)
     (effects (font (size 1.27 1.27)) (justify right))
   )
@@
     (pin "2")
   )
+  (symbol (lib_id "Switch:SW_Push_Dual") (at 119.38 113.03 90) (unit 1)
+    (in_bom yes) (on_board yes)
+    (property "Reference" "SW1" (id 0) (at 119.38 104.14 90)
+      (effects (font (size 1.27 1.27)) (justify right))
+    )
+    (property "Value" "SW_Push" (id 1) (at 116.84 106.68 90)
+      (effects (font (size 1.27 1.27)) (justify right))
+    )
+    (property "Footprint" "Button_Switch_SMD:13019319" (id 2) (at 114.3 113.03 0)
+      (effects (font (size 1.27 1.27)) hide)
+    )
+    (property "Datasheet" "~" (id 3) (at 114.3 113.03 0)
+      (effects (font (size 1.27 1.27)) hide)
+    )
+    (pin "1")
+    (pin "2")
+    (pin "3")
+    (pin "4")
+  )
   (symbol (lib_id "Connector:AVR-ISP-6") (at 102.87 90.17 0) (unit 1)
     (in_bom yes) (on_board yes) (fields_autoplaced)
@@
       (effects (font (size 1.27 1.27)) hide)
     )
-    (pin "1")
-    (pin "2")
-  )
-  (symbol (lib_id "Switch:SW_Push") (at 129.54 113.03 0) (unit 1)
-    (in_bom yes) (on_board yes) (fields_autoplaced)
-    (property "Reference" "SW1" (id 0) (at 129.54 105.41 0))
-    (property "Value" "SW_Push" (id 1) (at 129.54 107.95 0))
-    (property "Footprint" "Button_Switch_SMD:Panasonic_EVQPUK_EVQPUB" (id 2) (at 129.54 107.95 0)
-      (effects (font (size 1.27 1.27)) hide)
-    )
-    (property "Datasheet" "~" (id 3) (at 129.54 107.95 0)
-      (effects (font (size 1.27 1.27)) hide)
-    )
