File: pendulum_daughterboard/Driver PCB/Driver PCB.kicad_sch (KiCad schematic)
At the start: 6 parts, among them J5 GND, J7 5V

Commit message: Today's Progress on the PCB
22/06/22
Parts:
- J5: value GND -> DRIVE_GND
- J7: value 5V -> DRIVE_5V_IN
Connections:
- net CURRENT_SIGN_OUT: now reaches A1.10 (IS_2)
- net D_5V: now reaches A1.5 (5V)
- net D_GND: now reaches A1.7 (GND)
- net CURRENT_SENSE_OUT: now reaches A1.9 (IS_1)
- net 5V renamed DRIVE_5V
- net DRIVE_5V: no longer A1.36 (M_GND)
- net DRIVE renamed DRIVE_INPUT
- net GND renamed DRIVE_GND
- net DRIVE_GND: no longer A1.33 (PWRGND)
- net LOAD renamed LOAD_INPUT
- no-connect marks 14 -> 12
Other:
- added sheet Drive Circuit (Drive_Circuit.kicad_sch)
- sheet LED_Circit ports: added STUDENT_ENABLE; removed ENABLE
- sheet Microcontroller Circuit ports: added DRIVE, DRIVE_MCU, LOAD_MCU; removed DRIVE_ENABLE
- note added: "Capacitors to supply current to the Coil"
- moved on the sheet: C1, C2, C3, J5, J7
