File: pendulum_daughterboard/Driver PCB/_autosave-Drive_Circuit.kicad_sch (KiCad schematic)
At the start: 17 parts, among them IC5 MAX9928FAUA+, J2 Coil, Q1 BC557, Q2 BC547

Commit message: Penduino Daughterboard Update
The complete design before checks.
Parts:
- removed NT12: NetTie_2, NetTie:NetTie-2_SMD_Pad0.5mm, symbol Device:NetTie_2
Connections:
- net DRIVE_GND: now also Q2.3 (E)
Changed lines of the file:
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@@
     (stroke (width 0) (type default) (color 0 0 0 0))
   )
-  (wire (pts (xy 119.2062 110.49) (xy 113.03 110.49))
+  (wire (pts (xy 113.03 110.49) (xy 133.35 110.49))
     (stroke (width 0) (type default) (color 0 0 0 0))
   )
@@
     (stroke (width 0) (type default) (color 0 0 0 0))
   )
-  (wire (pts (xy 133.35 110.49) (xy 124.2862 110.49))
-    (stroke (width 0) (type default) (color 0 0 0 0))
-  )
   (hierarchical_label "D_GND" (shape input) (at 269.24 77.47 0)
     (effects (font (size 1.27 1.27)) (justify left))
@@
     (effects (font (size 1.27 1.27)) (justify right))
   )
-  (symbol (lib_id "Device:NetTie_2") (at 121.7462 110.49 0) (unit 1)
-    (in_bom yes) (on_board yes)
-    (property "Reference" "NT12" (id 0) (at 120.4762 109.22 0))
-    (property "Value" "NetTie_2" (id 1) (at 121.8031 105.41 0))
-    (property "Footprint" "NetTie:NetTie-2_SMD_Pad0.5mm" (id 2) (at 121.7462 110.49 0)
-      (effects (font (size 1.27 1.27)) hide)
-    )
-    (property "Datasheet" "~" (id 3) (at 121.7462 110.49 0)
-      (effects (font (size 1.27 1.27)) hide)
-    )
-    (pin "1")
-    (pin "2")
-  )
   (symbol (lib_id "Device:R") (at 92.71 91.44 270) (unit 1)
