File: pendulum_daughterboard/Driver PCB/Drive_Circuit.kicad_sch (KiCad schematic)
At the start: 16 parts, among them IC5 MAX9928FAUA+, J2 Coil, Q1 BC557, Q2 BC547

Commit message: Changed Diode
Parts:
- D4: footprint Diode_SMD:D_0603_1608Metric_Pad1.05x0.95mm_HandSolder -> Diode_THT:D_5KPW_P12.70mm_Horizontal
Changed lines of the file:
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@@
     (property "Reference" "D4" (id 0) (at 165.1 92.71 0))
     (property "Value" "1N4002" (id 1) (at 160.02 92.71 0))
-    (property "Footprint" "Diode_SMD:D_0603_1608Metric_Pad1.05x0.95mm_HandSolder" (id 2) (at 162.56 92.71 0)
+    (property "Footprint" "Diode_THT:D_5KPW_P12.70mm_Horizontal" (id 2) (at 162.56 92.71 0)
       (effects (font (size 1.27 1.27)) hide)
     )
