File: Interns_PCBs/Intern_PCB_FAB/Intern_PCB_FAB.kicad_pcb (KiCad board)
At the start: 2 copper layers, 160 x 100 mm, 13 parts, among them J1 Fan, J2 Arduino Serial, J3 Pi Header

Commit message: sdfgsrfg
Parts:
- added A1: Infineon Motor Shield MOD, Audio_Module:Infineon Motor Sheild hiddenPins, F.Cu at (204.3, 122.4)
- added A1: Infineon Motor Shield MOD, Audio_Module:Infineon Motor Sheild hiddenPins, F.Cu at (144.9, 124.4)
- added C1: 470u, Capacitor_SMD:C_Elec_8x10.2, F.Cu at (154.8, 70.2)
- added C1: 470u, Capacitor_SMD:C_Elec_8x10.2, F.Cu at (214.3, 68.1)
- added C2: 10u, Capacitor_SMD:CP_Elec_3x5.3, F.Cu at (222.8, 111.1)
- added C2: 10u, Capacitor_SMD:CP_Elec_3x5.3, F.Cu at (163.3, 113.1)
- added C3: 0.1u, Capacitor_SMD:C_0805_2012Metric_Pad1.18x1.45mm_HandSolder, F.Cu at (223.5, 114.6)
- added C3: 0.1u, Capacitor_SMD:C_0805_2012Metric_Pad1.18x1.45mm_HandSolder, F.Cu at (164.0, 116.7)
- added C4: 100nF, Capacitor_SMD:C_0805_2012Metric_Pad1.18x1.45mm_HandSolder, F.Cu at (134.3, 95.3)
- added C4: 100nF, Capacitor_SMD:C_0805_2012Metric_Pad1.18x1.45mm_HandSolder, F.Cu at (193.8, 93.3)
- added C5: 100nF, Capacitor_SMD:C_0805_2012Metric_Pad1.18x1.45mm_HandSolder, F.Cu at (123.1, 109.3)
- added C5: 100nF, Capacitor_SMD:C_0805_2012Metric_Pad1.18x1.45mm_HandSolder, F.Cu at (182.6, 107.3)
- added C6: 100nF, Capacitor_SMD:C_0805_2012Metric_Pad1.18x1.45mm_HandSolder, F.Cu at (182.1, 68.2)
- added C6: 100nF, Capacitor_SMD:C_0805_2012Metric_Pad1.18x1.45mm_HandSolder, F.Cu at (122.6, 70.2)
- added C7: 100nF, Capacitor_SMD:C_0805_2012Metric_Pad1.18x1.45mm_HandSolder, F.Cu at (208.7, 116.7)
- added C7: 100nF, Capacitor_SMD:C_0805_2012Metric_Pad1.18x1.45mm_HandSolder, F.Cu at (149.3, 118.7)
- added C8: 100nF, Capacitor_SMD:C_0805_2012Metric_Pad1.18x1.45mm_HandSolder, F.Cu at (218.9, 80.8)
- added C8: 100nF, Capacitor_SMD:C_0805_2012Metric_Pad1.18x1.45mm_HandSolder, F.Cu at (159.5, 82.9)
- added C9: 0.1uF, Capacitor_SMD:C_0805_2012Metric_Pad1.18x1.45mm_HandSolder, F.Cu at (219.4, 77.5)
- added C9: 0.1uF, Capacitor_SMD:C_0805_2012Metric_Pad1.18x1.45mm_HandSolder, F.Cu at (160.0, 79.6)
- added D1: LED, LED_SMD:LED_0805_2012Metric_Pad1.15x1.40mm_HandSolder, F.Cu at (129.2, 121.5)
- added D1: LED, LED_SMD:LED_0805_2012Metric_Pad1.15x1.40mm_HandSolder, F.Cu at (188.7, 119.4)
- added D2: LED, LED_SMD:LED_0805_2012Metric_Pad1.15x1.40mm_HandSolder, F.Cu at (129.2, 125.3)
- added D2: LED, LED_SMD:LED_0805_2012Metric_Pad1.15x1.40mm_HandSolder, F.Cu at (188.7, 123.3)
- added D3: LED, LED_SMD:LED_0805_2012Metric_Pad1.15x1.40mm_HandSolder, F.Cu at (188.7, 127.1)
- added D3: LED, LED_SMD:LED_0805_2012Metric_Pad1.15x1.40mm_HandSolder, F.Cu at (129.2, 129.1)
- added D4: 1N4002, Diode_THT:D_T-1_P5.08mm_Horizontal, F.Cu at (198.1, 72.2)
- added D4: 1N4002, Diode_THT:D_T-1_P5.08mm_Horizontal, F.Cu at (138.6, 74.3)
- added G***: LOGO, 000_Graphics_Immo:practactable.io_text_30x11_SM, F.Cu at (96.3, 130.7)
- added G***: LOGO, 000_Graphics_Immo:practactable.io_text_10x4, F.Cu at (215.1, 122.5)
- added G***: LOGO, 000_Graphics_Immo:practactable.io_text_10x4, F.Cu at (155.7, 124.5)
- added G***: LOGO, 000_Graphics_Immo:practactable.io_text_30x11_SM, F.Cu at (88.3, 115.7)
- added IC1: AND GATES, ICPINS:SOIC127P600X175-14N, F.Cu at (188.7, 87.5)
- added IC1: AND GATES, ICPINS:SOIC127P600X175-14N, F.Cu at (129.2, 89.5)
- added IC2: NAND (Used as AND), ICPINS:SOIC127P600X175-14N, F.Cu at (130.0, 111.1)
- added IC2: NAND (Used as AND), ICPINS:SOIC127P600X175-14N, F.Cu at (189.5, 109.0)
- added IC3: NAND (Used as Inverter), ICPINS:SOIC127P600X175-14N, F.Cu at (129.2, 72.0)
- added IC3: NAND (Used as Inverter), ICPINS:SOIC127P600X175-14N, F.Cu at (188.7, 69.9)
- added IC4: OR, ICPINS:SOIC127P600X175-14N, F.Cu at (147.3, 125.1)
- added IC4: OR, ICPINS:SOIC127P600X175-14N, F.Cu at (206.7, 123.0)
- added IC5: MAX9928FAUA+, Sensor_Current:SOP65P490X110-8N, F.Cu at (153.3, 78.9)
- added IC5: MAX9928FAUA+, Sensor_Current:SOP65P490X110-8N, F.Cu at (212.7, 76.8)
- added J1: Fan, Connector_Molex:Molex_KK-254_AE-6410-02A_1x02_P2.54mm_Vertical, F.Cu at (84.7, 61.3)
- added J1: AVR-ISP-6, Connector_PinHeader_2.00mm:PinHeader_2x03_P2.00mm_Vertical, F.Cu at (146.3, 96.6)
- added J1: AVR-ISP-6, Connector_PinHeader_2.00mm:PinHeader_2x03_P2.00mm_Vertical, F.Cu at (205.7, 94.6)
- added J2: Coil, Connector_Molex:RSPROPenduinoTerminal, F.Cu at (142.9, 68.4)
- added J2: Coil, Connector_Molex:RSPROPenduinoTerminal, F.Cu at (202.4, 66.4)
- added J2: Arduino Serial, Connector_Molex:Molex_KK-254_AE-6410-05A_1x05_P2.54mm_Vertical, F.Cu at (84.6, 92.2)
- added J3: Pi Header, Connector_PinHeader_2.54mm:PinHeader_2x20_P2.54mm_Vertical, F.Cu at (75.9, 56.1)
- added J4: Conn_01x04, Connector_PinHeader_1.27mm:PinHeader_1x04_P1.27mm_Vertical, F.Cu at (115.8, 126.7)
- added J4: Conn_01x04, Connector_PinHeader_1.27mm:PinHeader_1x04_P1.27mm_Vertical, F.Cu at (175.2, 124.6)
- added J5: DRIVE_GND, Connector_Pin:Pin_D1.3mm_L11.0mm, F.Cu at (223.7, 118.2)
- added J5: DRIVE_GND, Connector_Pin:Pin_D1.3mm_L11.0mm, F.Cu at (164.3, 120.2)
- added J7: DRIVE_5V_IN, Connector_Pin:Pin_D1.3mm_L11.0mm, F.Cu at (206.5, 65.1)
- added J7: DRIVE_5V_IN, Connector_Pin:Pin_D1.3mm_L11.0mm, F.Cu at (147.0, 67.1)
- added JP1: Shunt Bypass, Jumper:SolderJumper-2_P1.3mm_Open_Pad1.0x1.5mm, F.Cu at (202.4, 77.7)
- added JP1: Shunt Bypass, Jumper:SolderJumper-2_P1.3mm_Open_Pad1.0x1.5mm, F.Cu at (142.9, 79.8)
- added NT1: NetTie_2, NetTie:NetTie-2_SMD_Pad0.5mm, F.Cu at (217.1, 77.9)
- added NT1: NetTie_2, NetTie:NetTie-2_SMD_Pad0.5mm, F.Cu at (157.6, 79.9)
- added NT2: NetTie_2, NetTie:NetTie-2_SMD_Pad0.5mm, F.Cu at (217.1, 76.5)
- added NT2: NetTie_2, NetTie:NetTie-2_SMD_Pad0.5mm, F.Cu at (157.6, 78.5)
- added NT3: NetTie_2, NetTie:NetTie-2_SMD_Pad0.5mm, F.Cu at (149.0, 76.5)
- added NT3: NetTie_2, NetTie:NetTie-2_SMD_Pad0.5mm, F.Cu at (208.5, 74.5)
- added NT4: NetTie_2, NetTie:NetTie-2_SMD_Pad0.5mm, F.Cu at (208.2, 77.3)
- added NT4: NetTie_2, NetTie:NetTie-2_SMD_Pad0.5mm, F.Cu at (148.8, 79.3)
- added NT5: NetTie_2, NetTie:NetTie-2_SMD_Pad0.5mm, F.Cu at (210.5, 74.2)
- added NT5: NetTie_2, NetTie:NetTie-2_SMD_Pad0.5mm, F.Cu at (151.1, 76.3)
- added NT6: NetTie_2, NetTie:NetTie-2_SMD_Pad0.5mm, F.Cu at (217.1, 75.3)
- added NT6: NetTie_2, NetTie:NetTie-2_SMD_Pad0.5mm, F.Cu at (157.6, 77.4)
- added Q1: BC557, Package_TO_SOT_SMD:SOT-23, F.Cu at (201.1, 82.4)
- added Q1: BC557, Package_TO_SOT_SMD:SOT-23, F.Cu at (141.7, 84.4)
- added Q2: BC547, Package_TO_SOT_SMD:SOT-23, F.Cu at (204.9, 84.5)
- added Q2: BC547, Package_TO_SOT_SMD:SOT-23, F.Cu at (145.4, 86.6)
- added R1: 120, Resistor_SMD:R_0805_2012Metric_Pad1.20x1.40mm_HandSolder, F.Cu at (134.1, 121.5)
- added R1: 120, Resistor_SMD:R_0805_2012Metric_Pad1.20x1.40mm_HandSolder, F.Cu at (193.5, 119.4)
- added R2: 120, Resistor_SMD:R_0805_2012Metric_Pad1.20x1.40mm_HandSolder, F.Cu at (134.1, 125.3)
- added R2: 120, Resistor_SMD:R_0805_2012Metric_Pad1.20x1.40mm_HandSolder, F.Cu at (193.5, 123.3)
- added R3: 120, Resistor_SMD:R_0805_2012Metric_Pad1.20x1.40mm_HandSolder, F.Cu at (134.1, 129.1)
- added R3: 120, Resistor_SMD:R_0805_2012Metric_Pad1.20x1.40mm_HandSolder, F.Cu at (193.5, 127.1)
- added R4: 2k2, Resistor_SMD:R_0805_2012Metric_Pad1.20x1.40mm_HandSolder, F.Cu at (201.9, 89.0)
- added R4: 2k2, Resistor_SMD:R_0805_2012Metric_Pad1.20x1.40mm_HandSolder, F.Cu at (142.4, 91.0)
- added R5: 2k2, Resistor_SMD:R_0805_2012Metric_Pad1.20x1.40mm_HandSolder, F.Cu at (146.1, 90.8)
- added R5: 2k2, Resistor_SMD:R_0805_2012Metric_Pad1.20x1.40mm_HandSolder, F.Cu at (205.6, 88.7)
- added R6: 100k, Resistor_SMD:R_0805_2012Metric_Pad1.20x1.40mm_HandSolder, F.Cu at (151.8, 82.6)
- added R6: 100k, Resistor_SMD:R_0805_2012Metric_Pad1.20x1.40mm_HandSolder, F.Cu at (211.3, 80.6)
- added R7: 10R, Resistor_SMD:R_0805_2012Metric_Pad1.20x1.40mm_HandSolder, F.Cu at (202.7, 74.5)
- added R7: 10R, Resistor_SMD:R_0805_2012Metric_Pad1.20x1.40mm_HandSolder, F.Cu at (143.3, 76.6)
- added SW1: SW_Push, Button_Switch_SMD:13019319, F.Cu at (152.3, 107.5)
- added SW1: SW_Push, Button_Switch_SMD:13019319, F.Cu at (211.8, 105.5)
- added U10: ATtiny85-20S, Package_SO:SOIC-8W_5.3x5.3mm_P1.27mm, F.Cu at (154.6, 87.1)
- added U10: ATtiny85-20S, Package_SO:SOIC-8W_5.3x5.3mm_P1.27mm, F.Cu at (214.1, 85.0)
- moved J3 111.3 mm to (216.3, 45.0), turned to -90 degrees
- moved J1 107.8 mm to (211.2, 53.8), turned to 0 degrees
- moved J3 81.5 mm to (160.3, 44.7), turned to -90 degrees
- moved J1 74.8 mm to (155.1, 53.5), turned to 0 degrees
- moved J2 68.3 mm to (180.3, 53.6), turned to 180 degrees
- moved J3 47.8 mm to (93.0, 56.9), turned to 0 degrees
- moved J1 44.1 mm to (101.8, 62.1), turned to 90 degrees
- moved J2 34.1 mm to (101.6, 93.0), turned to -90 degrees
- moved J2 31.9 mm to (124.2, 53.3), turned to 180 degrees
Routing:
- net (no net): track 700.3 -> 4298.4 mm, vias 18 -> 150
- added copper zone on B.Cu, net (none)
Other:
- outline, holes or cut-outs redrawn
- board text added: "DRIVE_5V"
- board text added: "DRIVE_GND"
- board text added: "Eralp Calhan github.com/eralpcalhan"
- board text added: "Penduino Daughterboard"
