File: Interns_PCBs/pendulum_daughterboard/Driver PCB Version 2/Driver PCB Vol2/Driver PCB Vol2.kicad_pcb (KiCad board)
At the start: 2 copper layers, 69.2 x 54 mm, 79 parts, among them IC5 MAX9928FAUA+, J1 AVR-ISP-6, J2 Coil, J4 Conn_01x04, J5 DRIVE_GND, J7 DRIVE_5V_IN, Q1 BC557, Q2 BC547, SW1 SW_Push, U1 4081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

Commit message: One Connection Left
Routing:
- net Net-(D2-Pad2): track 44.2 -> 21.4 mm
- net Net-(D1-Pad2): track 52.2 -> 31.8 mm
- net Net-(R21-Pad2): track 59.1 -> 67.8 mm, vias 2 -> 3
- net D_GND: track 223.8 -> 220.2 mm, vias 12 -> 14
- net STU_LED_2: track 9.30 -> 12.4 mm
- net D_5V: track 201.0 -> 202.6 mm
