File: Interns_PCBs/pendulum_daughterboard/Driver PCB Version 3/Driver PCB Vol3/Microcontroller_Circuit_sch.kicad_sch (KiCad schematic)
At the start: 7 parts, among them J1 AVR-ISP-6, SW1 SW_Push, U10 ATtiny85-20S

Commit message: Flipped Diode on schematic
Connections:
- net GND: now also D5.1 (K); no longer D5.2 (A)
- net at R8.2: now also D5.2 (A); no longer D5.1 (K)
Other:
- moved on the sheet: D5
Changed lines of the file:
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@@
     (pin "2")
   )
-  (symbol (lib_id "Device:LED") (at 167.64 52.07 90) (unit 1)
+  (symbol (lib_id "Device:LED") (at 167.64 52.07 270) (unit 1)
     (in_bom yes) (on_board yes)
-    (property "Reference" "D5" (id 0) (at 165.1 52.07 0))
-    (property "Value" "LED" (id 1) (at 170.18 52.07 0))
+    (property "Reference" "D5" (id 0) (at 170.18 52.07 0))
+    (property "Value" "LED" (id 1) (at 165.1 52.07 0))
     (property "Footprint" "LED_SMD:LED_0805_2012Metric_Pad1.15x1.40mm_HandSolder" (id 2) (at 167.64 52.07 0)
       (effects (font (size 1.27 1.27)) hide)
