File: Interns_PCBs/pendulum_daughterboard/Driver PCB Version 3/Driver PCB Vol3/Driver PCB Vol3.kicad_pcb (KiCad board)
At the start: 2 copper layers, 69.2 x 54 mm, 66 parts, among them IC5 MAX9928FAUA+, J1 AVR-ISP-6, J2 Coil, J4 Conn_01x04, J5 DRIVE_GND, J7 DRIVE_5V_IN, Q1 BC557, Q2 BC547, SW1 SW_Push, U1 4081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

Commit message: changes on driver PCB
Parts:
- turned D5 to 180 degrees
Connections:
- D5 pad 1: Net-(D5-Pad1) -> D_GND
- D5 pad 2: D_GND -> Net-(D5-Pad2)
- R8 pad 2: Net-(D5-Pad1) -> Net-(D5-Pad2)
Routing:
- net Net-(D5-Pad2): track 0.00 -> 2.55 mm
- net Net-(D5-Pad1): track 2.55 -> 0.00 mm
