File: Interns_PCBs/pendulum_daughterboard/Driver PCB Version 4/LED_Circuit.kicad_sch (KiCad schematic)
At the start: 40 parts, among them J4 Conn_01x04, U1 4081, U2 4011, U3 4011, U4 4071

Commit message: Another Drive PCB
Parts:
- removed R10, R11, R12, R14, R16: 10k, Resistor_SMD:R_0805_2012Metric_Pad1.20x1.40mm_HandSolder, symbol Device:R
Connections:
- net 5V renamed 3.3V
