File: Interns_PCBs/pendulum_daughterboard/Driver PCB Version 4/untitled.kicad_sch (KiCad schematic)
At the start: 6 parts, among them U5 AMS1117-3.3, U6 AMS1117-3.3

Commit message: 3.3V PCB Design
PCB with 2 voltage regulators, regulating both the 5V input from the digital pins and the external 5V from the terminal block.
Changed lines of the file:
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@@
     (pin "2")
   )
-  (symbol (lib_id "000_Capacitor_Electrolytic_Immo:22u") (at 101.6 81.28 0) (unit 1)
+  (symbol (lib_id "000_Capacitor_Electrolytic_Immo:22u") (at 101.6 81.28 0) (mirror y) (unit 1)
     (in_bom yes) (on_board yes) (fields_autoplaced)
     (property "Reference" "EC1" (id 0) (at 105.41 79.1209 0)
-      (effects (font (size 1.27 1.27)) (justify left))
+      (effects (font (size 1.27 1.27)) (justify right))
     )
     (property "Value" "10u" (id 1) (at 105.41 81.6609 0)
-      (effects (font (size 1.27 1.27)) (justify left))
+      (effects (font (size 1.27 1.27)) (justify right))
     )
-    (property "Footprint" "Capacitor_SMD:CP_Elec_4x5.4" (id 2) (at 102.5652 85.09 0)
+    (property "Footprint" "Capacitor_SMD:CP_Elec_4x5.4" (id 2) (at 100.6348 85.09 0)
       (effects (font (size 1.27 1.27)) hide)
     )
