File: Interns_PCBs/pendulum_daughterboard/Driver PCB Level Shifter/Drive_Circuit.kicad_sch (KiCad schematic)
At the start: 13 parts, among them IC1 MAX9928FAUA+, J2 Coil, Q1 BC858W, Q2 BD911

Commit message: Penduino Daughterboard with Level Shifter
Connections:
- net PEND_3.3V renamed 5V
Changed lines of the file:
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@@
     (effects (font (size 1.27 1.27)) (justify right))
   )
-  (hierarchical_label "PEND_3.3V" (shape input) (at 279.4 66.04 90)
+  (hierarchical_label "5V" (shape input) (at 279.4 66.04 90)
     (effects (font (size 1.27 1.27)) (justify left))
   )
@@
     (effects (font (size 1.27 1.27)) (justify right))
   )
-  (hierarchical_label "PEND_3.3V" (shape input) (at 66.04 74.93 90)
+  (hierarchical_label "5V" (shape input) (at 66.04 74.93 90)
     (effects (font (size 1.27 1.27)) (justify left))
   )
