File: Interns_PCBs/pendulum_daughterboard/Driver PCB Level Shifter/Driver PCB Level Shifter.kicad_sch (KiCad schematic)
At the start: 4 parts

Commit message: Pin update
Connections:
- net DRIVE_INPUT: now also A1.19 (D4); no longer A1.27 (INH_1), A1.28 (INH_2)
- net LOAD_INPUT: now also A1.27 (INH_1), A1.28 (INH_2); no longer A1.19 (D4)
Changed lines of the file:
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@@
     )
   )
-  (global_label "DRIVE_INPUT" (shape output) (at 177.8 54.61 0) (fields_autoplaced)
-    (effects (font (size 1.27 1.27)) (justify left))
-    (property "Intersheet References" "${INTERSHEET_REFS}" (id 0) (at 192.0664 54.5306 0)
+  (global_label "LOAD_INPUT" (shape output) (at 177.8 54.61 0) (fields_autoplaced)
+    (effects (font (size 1.27 1.27)) (justify left))
+    (property "Intersheet References" "${INTERSHEET_REFS}" (id 0) (at 191.4012 54.5306 0)
       (effects (font (size 1.27 1.27)) (justify left) hide)
     )
@@
     )
   )
-  (global_label "LOAD_INPUT" (shape output) (at 177.8 77.47 0) (fields_autoplaced)
-    (effects (font (size 1.27 1.27)) (justify left))
-    (property "Intersheet References" "${INTERSHEET_REFS}" (id 0) (at 191.4012 77.3906 0)
+  (global_label "DRIVE_INPUT" (shape output) (at 177.8 77.47 0) (fields_autoplaced)
+    (effects (font (size 1.27 1.27)) (justify left))
+    (property "Intersheet References" "${INTERSHEET_REFS}" (id 0) (at 192.0664 77.3906 0)
       (effects (font (size 1.27 1.27)) (justify left) hide)
     )
@@
       (reference "C9") (unit 1) (value "0.1uF") (footprint "Capacitor_SMD:C_0805_2012Metric_Pad1.18x1.45mm_HandSolder")
     )
+    (path "/21780cc4-9565-4c48-acf2-9e239c61d608/c37e6299-d39f-48ad-b9e6-545b3ac22c42"
+      (reference "C10") (unit 1) (value "100nF") (footprint "Capacitor_SMD:C_0805_2012Metric_Pad1.18x1.45mm_HandSolder")
+    )
+    (path "/21780cc4-9565-4c48-acf2-9e239c61d608/307442c4-2d7f-45ee-8835-fc08eb57c8f2"
+      (reference "C11") (unit 1) (value "100nF") (footprint "Capacitor_SMD:C_0805_2012Metric_Pad1.18x1.45mm_HandSolder")
+    )
     (path "/1a3370a0-6778-4601-bc8e-4c18ed659ac3/90554270-e835-46bf-8bb7-64ab2c34bc4f"
