File: Interns_PCBs/pendulum_daughterboard/Driver PCB Level Shifter/untitled.kicad_sch (KiCad schematic)
At the start: 8 parts, among them U5 AMS1117-3.3, U6 SN74LVC2T45DCUR

Commit message: Pin update
Parts:
- added C10, C11: 100nF, Capacitor_SMD:C_0805_2012Metric_Pad1.18x1.45mm_HandSolder, symbol Device:C
Connections:
- net 3.3V: now also C11.1
- net 5V: now also C10.1
- net GND: now also C10.2, C11.2
Changed lines of the file:
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@@
   (junction (at 186.69 73.66) (diameter 0) (color 0 0 0 0)
   )
+  (junction (at 205.74 59.69) (diameter 0) (color 0 0 0 0)
+  )
   (junction (at 226.06 78.74) (diameter 0) (color 0 0 0 0)
   )
@@
   (junction (at 85.09 69.85) (diameter 0) (color 0 0 0 0)
   )
+  (junction (at 210.82 60.96) (diameter 0) (color 0 0 0 0)
+  )
   (junction (at 208.28 88.9) (diameter 0) (color 0 0 0 0)
   )
@@
     (stroke (width 0) (type default) (color 0 0 0 0))
   )
+  (wire (pts (xy 226.06 57.15) (xy 226.06 62.23))
+    (stroke (width 0) (type default) (color 0 0 0 0))
+  )
   (wire (pts (xy 226.06 73.66) (xy 233.68 73.66))
     (stroke (width 0) (type default) (color 0 0 0 0))
@@
     (stroke (width 0) (type default) (color 0 0 0 0))
   )
+  (wire (pts (xy 205.74 59.69) (xy 205.74 63.5))
+    (stroke (width 0) (type default) (color 0 0 0 0))
+  )
   (wire (pts (xy 85.09 69.85) (xy 93.98 69.85))
     (stroke (width 0) (type default) (color 0 0 0 0))
@@
     (stroke (width 0) (type default) (color 0 0 0 0))
   )
-  (wire (pts (xy 226.06 57.15) (xy 226.06 62.23))
-    (stroke (width 0) (type default) (color 0 0 0 0))
-  )
   (wire (pts (xy 101.6 77.47) (xy 101.6 80.01))
     (stroke (width 0) (type default) (color 0 0 0 0))
   )
-  (wire (pts (xy 205.74 57.15) (xy 205.74 63.5))
+  (wire (pts (xy 210.82 60.96) (xy 210.82 63.5))
+    (stroke (width 0) (type default) (color 0 0 0 0))
+  )
+  (wire (pts (xy 205.74 57.15) (xy 205.74 59.69))
     (stroke (width 0) (type default) (color 0 0 0 0))
   )
@@
     (stroke (width 0) (type default) (color 0 0 0 0))
   )
-  (wire (pts (xy 210.82 57.15) (xy 210.82 63.5))
+  (wire (pts (xy 210.82 57.15) (xy 210.82 60.96))
+    (stroke (width 0) (type default) (color 0 0 0 0))
+  )
+  (wire (pts (xy 210.82 60.96) (xy 212.09 60.96))
     (stroke (width 0) (type default) (color 0 0 0 0))
   )
@@
     (effects (font (size 1.27 1.27)) (justify right))
   )
+  (hierarchical_label "GND" (shape input) (at 219.71 60.96 0)
+    (effects (font (size 1.27 1.27)) (justify left))
+  )
   (hierarchical_label "DRIVE_INPUT" (shape input) (at 233.68 73.66 0)
     (effects (font (size 1.27 1.27)) (justify left))
@@
     (effects (font (size 1.27 1.27)) (justify right))
   )
+  (hierarchical_label "GND" (shape input) (at 198.12 59.69 180)
+    (effects (font (size 1.27 1.27)) (justify right))
+  )
   (symbol (lib_id "Device:R") (at 186.69 85.09 0) (unit 1)
     (in_bom yes) (on_board yes) (fields_autoplaced)
@@
     )
     (property "Datasheet" "~" (id 3) (at 85.09 74.93 0)
+      (effects (font (size 1.27 1.27)) hide)
+    )
+    (pin "1")
+    (pin "2")
+  )
+  (symbol (lib_id "Device:C") (at 215.9 60.96 90) (unit 1)
+    (in_bom yes) (on_board yes) (fields_autoplaced)
+    (property "Reference" "C11" (id 0) (at 214.6299 57.15 0)
+      (effects (font (size 1.27 1.27)) (justify left))
+    )
+    (property "Value" "100nF" (id 1) (at 217.1699 57.15 0)
+      (effects (font (size 1.27 1.27)) (justify left))
+    )
+    (property "Footprint" "Capacitor_SMD:C_0805_2012Metric_Pad1.18x1.45mm_HandSolder" (id 2) (at 219.71 59.9948 0)
+      (effects (font (size 1.27 1.27)) hide)
+    )
+    (property "Datasheet" "~" (id 3) (at 215.9 60.96 0)
       (effects (font (size 1.27 1.27)) hide)
     )
@@
     (pin "3")
   )
+  (symbol (lib_id "Device:C") (at 201.93 59.69 270) (unit 1)
+    (in_bom yes) (on_board yes)
+    (property "Reference" "C10" (id 0) (at 203.2 52.07 0)
+      (effects (font (size 1.27 1.27)) (justify left))
+    )
+    (property "Value" "100nF" (id 1) (at 200.66 50.8 0)
+      (effects (font (size 1.27 1.27)) (justify left))
+    )
+    (property "Footprint" "Capacitor_SMD:C_0805_2012Metric_Pad1.18x1.45mm_HandSolder" (id 2) (at 198.12 60.6552 0)
+      (effects (font (size 1.27 1.27)) hide)
+    )
+    (property "Datasheet" "~" (id 3) (at 201.93 59.69 0)
+      (effects (font (size 1.27 1.27)) hide)
+    )
+    (pin "1")
+    (pin "2")
+  )
 )

Commit message: new PCB design started
Parts:
- removed C10, C11: 100nF, Capacitor_SMD:C_0805_2012Metric_Pad1.18x1.45mm_HandSolder, symbol Device:C
- removed EC1, EC2: 10u, Capacitor_SMD:CP_Elec_4x5.4, symbol 000_Capacitor_Electrolytic_Immo:22u
- removed U5: AMS1117-3.3, Package_TO_SOT_SMD:SOT-223-3_TabPin2, symbol Regulator_Linear:AMS1117-3.3
- removed U6: SN74LVC2T45DCUR, Package_SO:VSSOP-8_2.4x2.1mm_P0.5mm, symbol Logic_LevelTranslator:SN74LVC2T45DCUR
- added Q3, Q4: BSS138, Package_TO_SOT_SMD:SOT-23, symbol Transistor_FET:BSS138
- R10, R11, R12, R14: value 10K -> 10k; footprint Resistor_SMD:R_0805_2012Metric_Pad1.20x1.40mm_HandSolder -> (none)
Connections:
- net LOAD_INPUT is gone; now on net 5V: R14.1
- net 3.3V: now also R10.1, R12.1, Q3.1 (G), Q4.1 (G)
- net 5V: now also R11.1
- net DRIVE: now also R11.2, Q3.3 (D); no longer R10.2
- net LOAD: now also R14.2, Q4.3 (D); no longer R11.1
- net DRIVE_INPUT renamed LOAD_IN
- net LOAD_IN: now also Q4.2 (S)
- removed net GND: R10.1, R11.2, R12.1, R14.2
- new net DRIVE_IN: Q3.2 (S), R10.2

Commit message: Level Shifting Daughterboard
Parts:
- R10, R11, R12, R14: footprint (none) -> Resistor_SMD:R_0805_2012Metric_Pad1.20x1.40mm_HandSolder
Changed lines of the file:
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@@
       (effects (font (size 1.27 1.27)) (justify left))
     )
-    (property "Footprint" "" (id 2) (at 174.752 50.8 90)
+    (property "Footprint" "Resistor_SMD:R_0805_2012Metric_Pad1.20x1.40mm_HandSolder" (id 2) (at 174.752 50.8 90)
       (effects (font (size 1.27 1.27)) hide)
     )
@@
       (effects (font (size 1.27 1.27)) (justify left))
     )
-    (property "Footprint" "" (id 2) (at 107.442 50.8 90)
+    (property "Footprint" "Resistor_SMD:R_0805_2012Metric_Pad1.20x1.40mm_HandSolder" (id 2) (at 107.442 50.8 90)
       (effects (font (size 1.27 1.27)) hide)
     )
@@
       (effects (font (size 1.27 1.27)) (justify left))
     )
-    (property "Footprint" "" (id 2) (at 195.072 50.8 90)
+    (property "Footprint" "Resistor_SMD:R_0805_2012Metric_Pad1.20x1.40mm_HandSolder" (id 2) (at 195.072 50.8 90)
       (effects (font (size 1.27 1.27)) hide)
     )
@@
       (effects (font (size 1.27 1.27)) (justify left))
     )
-    (property "Footprint" "" (id 2) (at 87.122 50.8 90)
+    (property "Footprint" "Resistor_SMD:R_0805_2012Metric_Pad1.20x1.40mm_HandSolder" (id 2) (at 87.122 50.8 90)
       (effects (font (size 1.27 1.27)) hide)
     )
