File: Interns_PCBs/pendulum_daughterboard/Driver PCB Level Shifter/Microcontroller_Circuit_sch.kicad_sch (KiCad schematic)
At the start: 7 parts, among them J1 AVR-ISP-6, SW1 SW_Push, U7 ATtiny85-20S

Commit message: Penduino Daughterboard with Level Shifter
Connections:
- net 3.3V renamed 5V
Changed lines of the file:
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@@
     (stroke (width 0) (type default) (color 0 0 0 0))
   )
-  (wire (pts (xy 146.05 30.48) (xy 146.05 33.02))
+  (wire (pts (xy 146.05 29.21) (xy 146.05 33.02))
     (stroke (width 0) (type default) (color 0 0 0 0))
   )
@@
     (stroke (width 0) (type default) (color 0 0 0 0))
   )
-  (global_label "3.3V" (shape input) (at 146.05 30.48 90) (fields_autoplaced)
-    (effects (font (size 1.27 1.27)) (justify left))
-    (property "Intersheet References" "${INTERSHEET_REFS}" (id 0) (at 145.9706 23.9545 90)
-      (effects (font (size 1.27 1.27)) (justify left) hide)
-    )
-  )
   (hierarchical_label "GND" (shape input) (at 104.14 104.14 90)
     (effects (font (size 1.27 1.27)) (justify left))
@@
   (hierarchical_label "DRIVE_OUT" (shape output) (at 168.91 90.17 180)
     (effects (font (size 1.27 1.27)) (justify right))
+  )
+  (hierarchical_label "5V" (shape input) (at 146.05 29.21 90)
+    (effects (font (size 1.27 1.27)) (justify left))
   )
   (hierarchical_label "GND" (shape input) (at 143.51 153.67 270)
@@
     (effects (font (size 1.27 1.27)) (justify left))
   )
-  (hierarchical_label "3.3V" (shape input) (at 158.75 113.03 0)
+  (hierarchical_label "5V" (shape input) (at 158.75 113.03 0)
     (effects (font (size 1.27 1.27)) (justify left))
   )

Commit message: Truss Test
Parts:
- renumbered U7 to U5
Changed lines of the file:
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@@
   (symbol (lib_id "MCU_Microchip_ATtiny:ATtiny85-20S") (at 190.5 87.63 0) (mirror y) (unit 1)
     (in_bom yes) (on_board yes) (fields_autoplaced)
-    (property "Reference" "U7" (id 0) (at 204.47 86.3599 0)
+    (property "Reference" "U5" (id 0) (at 204.47 86.3599 0)
       (effects (font (size 1.27 1.27)) (justify right))
     )
