File: Interns_PCBs/pendulum_daughterboard/Drive PCB Level Shifting External Sources/Drive PCB Level Shifting External Sources.kicad_sch (KiCad schematic)
At the start: 7 parts, among them J3 DRIVE_GND, J4 DRIVE_5V, J5 3.3V

Commit message: new PCB design started
Parts:
- removed J3: DRIVE_GND, Connector_Pin:Pin_D1.3mm_L11.0mm, symbol Connector_Generic:Conn_01x01
- removed J4: DRIVE_5V, Connector_Pin:Pin_D1.3mm_L11.0mm, symbol Connector_Generic:Conn_01x01
- removed J5: 3.3V, Connector_Pin:Pin_D1.3mm_L11.0mm, symbol Connector_Generic:Conn_01x01
Connections:
- net D_5V is gone; now on net 5V: A1.5 (5V)
- net D_GND is gone; now on net GND: A1.7 (GND)
Other:
- sheet Linear Voltage Conversion ports: added DRIVE_INPUT, GND, LOAD_INPUT; removed 3.3V, DRIVE_IN, LOAD_IN
