File: Interns_PCBs/pendulum_daughterboard/Drive PCB Level Shifting External Sources/LED_Circuit.kicad_sch (KiCad schematic)
At the start: 35 parts, among them J6 Conn_01x04, U1 4081, U2 4011, U3 4011, U4 4071

Commit message: new PCB design started
Parts:
- renumbered J6 to J4
Changed lines of the file:
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@@
   (symbol (lib_id "Connector_Generic:Conn_01x04") (at 281.94 86.36 0) (mirror x) (unit 1)
     (in_bom yes) (on_board yes) (fields_autoplaced)
-    (property "Reference" "J6" (id 0) (at 281.94 74.93 0))
+    (property "Reference" "J4" (id 0) (at 281.94 74.93 0))
     (property "Value" "Conn_01x04" (id 1) (at 281.94 77.47 0))
     (property "Footprint" "Connector_PinHeader_2.54mm:PinHeader_1x04_P2.54mm_Vertical" (id 2) (at 281.94 86.36 0)
